Commit message: El diablooo

File: robot_description/frida_description/urdf/lidar.xacro (robot description, xacro)
@@ -1,5 +1,5 @@
 <?xml version="1.0" encoding="utf-8"?>
 <robot xmlns:xacro="http://www.ros.org/wiki/xacro">
-<link name="LIDAR">
+<link name="laser">
     <inertial>
       <origin xyz="-1.3878E-17 3.3818E-34 -0.0125" rpy="0 0 0" />
@@ -25,7 +25,7 @@
   </link>
   <joint name="lidar" type="fixed">
-    <origin xyz="0.15026 0 0.002" rpy="3.1416 0 0" />
+    <origin xyz="0.15026 0 0.002" rpy="0 0 -1.57" />
     <parent link="base_link" />
-    <child link="LIDAR" />
+    <child link="laser" />
     <axis xyz="0 0 0" />
   </joint>
