Commit message: Fixed xacro insano

File: robot_description/frida_description/urdf/FRIDA_Real.urdf.xacro (robot description, xacro)
@@ -1,4 +1,5 @@
 <?xml version="1.0" encoding="utf-8"?>
 <robot name="FRIDA" xmlns:xacro="http://www.ros.org/wiki/xacro">
+<!-- XARM ARGUMENTS -->
   <xacro:arg name="prefix" default=""/>
   <xacro:arg name="hw_ns" default="xarm"/>
@@ -39,6 +40,16 @@
   <xacro:arg name="mesh_suffix" default="stl"/>
   <xacro:arg name="kinematics_suffix" default=""/>
-  <xacro:arg name="sim_mode" default="true"/>
+  <!-- ZED ARGUMENTS -->
+  <xacro:arg name="camera_name"   default="zed" />
+  <xacro:arg name="camera_model"  default="zed2" />
+  <xacro:arg name="custom_baseline"  default="0.0" />
+  <!-- If GNSS fusion is enabled the position of the antenna with respect to the camera mount point is required -->
+  <xacro:arg name="enable_gnss"   default="false" />
+  <xacro:arg name="gnss_x" default="0.0" />
+  <xacro:arg name="gnss_y" default="0.0" />
+  <xacro:arg name="gnss_z" default="0.0" />
+  <!-- ROBOT COMPONENTS -->
   <xacro:include filename="robot_real.xacro"/>
+  <!-- XARM MACRO -->
   <xacro:include filename="$(find xarm_description)/urdf/xarm_device_macro.xacro" />
     <xacro:xarm_device prefix="$(arg prefix)" hw_ns="$(arg hw_ns)" limited="$(arg limited)"
@@ -61,22 +72,13 @@
     model1300="$(arg model1300)" attach_to="$(arg attach_to)" attach_xyz="$(arg attach_xyz)" attach_rpy="$(arg attach_rpy)"
     robot_sn="$(arg robot_sn)" use_gazebo_camera="$(arg use_gazebo_camera)" mesh_suffix="$(arg mesh_suffix)" kinematics_suffix="$(arg kinematics_suffix)" />
- <!-- Gripper -->
+  <!-- Gripper -->
   <xacro:include filename="gripper.xacro" />
-  <xacro:load_gripper attach_to="link_eef" xyz="0 0 0" rpy="2.3562 -1.5708 0" />
-  <!-- <xacro:include filename="zed.xacro" /> -->
-  <!-- <xacro:load_zed attach_to="gripper" xyz="0.030461 0 -0.050649" rpy="0 0.81804 0" /> -->
-  <!-- <xacro:arg name="camera_name"   default="zed" />
-  <xacro:arg name="camera_model"  default="zed2" />
-  <xacro:arg name="custom_baseline"  default="0.0" /> -->
-  <!-- If GNSS fusion is enabled the position of the antenna with respect to the camera mount point is required -->
-  <!-- <xacro:arg name="enable_gnss"   default="false" />
-  <xacro:arg name="gnss_x" default="0.0" />
-  <xacro:arg name="gnss_y" default="0.0" />
-  <xacro:arg name="gnss_z" default="0.0" />
+    <xacro:load_gripper attach_to="link_eef" xyz="0 0 0" rpy="2.3562 -1.5708 0" />
+   <!-- ZED MACRO -->
   <xacro:include filename="$(find frida_description)/urdf/zed_macro.urdf.xacro" />
-  <xacro:zed_camera name="$(arg camera_name)" model="$(arg camera_model)" custom_baseline="$(arg custom_baseline)" enable_gnss="$(arg enable_gnss)">
-	    <origin xyz="$(arg gnss_x) $(arg gnss_y) $(arg gnss_z)" rpy="0 0 0"/>
-  </xacro:zed_camera>
-  <joint name="base_footprint_joint" type="fixed">
+    <xacro:zed_camera name="$(arg camera_name)" model="$(arg camera_model)" custom_baseline="$(arg custom_baseline)" enable_gnss="$(arg enable_gnss)">
+	      <origin xyz="$(arg gnss_x) $(arg gnss_y) $(arg gnss_z)" rpy="0 0 0"/>
+    </xacro:zed_camera>
+  <!-- <joint name="base_footprint_joint" type="fixed">
       <origin xyz="0 0 ${base_length/2 + caster_radius*2}" rpy="0 0 0" />
       <parent link="base_footprint"/>

File: robot_description/frida_description/urdf/zed_macro.urdf.xacro (robot description, xacro)
@@ -107,5 +107,5 @@
     </xacro:if>
     <!-- Camera mounting point (the threaded screw hole in the bottom) -->
-    <link name="${name}_camera_link" />
+    <!-- <link name="${name}_camera_link" /> -->
     <!-- Camera Center -->
     <link name="${name}_camera_center">
@@ -127,7 +127,9 @@
     </link>
     <joint name="${name}_camera_center_joint" type="fixed">
-      <parent link="${name}_camera_link"/>
+      <!-- <parent link="${name}_camera_link"/> -->
+      <parent link="gripper"/>
       <child link="${name}_camera_center"/>
-      <origin xyz="0 0 ${height/2}" rpy="0 ${bottom_slope} 0" />
+      <!-- <origin xyz="0 0 ${height/2}" rpy="0 ${bottom_slope} 0" /> -->
+      <origin xyz="0.030461 0 -0.050649" rpy="0 0.81804 0" />
     </joint>
     <xacro:unless value="${mono}">
@@ -236,5 +238,6 @@
       <link name="${name}_gnss_link" />
       <joint name="${name}_gnss_joint" type="fixed">
-        <parent link="${name}_camera_link"/>
+        <!-- <parent link="${name}_camera_link"/> -->
+        <parent link="gripper"/>
         <child link="${name}_gnss_link"/>
         <xacro:insert_block name="gnss_origin" />

Commit message: Added fixed urdf real zed

File: robot_description/frida_description/urdf/FRIDA_Real.urdf.xacro (robot description, xacro)
@@ -41,12 +41,4 @@
   <xacro:arg name="kinematics_suffix" default=""/>
   <!-- ZED ARGUMENTS -->
-  <xacro:arg name="camera_name"   default="zed" />
-  <xacro:arg name="camera_model"  default="zed2" />
-  <xacro:arg name="custom_baseline"  default="0.0" />
-  <!-- If GNSS fusion is enabled the position of the antenna with respect to the camera mount point is required -->
-  <xacro:arg name="enable_gnss"   default="false" />
-  <xacro:arg name="gnss_x" default="0.0" />
-  <xacro:arg name="gnss_y" default="0.0" />
-  <xacro:arg name="gnss_z" default="0.0" />
   <!-- ROBOT COMPONENTS -->
   <xacro:include filename="robot_real.xacro"/>
@@ -76,8 +68,6 @@
     <xacro:load_gripper attach_to="link_eef" xyz="0 0 0" rpy="2.3562 -1.5708 0" />
    <!-- ZED MACRO -->
-  <xacro:include filename="$(find frida_description)/urdf/zed_macro.urdf.xacro" />
-    <xacro:zed_camera name="$(arg camera_name)" model="$(arg camera_model)" custom_baseline="$(arg custom_baseline)" enable_gnss="$(arg enable_gnss)">
-	      <origin xyz="$(arg gnss_x) $(arg gnss_y) $(arg gnss_z)" rpy="0 0 0"/>
-    </xacro:zed_camera>
+    <xacro:include filename="zed.xacro" />
+  <xacro:load_zed attach_to="gripper" xyz="0.030461 0 -0.050649" rpy="0 0.81804 0" />
   <!-- <joint name="base_footprint_joint" type="fixed">
       <origin xyz="0 0 ${base_length/2 + caster_radius*2}" rpy="0 0 0" />

File: robot_description/frida_description/urdf/zed.xacro (robot description, xacro)
@@ -6,9 +6,9 @@
       <joint name="zed" type="fixed">
         <parent link="${attach_to}"/>
-        <child link="ZED"/>
+        <child link="zed_camera_link"/>
         <origin xyz="${xyz}" rpy="${rpy}"/>
       </joint>
     </xacro:unless>
-<link name="ZED">
+<link name="zed_camera_link">
     <inertial>
       <origin xyz="0.00022189 -2.7346E-06 1.8693E-05" rpy="0 0 0" />
@@ -33,14 +33,4 @@
     </collision>
   </link>
-  <!--
-  <joint
-    name="zed"
-    type="fixed">
-    <origin xyz="0.030461 0 -0.050649" rpy="0 0.81804 0" />
-    <parent link="gripper" />
-    <child link="ZED" />
-    <axis xyz="0 0 0" />
-  </joint>
-  -->
 </xacro:macro>
 </robot>
