Commit message: Temporary workaround to avoid the robot moving by itself when is stationary in the gazebo simulation

File: robot_description/frida_description/urdf/wheels.xacro (robot description, xacro)
@@ -5,5 +5,5 @@
       <inertial>
         <origin xyz="-1.3878E-17 0 2.7756E-17" rpy="0 0 0" />
-        <mass value="0.52892" />
+        <mass value="100.52892" />
         <inertia ixx="0.00063131" ixy="${ixy}" ixz="${ixz}"
                  iyy="0.00063131" iyz="${iyz}" izz="0.0011216" />
