Commit message: Frida_description updated

File: robot_description/frida_description/urdf/FRIDA.urdf.xacro (robot description, xacro)
@@ -1,223 +1,4 @@
 <?xml version="1.0" encoding="utf-8"?>
 <robot name="FRIDA" xmlns:xacro="http://www.ros.org/wiki/xacro">
-<!-- Properties -->
-<xacro:property name="mesh_path" value="package://frida_description/urdf/meshes/" />
-<xacro:property name="material_rgba" value="0.792 0.820 0.933 1" />
-<xacro:property name="lidar_rgba" value="0.102 0.102 0.102 1" />
-<xacro:property name="intel_rgba" value="0.776 0.757 0.737 1" />
-  <!-- Base Link -->
-  <link name="base_link">
-    <inertial>
-      <origin xyz="-0.017897 -0.0059216 0.12557" rpy="0 0 0" />
-      <mass value="31.075" />
-      <inertia ixx="0.67537" ixy="-0.00030935" ixz="-0.0025852"
-               iyy="0.61552" iyz="-0.0003748" izz="0.65918" />
-    </inertial>
-    <visual>
-      <origin xyz="0 0 0" rpy="0 0 0" />
-      <geometry>
-        <mesh filename="${mesh_path}base_link.STL" />
-      </geometry>
-      <material name="">
-        <color rgba="${material_rgba}" />
-      </material>
-    </visual>
-    <collision>
-      <origin xyz="0 0 0" rpy="0 0 0" />
-      <geometry>
-        <mesh filename="${mesh_path}base_link.STL" />
-      </geometry>
-    </collision>
-  </link>
-  <!-- Wheels -->
-  <xacro:macro name="wheel_link" params="prefix ixy ixz iyz joint_origin">
-    <link name="${prefix}_wheel">
-      <inertial>
-        <origin xyz="-1.3878E-17 0 2.7756E-17" rpy="0 0 0" />
-        <mass value="0.52892" />
-        <inertia ixx="0.00063131" ixy="${ixy}" ixz="${ixz}"
-                 iyy="0.00063131" iyz="${iyz}" izz="0.0011216" />
-      </inertial>
-      <visual>
-        <origin xyz="0 0 0" rpy="0 0 0" />
-        <geometry>
-          <mesh filename="${mesh_path}${prefix}_wheel.STL" />
-        </geometry>
-        <material name="">
-          <color rgba="${lidar_rgba}" />
-        </material>
-      </visual>
-      <collision>
-        <origin xyz="0 0 0" rpy="0 0 0" />
-        <geometry>
-          <mesh filename="${mesh_path}${prefix}_wheel.STL" />
-        </geometry>
-      </collision>
-    </link>
-    <joint name="${prefix}wheel" type="continuous">
-      <origin xyz="${joint_origin}" rpy="-1.5708 0 0" />
-      <parent link="base_link" />
-      <child link="${prefix}_wheel" />
-      <axis xyz="0 0 1" />
-    </joint>
-  </xacro:macro>
-  <xacro:wheel_link prefix="right" ixy="-9.9049E-20" ixz="5.8265E-21" iyz="-2.2717E-21" joint_origin="-0.075244 -0.166 -0.0775" />
-  <xacro:wheel_link prefix="left" ixy="4.5051E-20" ixz="1.2238E-21" iyz="7.2483E-21" joint_origin="-0.075244 0.166 -0.0775" />
-  <!-- Castor Wheels Brackets-->
-  <xacro:macro name="castwheel_bracket" params="prefix inertial_origin ixy ixz iyz joint_origin">
-    <link name="${prefix}_castwheel_bracket">
-      <inertial>
-        <origin xyz="${inertial_origin}" rpy="0 0 0" />
-        <mass value="0.045185" />
-        <inertia ixx="1.9146E-05" ixy="${ixy}" ixz="${ixz}"
-                 iyy="2.036E-05" iyz="${iyz}" izz="1.5813E-05" />
-      </inertial>
-      <visual>
-        <origin xyz="0 0 0" rpy="0 0 0" />
-        <geometry>
-          <mesh filename="${mesh_path}${prefix}_castwheel_bracket.STL" />
-        </geometry>
-        <material name="">
-          <color rgba="${intel_rgba}" />
-        </material>
-      </visual>
-      <collision>
-        <origin xyz="0 0 0" rpy="0 0 0" />
-        <geometry>
-          <mesh filename="${mesh_path}${prefix}_castwheel_bracket.STL" />
-        </geometry>
-      </collision>
-    </link>
-    <joint name="${prefix}castwheelbracket" type="continuous">
-      <origin xyz="${joint_origin}" rpy="3.1416 0 0" />
-      <parent link="base_link" />
-      <child link="${prefix}_castwheel_bracket" />
-      <axis xyz="0 0 -1" />
-    </joint>
-  </xacro:macro>
-  <xacro:castwheel_bracket prefix="right" inertial_origin="-6.9389E-17 -1.3878E-17 0.012445" ixy="-5.23501237066605E-21" ixz="1.02910979879346E-20" iyz="1.03781586309714E-20" joint_origin="0.11226 -0.09 -0.068" />
-  <xacro:castwheel_bracket prefix="left" inertial_origin="0 -4.1633E-17 0.012445" ixy="2.58235447481398E-21" ixz="-2.02138625848788E-21" iyz="-2.42344897559804E-22" joint_origin="0.11226 0.09 -0.068" />
-  <!-- Castor Wheels -->
-  <xacro:macro name="castwheel" params="prefix inertial_origin ixy ixz iyz">
-    <link name="${prefix}_cast_wheel">
-      <inertial>
-        <origin xyz="${inertial_origin}" rpy="0 0 0" />
-        <mass value="0.069429" />
-        <inertia ixx="1.9537E-05" ixy="${ixy}" ixz="${ixz}"
-                 iyy="1.9515E-05" iyz="${iyz}" izz="3.1777E-05" />
-      </inertial>
-      <visual>
-        <origin xyz="0 0 0" rpy="0 0 0" />
-        <geometry>
-          <mesh filename="${mesh_path}${prefix}_cast_wheel.STL" />
-        </geometry>
-        <material name="">
-          <color rgba="${lidar_rgba}" />
-        </material>
-      </visual>
-      <collision>
-        <origin xyz="0 0 0" rpy="0 0 0" />
-        <geometry>
-          <mesh filename="${mesh_path}${prefix}_cast_wheel.STL" />
-        </geometry>
-      </collision>
-    </link>
-    <joint name="${prefix}castwheel" type="continuous">
-      <origin xyz="0 0 0.044416" rpy="1.5708 0 0" />
-      <parent link="${prefix}_castwheel_bracket" />
-      <child link="${prefix}_cast_wheel" />
-      <axis xyz="0 0 1" />
-    </joint>
-  </xacro:macro>
-  <xacro:castwheel prefix="right" inertial_origin="6.93889390390723E-17 4.16333634234434E-17 1.11022302462516E-16" ixy="2.0056E-21" ixz="1.5647E-227" iyz="2.0594E-22" />
-  <xacro:castwheel prefix="left" inertial_origin="5.5511E-17 1.9082E-17 -6.9389E-17" ixy="-4.5297E-22" ixz="1.137E-217" iyz="-3.028E-21" />
-  <!-- LIDAR -->
-  <link name="LIDAR">
-    <inertial>
-      <origin xyz="-1.3878E-17 3.3818E-34 -0.0125" rpy="0 0 0" />
-      <mass value="0.096211" />
-      <inertia ixx="3.4476E-05" ixy="-1.3255E-52" ixz="6.0099E-37"
-               iyy="3.4476E-05" iyz="8.1342E-38" izz="5.8929E-05" />
-    </inertial>
-    <visual>
-      <origin xyz="0 0 0" rpy="0 0 0" />
-      <geometry>
-        <mesh filename="${mesh_path}LIDAR.STL" />
-      </geometry>
-      <material name="">
-        <color rgba="${lidar_rgba}" />
-      </material>
-    </visual>
-    <collision>
-      <origin xyz="0 0 0" rpy="0 0 0" />
-      <geometry>
-        <mesh filename="${mesh_path}LIDAR.STL" />
-      </geometry>
-    </collision>
-  </link>
-  <joint name="lidar" type="fixed">
-    <origin xyz="0.15026 0 0.002" rpy="3.1416 0 0" />
-    <parent link="base_link" />
-    <child link="LIDAR" />
-    <axis xyz="0 0 0" />
-  </joint>
-  <!-- RealSense Camera -->
-  <link name="intel_realsense">
-    <inertial>
-      <origin xyz="-0.00027987 -3.7238E-07 -4.8169E-05" rpy="0 0 0" />
-      <mass value="0.048201" />
-      <inertia ixx="2.7391E-05" ixy="-4.2599E-07" ixz="7.5493E-09"
-               iyy="3.3506E-06" iyz="2.1161E-09" izz="2.6652E-05" />
-    </inertial>
-    <visual>
-      <origin xyz="0 0 0" rpy="0 0 0" />
-      <geometry>
-        <mesh filename="${mesh_path}intel_realsense.STL" />
-      </geometry>
-      <material name="">
-        <color rgba="${intel_rgba}" />
-      </material>
-    </visual>
-    <collision>
-      <origin xyz="0 0 0" rpy="0 0 0" />
-      <geometry>
-        <mesh filename="${mesh_path}intel_realsense.STL" />
-      </geometry>
-    </collision>
-  </link>
-  <joint name="intelrealsense" type="fixed">
-    <origin xyz="0.07723 0 0.44126" rpy="0 0 0" />
-    <parent link="base_link" />
-    <child link="intel_realsense" />
-    <axis xyz="0 0 0" />
-  </joint>
-  <!-- Xarm -->
-  <link name="Xarm">
-  </link>
-  <joint name="xarm" type="fixed">
-    <origin xyz="0.0049756 0 0.34" rpy="0 0 1.57" />
-    <parent link="base_link" />
-    <child link="Xarm" />
-    <axis xyz="0 0 0" />
-  </joint>
-  <xacro:arg name="prefix" default="" />
-  <xacro:arg name="add_gripper" default="false" />
-  <xacro:arg name="add_vacuum_gripper" default="false" />
-  <xacro:arg name="robot_type" default="xarm" />
-  <xacro:arg name="model1300" default="false" />
-  <xacro:arg name="add_realsense_d435i" default="false" />
-  <xacro:arg name="add_d435i_links" default="false" />
-  <xacro:arg name="robot_sn" default="" />
-  <xacro:arg name="dof" default="6" />
-  <xacro:include filename="$(find xarm_description)/urdf/xarm_device_macro.xacro" />
-  <xacro:xarm_device prefix="$(arg prefix)" dof="$(arg dof)" attach_to="Xarm" model1300="$(arg model1300)" add_gripper="$(arg add_gripper)" add_vacuum_gripper="$(arg add_vacuum_gripper)" add_realsense_d435i="$(arg add_realsense_d435i)" add_d435i_links="$(arg add_d435i_links)" robot_sn="$(arg robot_sn)" />
-  <!-- Gripper
-  <xacro:include filename="$(find robot_description)/urdf/gripper/gripper.urdf.xacro" />
-  <xacro:include filename="$(find robot_description)/urdf/gripper/gripperP.urdf.xacro" />
-  <xacro:include filename="$(find robot_description)/urdf/gripper/gripperFakeSF.urdf.xacro" />
-  <xacro:include filename="$(find robot_description)/urdf/gripper/gripperSF.urdf.xacro" />
-  <xacro:load_gripperSF attach_to="$(arg prefix)link_eef" xyz="0 0 0.007" rpy="-1.57 0 2.3554" />
-  <xacro:include filename="$(find robot_description)/urdf/camera.urdf.xacro" />
-  <xacro:load_camera name="Cam1" attach_to="Base_Gripper" x="0.068098" y="-0.035446" z="0.0" r_p="-0.785398" r_r="1.5707" r_y="0.0" />
-  -->
+<xacro:include filename="robot.xacro"/>
 </robot>

Commit message: Added gazebo plugins

File: robot_description/frida_description/urdf/FRIDA.urdf.xacro (robot description, xacro)
@@ -1,4 +1,23 @@
 <?xml version="1.0" encoding="utf-8"?>
 <robot name="FRIDA" xmlns:xacro="http://www.ros.org/wiki/xacro">
+<xacro:arg name="sim_mode" default="false"/>
 <xacro:include filename="robot.xacro"/>
+<gazebo>
+<plugin filename="gz-sim-diff-drive-system" name="gz::sim::systems::DiffDrive">
+  <!-- wheels -->
+  <left_joint>leftwheel</left_joint>
+  <right_joint>rightwheel</right_joint>
+  <!-- kinematics -->
+  <wheel_separation>0.287</wheel_separation>
+  <wheel_radius>0.033</wheel_radius> <!-- computed from <wheel_diameter> in the original plugin-->
+  <!-- limits -->
+  <max_linear_acceleration>0.033</max_linear_acceleration> <!-- computed from <max_linear_acceleration> in the original plugin-->
+  <topic>cmd_vel</topic> <!-- from <commant_topic> -->
+  <odom_topic>odom</odom_topic> <!-- from <odometry_topic> -->
+  <frame_id>odom</frame_id> <!-- from <odometry_frame> -->
+  <child_frame_id>base_link</child_frame_id> <!-- from <robot_base_frame> -->
+  <odom_publisher_frequency>30</odom_publisher_frequency> <!-- from <update_rate>-->
+  <tf_topic>/tf</tf_topic> <!-- Short topic name for tf output -->
+</plugin>
+</gazebo>
 </robot>

File: robot_description/frida_description/urdf/base.xacro (robot description, xacro)
@@ -24,3 +24,9 @@
     </collision>
   </link>
+   <gazebo reference="base_link">
+    <mu1>200</mu1>
+    <mu2>200</mu2>
+    <kp>1000000</kp>
+    <kd>1</kd>
+  </gazebo>
 </robot>

File: robot_description/frida_description/urdf/robot.xacro (robot description, xacro)
@@ -2,5 +2,5 @@
 <robot xmlns:xacro="http://www.ros.org/wiki/xacro">
 <xacro:property name="mesh_path" value="package://frida_description/urdf/meshes/" />
-<xacro:property name="material_rgba" value="0.792 0.820 0.933 1" />
+<xacro:property name="material_rgba" value="0.745 0.203 0.482 1" />
 <xacro:property name="lidar_rgba" value="0.102 0.102 0.102 1" />
 <xacro:property name="intel_rgba" value="0.776 0.757 0.737 1" />
@@ -12,4 +12,18 @@
 <xacro:include filename="realsense.xacro"/>
 <xacro:include filename="xarm.xacro"/>
+<!-- <link name="base_footprint">
+      <visual>
+        <origin xyz="0 0 0" rpy="0 0 0" />
+        <geometry>
+          <box size="0.05 0.05 0.001" />
+        </geometry>
+        <material name="TransparentGreen" />
+      </visual>
+  </link>
+  <joint name="base_joint" type="fixed">
+    <origin xyz="0 0 0" rpy="0 0 0" />
+    <parent link="base_footprint"/>
+    <child link="base_link" />
+  </joint> -->
   <!-- Gripper
   <xacro:include filename="$(find robot_description)/urdf/gripper/gripper.urdf.xacro" />

Commit message: Frida xacro fixed

File: robot_description/frida_description/urdf/FRIDA.urdf.xacro (robot description, xacro)
@@ -41,6 +41,6 @@
   <xacro:arg name="sim_mode" default="false"/>
   <xacro:include filename="robot.xacro"/>
-<xacro:include filename="$(find xarm_description)/urdf/xarm_device_macro.xacro" />
- <xacro:xarm_device prefix="$(arg prefix)" hw_ns="$(arg hw_ns)" limited="$(arg limited)"
+  <xacro:include filename="$(find xarm_description)/urdf/xarm_device_macro.xacro" />
+    <xacro:xarm_device prefix="$(arg prefix)" hw_ns="$(arg hw_ns)" limited="$(arg limited)"
     effort_control="$(arg effort_control)" velocity_control="$(arg velocity_control)"
     add_gripper="$(arg add_gripper)" add_vacuum_gripper="$(arg add_vacuum_gripper)"
@@ -61,3 +61,8 @@
     model1300="$(arg model1300)" attach_to="$(arg attach_to)" attach_xyz="$(arg attach_xyz)" attach_rpy="$(arg attach_rpy)"
     robot_sn="$(arg robot_sn)" use_gazebo_camera="$(arg use_gazebo_camera)" mesh_suffix="$(arg mesh_suffix)" kinematics_suffix="$(arg kinematics_suffix)" />
+ <!-- Gripper -->
+  <xacro:include filename="gripper.xacro" />
+  <xacro:load_gripper attach_to="link_eef" xyz="0 0 0" rpy="0 -1.5708 0" />
+  <xacro:include filename="zed.xacro" />
+  <xacro:load_zed attach_to="gripper" xyz="0.030461 0 -0.050649" rpy="0 0.81804 0" />
 </robot>

File: robot_description/frida_description/urdf/robot.xacro (robot description, xacro)
@@ -11,29 +11,5 @@
 <xacro:include filename="lidar.xacro"/>
 <xacro:include filename="realsense.xacro"/>
-<!-- <xacro:include filename="xarm.xacro"/> -->
-<xacro:include filename="gripper.xacro"/>
-<xacro:include filename="zed.xacro"/>
-<!-- <link name="base_footprint">
-      <visual>
-        <origin xyz="0 0 0" rpy="0 0 0" />
-        <geometry>
-          <box size="0.05 0.05 0.001" />
-        </geometry>
-        <material name="TransparentGreen" />
-      </visual>
-  </link>
-  <joint name="base_joint" type="fixed">
-    <origin xyz="0 0 0" rpy="0 0 0" />
-    <parent link="base_footprint"/>
-    <child link="base_link" />
-  </joint> -->
-  <!-- Gripper
-  <xacro:include filename="$(find robot_description)/urdf/gripper/gripper.urdf.xacro" />
-  <xacro:include filename="$(find robot_description)/urdf/gripper/gripperP.urdf.xacro" />
-  <xacro:include filename="$(find robot_description)/urdf/gripper/gripperFakeSF.urdf.xacro" />
-  <xacro:include filename="$(find robot_description)/urdf/gripper/gripperSF.urdf.xacro" />
-  <xacro:load_gripperSF attach_to="$(arg prefix)link_eef" xyz="0 0 0.007" rpy="-1.57 0 2.3554" />
-  <xacro:include filename="$(find robot_description)/urdf/camera.urdf.xacro" />
-  <xacro:load_camera name="Cam1" attach_to="Base_Gripper" x="0.068098" y="-0.035446" z="0.0" r_p="-0.785398" r_r="1.5707" r_y="0.0" />
-  -->
+<!-- <xacro:include filename="gripper.xacro"/>
+<xacro:include filename="zed.xacro"/> -->
 </robot>

Commit message: test_urdf

File: robot_description/frida_description/urdf/FRIDA.urdf.xacro (robot description, xacro)
@@ -39,5 +39,5 @@
   <xacro:arg name="mesh_suffix" default="stl"/>
   <xacro:arg name="kinematics_suffix" default=""/>
-  <xacro:arg name="sim_mode" default="false"/>
+  <xacro:arg name="sim_mode" default="true"/>
   <xacro:include filename="robot.xacro"/>
   <xacro:include filename="$(find xarm_description)/urdf/xarm_device_macro.xacro" />
@@ -62,7 +62,7 @@
     robot_sn="$(arg robot_sn)" use_gazebo_camera="$(arg use_gazebo_camera)" mesh_suffix="$(arg mesh_suffix)" kinematics_suffix="$(arg kinematics_suffix)" />
  <!-- Gripper -->
-  <xacro:include filename="gripper.xacro" />
+  <!-- <xacro:include filename="gripper.xacro" />
   <xacro:load_gripper attach_to="link_eef" xyz="0 0 0" rpy="0 -1.5708 0" />
   <xacro:include filename="zed.xacro" />
-  <xacro:load_zed attach_to="gripper" xyz="0.030461 0 -0.050649" rpy="0 0.81804 0" />
+  <xacro:load_zed attach_to="gripper" xyz="0.030461 0 -0.050649" rpy="0 0.81804 0" /> -->
 </robot>

File: robot_description/frida_description/urdf/gripper.xacro (robot description, xacro)
@@ -1,5 +1,5 @@
 <?xml version="1.0" encoding="utf-8"?>
 <robot xmlns:xacro="http://www.ros.org/wiki/xacro">
-<xacro:property name="mesh_path" value="package://frida_description/urdf/meshes/" />
+<xacro:property name="mesh_path" value="file://$(find frida_description)/urdf/meshes/" />
 <xacro:macro name="load_gripper" params="attach_to:='' xyz:='0 0 0' rpy:='0 0 0'">
     <xacro:unless value="${attach_to == ''}">

File: robot_description/frida_description/urdf/robot.xacro (robot description, xacro)
@@ -1,5 +1,5 @@
 <?xml version="1.0" encoding="utf-8"?>
 <robot xmlns:xacro="http://www.ros.org/wiki/xacro">
-<xacro:property name="mesh_path" value="package://frida_description/urdf/meshes/" />
+<xacro:property name="mesh_path" value="file://$(find frida_description)/urdf/meshes/" />
 <xacro:property name="material_rgba" value="0.745 0.203 0.482 1" />
 <xacro:property name="lidar_rgba" value="0.102 0.102 0.102 1" />

Commit message: Added new urdf and simulation moveit

File: robot_description/frida_description/urdf/FRIDA.urdf.xacro (robot description, xacro)
@@ -62,7 +62,7 @@
     robot_sn="$(arg robot_sn)" use_gazebo_camera="$(arg use_gazebo_camera)" mesh_suffix="$(arg mesh_suffix)" kinematics_suffix="$(arg kinematics_suffix)" />
  <!-- Gripper -->
-  <!-- <xacro:include filename="gripper.xacro" />
+  <xacro:include filename="gripper.xacro" />
   <xacro:load_gripper attach_to="link_eef" xyz="0 0 0" rpy="0 -1.5708 0" />
   <xacro:include filename="zed.xacro" />
-  <xacro:load_zed attach_to="gripper" xyz="0.030461 0 -0.050649" rpy="0 0.81804 0" /> -->
+  <xacro:load_zed attach_to="gripper" xyz="0.030461 0 -0.050649" rpy="0 0.81804 0" />
 </robot>

File: robot_description/frida_description/urdf/base.xacro (robot description, xacro)
@@ -24,3 +24,10 @@
     </collision>
   </link>
+ <gazebo reference="base_link">
+    <mu1>200</mu1>
+    <mu2>200</mu2>
+    <kp>1000000</kp>
+    <kd>1</kd>
+    <material>Gazebo/Grey</material>
+  </gazebo>
 </robot>

File: robot_description/frida_description/urdf/castwheel.xacro (robot description, xacro)
@@ -34,3 +34,17 @@
   <xacro:castwheel prefix="right" inertial_origin="6.93889390390723E-17 4.16333634234434E-17 1.11022302462516E-16" ixy="2.0056E-21" ixz="1.5647E-227" iyz="2.0594E-22" />
   <xacro:castwheel prefix="left" inertial_origin="5.5511E-17 1.9082E-17 -6.9389E-17" ixy="-4.5297E-22" ixz="1.137E-217" iyz="-3.028E-21" />
+<gazebo reference="right_cast_wheel">
+    <mu1>0.1</mu1>
+    <mu2>0.1</mu2>
+    <kp>1000000</kp>
+    <kd>1</kd>
+    <material>Gazebo/Black</material>
+  </gazebo>
+  <gazebo reference="left_cast_wheel">
+    <mu1>0.1</mu1>
+    <mu2>0.1</mu2>
+    <kp>1000000</kp>
+    <kd>1</kd>
+    <material>Gazebo/Black</material>
+  </gazebo>
 </robot>

File: robot_description/frida_description/urdf/castwheelbraket.xacro (robot description, xacro)
@@ -34,3 +34,17 @@
   <xacro:castwheel_bracket prefix="right" inertial_origin="-6.9389E-17 -1.3878E-17 0.012445" ixy="-5.23501237066605E-21" ixz="1.02910979879346E-20" iyz="1.03781586309714E-20" joint_origin="0.11226 -0.09 -0.068" />
   <xacro:castwheel_bracket prefix="left" inertial_origin="0 -4.1633E-17 0.012445" ixy="2.58235447481398E-21" ixz="-2.02138625848788E-21" iyz="-2.42344897559804E-22" joint_origin="0.11226 0.09 -0.068" />
+<gazebo reference="right_castwheel_bracket">
+    <mu1>0.1</mu1>
+    <mu2>0.1</mu2>
+    <kp>1000000</kp>
+    <kd>1</kd>
+    <material>Gazebo/White</material>
+  </gazebo>
+  <gazebo reference="left_castwheel_bracket">
+    <mu1>0.1</mu1>
+    <mu2>0.1</mu2>
+    <kp>1000000</kp>
+    <kd>1</kd>
+    <material>Gazebo/White</material>
+  </gazebo>
 </robot>

File: robot_description/frida_description/urdf/gripper.xacro (robot description, xacro)
@@ -80,3 +80,6 @@
   </joint>
   </xacro:macro>
+  <gazebo reference="gripper">
+    <material>Gazebo/DarkGrey</material>
+  </gazebo>
 </robot>

File: robot_description/frida_description/urdf/realsense.xacro (robot description, xacro)
@@ -30,3 +30,10 @@
     <axis xyz="0 0 0" />
   </joint>
+  <gazebo reference="intel_realsense">
+    <mu1>200</mu1>
+    <mu2>200</mu2>
+    <kp>1000000</kp>
+    <kd>1</kd>
+    <material>Gazebo/Turquoise</material>
+  </gazebo>
 </robot>

File: robot_description/frida_description/urdf/robot.xacro (robot description, xacro)
@@ -11,5 +11,3 @@
 <xacro:include filename="lidar.xacro"/>
 <xacro:include filename="realsense.xacro"/>
-<!-- <xacro:include filename="gripper.xacro"/>
-<xacro:include filename="zed.xacro"/> -->
 </robot>

File: robot_description/frida_description/urdf/wheels.xacro (robot description, xacro)
@@ -34,3 +34,17 @@
   <xacro:wheel_link prefix="right" ixy="-9.9049E-20" ixz="5.8265E-21" iyz="-2.2717E-21" joint_origin="-0.075244 -0.166 -0.0775" />
   <xacro:wheel_link prefix="left" ixy="4.5051E-20" ixz="1.2238E-21" iyz="7.2483E-21" joint_origin="-0.075244 0.166 -0.0775" />
+  <gazebo reference="left_wheel">
+    <mu1>200</mu1>
+    <mu2>200</mu2>
+    <kp>1000000</kp>
+    <kd>1</kd>
+    <material>Gazebo/Black</material>
+  </gazebo>
+  <gazebo reference="right_wheel">
+    <mu1>200</mu1>
+    <mu2>200</mu2>
+    <kp>1000000</kp>
+    <kd>1</kd>
+    <material>Gazebo/Black</material>
+  </gazebo>
 </robot>

File: robot_description/frida_description/urdf/zed.xacro (robot description, xacro)
@@ -1,5 +1,5 @@
 <?xml version="1.0" encoding="utf-8"?>
 <robot xmlns:xacro="http://www.ros.org/wiki/xacro">
-<xacro:property name="mesh_path" value="package://frida_description/urdf/meshes/" />
+<xacro:property name="mesh_path" value="file://$(find frida_description)/urdf/meshes/" />
 <xacro:macro name="load_zed" params="attach_to:='' xyz:='0 0 0' rpy:='0 0 0'">
     <xacro:unless value="${attach_to == ''}">
