Commit message: Frida_sim v1

File: robot_description/frida_description/urdf/FRIDA.urdf.xacro (robot description, xacro)
@@ -39,5 +39,4 @@
   <xacro:arg name="mesh_suffix" default="stl"/>
   <xacro:arg name="kinematics_suffix" default=""/>
-  <xacro:arg name="sim_mode" default="true"/>
   <xacro:include filename="robot.xacro"/>
   <xacro:include filename="$(find xarm_description)/urdf/xarm_device_macro.xacro" />
@@ -61,8 +60,3 @@
     model1300="$(arg model1300)" attach_to="$(arg attach_to)" attach_xyz="$(arg attach_xyz)" attach_rpy="$(arg attach_rpy)"
     robot_sn="$(arg robot_sn)" use_gazebo_camera="$(arg use_gazebo_camera)" mesh_suffix="$(arg mesh_suffix)" kinematics_suffix="$(arg kinematics_suffix)" />
- <!-- Gripper -->
-  <xacro:include filename="gripper.xacro" />
-  <xacro:load_gripper attach_to="link_eef" xyz="0 0 0" rpy="0 -1.5708 0" />
-  <xacro:include filename="zed.xacro" />
-  <xacro:load_zed attach_to="gripper" xyz="0.030461 0 -0.050649" rpy="0 0.81804 0" />
 </robot>

File: robot_description/frida_description/urdf/base.xacro (robot description, xacro)
@@ -31,10 +31,3 @@
   <link name="base_footprint">
   </link>
- <gazebo reference="base_link">
-    <mu1>200</mu1>
-    <mu2>200</mu2>
-    <kp>1000000</kp>
-    <kd>1</kd>
-    <material>Gazebo/Grey</material>
-  </gazebo>
 </robot>

File: robot_description/frida_description/urdf/castwheel.xacro (robot description, xacro)
@@ -1,50 +1,56 @@
 <?xml version="1.0" encoding="utf-8"?>
 <robot xmlns:xacro="http://www.ros.org/wiki/xacro">
- <xacro:macro name="castwheel" params="prefix inertial_origin ixy ixz iyz">
-    <link name="${prefix}_cast_wheel">
-      <inertial>
-        <origin xyz="${inertial_origin}" rpy="0 0 0" />
-        <mass value="0.069429" />
-        <inertia ixx="1.9537E-05" ixy="${ixy}" ixz="${ixz}"
-                 iyy="1.9515E-05" iyz="${iyz}" izz="3.1777E-05" />
-      </inertial>
-      <visual>
-        <origin xyz="0 0 0" rpy="0 0 0" />
-        <geometry>
-          <mesh filename="${mesh_path}${prefix}_cast_wheel.STL" />
-        </geometry>
-        <material name="">
-          <color rgba="${lidar_rgba}" />
-        </material>
-      </visual>
-      <collision>
-        <origin xyz="0 0 0" rpy="0 0 0" />
-        <geometry>
-          <mesh filename="${mesh_path}${prefix}_cast_wheel.STL" />
-        </geometry>
-      </collision>
+<material name="black">
+        <color rgba="0 0 0 1"/>
+    </material>
+<joint name="caster_wheel_joint_left" type="fixed">
+        <parent link="base_link"/>
+        <child link="caster_wheel_left"/>
+        <origin xyz="0.11 0.1 -0.09"/>
+    </joint>
+    <link name="caster_wheel_left">
+        <visual>
+            <geometry>
+                <sphere radius="0.05"/>
+            </geometry>
+            <material name="black"/>
+        </visual>
+        <collision>
+            <geometry>
+                <sphere radius="0.05"/>
+            </geometry>
+        </collision>
+        <inertial>
+            <origin xyz="0 0 0" rpy="0 0 0"/>
+            <mass value="0.1" />
+            <inertia ixx="${(2/5) * 0.1 * (0.05*0.05)}" ixy="0.0" ixz="0.0"
+                    iyy="${(2/5) * 0.1 * (0.05*0.05)}" iyz="0.0"
+                    izz="${(2/5) * 0.1 * (0.05*0.05)}" />
+        </inertial>
     </link>
-    <joint name="${prefix}castwheel" type="continuous">
-      <origin xyz="0 0 0.044416" rpy="1.5708 0 0" />
-      <parent link="${prefix}_castwheel_bracket" />
-      <child link="${prefix}_cast_wheel" />
-      <axis xyz="0 0 1" />
+  <joint name="caster_wheel_joint_right" type="fixed">
+        <parent link="base_link"/>
+        <child link="caster_wheel_right"/>
+        <origin xyz="0.11 -0.1 -0.09"/>
     </joint>
-  </xacro:macro>
-  <xacro:castwheel prefix="right" inertial_origin="6.93889390390723E-17 4.16333634234434E-17 1.11022302462516E-16" ixy="2.0056E-21" ixz="1.5647E-227" iyz="2.0594E-22" />
-  <xacro:castwheel prefix="left" inertial_origin="5.5511E-17 1.9082E-17 -6.9389E-17" ixy="-4.5297E-22" ixz="1.137E-217" iyz="-3.028E-21" />
-<gazebo reference="right_cast_wheel">
-    <mu1>0.1</mu1>
-    <mu2>0.1</mu2>
-    <kp>1000000</kp>
-    <kd>1</kd>
-    <material>Gazebo/Black</material>
-  </gazebo>
-  <gazebo reference="left_cast_wheel">
-    <mu1>0.1</mu1>
-    <mu2>0.1</mu2>
-    <kp>1000000</kp>
-    <kd>1</kd>
-    <material>Gazebo/Black</material>
-  </gazebo>
+    <link name="caster_wheel_right">
+        <visual>
+            <geometry>
+                <sphere radius="0.05"/>
+            </geometry>
+            <material name="black"/>
+        </visual>
+        <collision>
+            <geometry>
+                <sphere radius="0.05"/>
+            </geometry>
+        </collision>
+        <inertial>
+            <origin xyz="0 0 0" rpy="0 0 0"/>
+            <mass value="0.1" />
+            <inertia ixx="${(2/5) * 0.1 * (0.05*0.05)}" ixy="0.0" ixz="0.0"
+                    iyy="${(2/5) * 0.1 * (0.05*0.05)}" iyz="0.0"
+                    izz="${(2/5) * 0.1 * (0.05*0.05)}" />
+        </inertial>
+    </link>
 </robot>

File: robot_description/frida_description/urdf/gripper.xacro (robot description, xacro)
@@ -80,6 +80,3 @@
   </joint>
   </xacro:macro>
-  <gazebo reference="gripper">
-    <material>Gazebo/DarkGrey</material>
-  </gazebo>
 </robot>

File: robot_description/frida_description/urdf/realsense.xacro (robot description, xacro)
@@ -30,10 +30,3 @@
     <axis xyz="0 0 0" />
   </joint>
-  <gazebo reference="intel_realsense">
-    <mu1>200</mu1>
-    <mu2>200</mu2>
-    <kp>1000000</kp>
-    <kd>1</kd>
-    <material>Gazebo/Turquoise</material>
-  </gazebo>
 </robot>

File: robot_description/frida_description/urdf/robot.xacro (robot description, xacro)
@@ -7,7 +7,8 @@
 <xacro:include filename="base.xacro"/>
 <xacro:include filename="wheels.xacro"/>
-<xacro:include filename="castwheelbraket.xacro"/>
 <xacro:include filename="castwheel.xacro"/>
 <xacro:include filename="lidar.xacro"/>
 <xacro:include filename="realsense.xacro"/>
+<xacro:include filename="imu.xacro"/>
+<xacro:include filename="gazebo.xacro"/>
 </robot>

File: robot_description/frida_description/urdf/wheels.xacro (robot description, xacro)
@@ -34,17 +34,3 @@
   <xacro:wheel_link prefix="right" ixy="-9.9049E-20" ixz="5.8265E-21" iyz="-2.2717E-21" joint_origin="-0.075244 -0.166 -0.0775" />
   <xacro:wheel_link prefix="left" ixy="4.5051E-20" ixz="1.2238E-21" iyz="7.2483E-21" joint_origin="-0.075244 0.166 -0.0775" />
-  <gazebo reference="left_wheel">
-    <mu1>200</mu1>
-    <mu2>200</mu2>
-    <kp>1000000</kp>
-    <kd>1</kd>
-    <material>Gazebo/Black</material>
-  </gazebo>
-  <gazebo reference="right_wheel">
-    <mu1>200</mu1>
-    <mu2>200</mu2>
-    <kp>1000000</kp>
-    <kd>1</kd>
-    <material>Gazebo/Black</material>
-  </gazebo>
 </robot>

Commit message: Added zed and Roborregos gripper simulation using realsense plugin

File: robot_description/frida_description/urdf/FRIDA.urdf.xacro (robot description, xacro)
@@ -39,4 +39,7 @@
   <xacro:arg name="mesh_suffix" default="stl"/>
   <xacro:arg name="kinematics_suffix" default=""/>
+  <!-- ZED ARGUMENTS -->
+  <xacro:arg name="load_zed" default="false"/>
+  <xacro:arg name="simulation" default="false"/>
   <xacro:include filename="robot.xacro"/>
   <xacro:include filename="$(find frida_description)/urdf/xarm/xarm_device_macro.xacro" />
@@ -60,3 +63,12 @@
     model1300="$(arg model1300)" attach_to="$(arg attach_to)" attach_xyz="$(arg attach_xyz)" attach_rpy="$(arg attach_rpy)"
     robot_sn="$(arg robot_sn)" use_gazebo_camera="$(arg use_gazebo_camera)" mesh_suffix="$(arg mesh_suffix)" kinematics_suffix="$(arg kinematics_suffix)" />
+    <xacro:if value="$(arg load_zed)">
+      <xacro:include filename="gripper.xacro" />
+      <xacro:load_gripper attach_to="link_eef" xyz="0 0 0" rpy="2.3562 -1.5708 0" />
+      <!-- ZED MACRO -->
+      <xacro:include filename="$(find frida_description)/urdf/zed_macro.urdf.xacro" />
+      <xacro:zed_camera name="zed" model="zed2" custom_baseline="0" enable_gnss="false" simulation="true" attach_to="gripper" xyz="0.030461 0 -0.050649" rpy="0 0.81804 0">
+          <origin xyz="0 0 0" rpy="0 0 0"/>
+      </xacro:zed_camera>
+    </xacro:if>
 </robot>

File: robot_description/frida_description/urdf/xarm/xarm6/xarm6.ros2_control.xacro (robot description, xacro)
@@ -105,5 +105,5 @@
         </command_interface>
         <state_interface name="position">
-         <param name="initial_value">1.571411</param>
+         <param name="initial_value">1.0472</param>
         </state_interface>
         <state_interface name="velocity"/>
@@ -120,5 +120,5 @@
         </command_interface>
         <state_interface name="position">
-         <param name="initial_value">-3.14</param>
+         <param name="initial_value">0.785</param>
         </state_interface>
         <state_interface name="velocity"/>

Commit message: Working object detector node and deprojection with ZED camera simulation

File: robot_description/frida_description/urdf/FRIDA.urdf.xacro (robot description, xacro)
@@ -65,5 +65,5 @@
     <xacro:if value="$(arg load_zed)">
       <xacro:include filename="gripper.xacro" />
-      <xacro:load_gripper attach_to="link_eef" xyz="0 0 0" rpy="2.3562 -1.5708 0" />
+      <xacro:load_gripper attach_to="link_eef" xyz="0 0 0" rpy="2.3562 -1.5708 0" fixed_joints="true"/>
       <!-- ZED MACRO -->
       <xacro:include filename="$(find frida_description)/urdf/zed_macro.urdf.xacro" />

File: robot_description/frida_description/urdf/gripper.xacro (robot description, xacro)
@@ -2,5 +2,5 @@
 <robot xmlns:xacro="http://www.ros.org/wiki/xacro">
 <xacro:property name="mesh_path" value="file://$(find frida_description)/urdf/meshes/" />
-<xacro:macro name="load_gripper" params="attach_to:='' xyz:='0 0 0' rpy:='0 0 0'">
+<xacro:macro name="load_gripper" params="attach_to:='' xyz:='0 0 0' rpy:='0 0 0' fixed_joints:='false'">
     <xacro:unless value="${attach_to == ''}">
       <joint name="gripper_fix" type="fixed">
@@ -61,5 +61,11 @@
 <xacro:finger prefix="right" inertial_origin="0.031796 -0.039646 -4.3517E-05" ixx="7.5207E-06" ixy="5.702E-06" ixz="2.7442E-21" iyy="1.0341E-05" iyz="-9.9772E-22" izz="1.4333E-05" />
 <xacro:finger prefix="left" inertial_origin="0.031901 0.039833 -2.5479E-17" ixx="7.4373E-06" ixy="-5.6549E-06" ixz="9.4292E-21" iyy="1.0294E-05" iyz="6.0945E-21" izz="1.4202E-05"/>
-  <joint name="rightfinger" type="revolute">
+  <xacro:if value="${fixed_joints}">
+    <xacro:property name="finger_joint_type" value="fixed" />
+  </xacro:if>
+  <xacro:unless value="${fixed_joints}">
+    <xacro:property name="finger_joint_type" value="revolute" />
+  </xacro:unless>
+  <joint name="rightfinger" type="${finger_joint_type}">
     <origin xyz="0.087 -0.01054 0.0008" rpy="0 0 0" />
     <parent link="gripper" />
@@ -70,5 +76,5 @@
   </joint>
   <joint
-    name="leftfinger" type="revolute">
+    name="leftfinger" type="${finger_joint_type}">
     <origin xyz="0.087 0.01346 0.0008" rpy="0 0 0" />
     <parent link="gripper" />

File: robot_description/frida_description/urdf/zed_gazebo.xacro (robot description, xacro)
@@ -4,5 +4,5 @@
     <!-- Depth camera sensor -->
     <gazebo reference="${prefix}_left_camera_frame">
-      <sensor name="zed_left_camera_frame_camera" type="depth">
+      <sensor name="zed" type="depth">
         <update_rate>20</update_rate>
         <camera>
@@ -18,27 +18,14 @@
           </clip>
         </camera>
-        <plugin name="zed__left_camera_frame_controller" filename="libgazebo_ros_openni_kinect.so">
-          <baseline>0.2</baseline>
-          <alwaysOn>true</alwaysOn>
-          <updateRate>1.0</updateRate>
-          <cameraName>zed_depth</cameraName>
-          <imageTopicName>/zed/zed_node/rgb/image_rect_color</imageTopicName>
-          <cameraInfoTopicName>/zed/zed_node/rgb/camera_info</cameraInfoTopicName>
-          <depthImageTopicName>/zed/zed_node/depth/depth_registered</depthImageTopicName>
-          <depthImageInfoTopicName>/zed/zed_node/depth/camera_info</depthImageInfoTopicName>
-          <pointCloudTopicName>/depth/color/points</pointCloudTopicName>
-          <frameName>zed_left_camera_optical_frame</frameName>
-          <pointCloudCutoff>0.5</pointCloudCutoff>
-          <pointCloudCutoffMax>3.0</pointCloudCutoffMax>
-          <distortionK1>0.00000001</distortionK1>
-          <distortionK2>0.00000001</distortionK2>
-          <distortionK3>0.00000001</distortionK3>
-          <distortionT1>0.00000001</distortionT1>
-          <distortionT2>0.00000001</distortionT2>
-          <CxPrime>0</CxPrime>
-          <Cx>0</Cx>
-          <Cy>0</Cy>
-          <focalLength>0</focalLength>
-          <hackBaseline>0</hackBaseline>
+        <plugin name="zed_left_camera_frame_controller" filename="libgazebo_ros_camera.so">
+          <visualize>true</visualize>
+              <imageTopicName>/zed/zed_node/rgb/image_rect_color</imageTopicName>
+              <cameraInfoTopicName>/zed/zed_node/rgb/camera_info</cameraInfoTopicName>
+              <depthImageTopicName>/zed/zed_node/depth/depth_registered</depthImageTopicName>
+              <depthImageCameraInfoTopicName>/zed/zed_node/depth/camera_info</depthImageCameraInfoTopicName>
+              <pointCloudTopicName>depth/color/points</pointCloudTopicName>
+              <frame_name>zed_left_camera_optical_frame</frame_name>
+              <min_depth>0.1</min_depth>
+              <max_depth>5.0</max_depth>
         </plugin>
       </sensor>

Commit message: Zed and gripper working on simulation (#243)
* Fix constants + added filter to consider picked object when

* fix ruff

* Added zed and Roborregos gripper simulation using realsense plugin

* fixes to detector node constants and added template for depth camera with kinect plugin

* Working object detector node and deprojection with ZED camera simulation

File: robot_description/frida_description/urdf/FRIDA.urdf.xacro (robot description, xacro)
@@ -39,4 +39,7 @@
   <xacro:arg name="mesh_suffix" default="stl"/>
   <xacro:arg name="kinematics_suffix" default=""/>
+  <!-- ZED ARGUMENTS -->
+  <xacro:arg name="load_zed" default="false"/>
+  <xacro:arg name="simulation" default="false"/>
   <xacro:include filename="robot.xacro"/>
   <xacro:include filename="$(find frida_description)/urdf/xarm/xarm_device_macro.xacro" />
@@ -60,3 +63,12 @@
     model1300="$(arg model1300)" attach_to="$(arg attach_to)" attach_xyz="$(arg attach_xyz)" attach_rpy="$(arg attach_rpy)"
     robot_sn="$(arg robot_sn)" use_gazebo_camera="$(arg use_gazebo_camera)" mesh_suffix="$(arg mesh_suffix)" kinematics_suffix="$(arg kinematics_suffix)" />
+    <xacro:if value="$(arg load_zed)">
+      <xacro:include filename="gripper.xacro" />
+      <xacro:load_gripper attach_to="link_eef" xyz="0 0 0" rpy="2.3562 -1.5708 0" fixed_joints="true"/>
+      <!-- ZED MACRO -->
+      <xacro:include filename="$(find frida_description)/urdf/zed_macro.urdf.xacro" />
+      <xacro:zed_camera name="zed" model="zed2" custom_baseline="0" enable_gnss="false" simulation="true" attach_to="gripper" xyz="0.030461 0 -0.050649" rpy="0 0.81804 0">
+          <origin xyz="0 0 0" rpy="0 0 0"/>
+      </xacro:zed_camera>
+    </xacro:if>
 </robot>
