Commit message: created nav_basics

File: robot_description/frida_description/urdf/base.xacro (robot description, xacro)
@@ -24,4 +24,11 @@
     </collision>
   </link>
+  <joint name = "base_footprint_joint" type="fixed">
+    <parent link="base_link"/>
+    <child link="base_footprint"/>
+    <origin xyz="0 0 0" rpy="0 0 0 "/>
+  </joint>
+  <link name="base_footprint">
+  </link>
  <gazebo reference="base_link">
     <mu1>200</mu1>

Commit message: Increased friction parameters and overall mass of the robot

File: robot_description/frida_description/urdf/base.xacro (robot description, xacro)
@@ -4,5 +4,5 @@
     <inertial>
       <origin xyz="-0.017897 -0.0059216 0.12557" rpy="0 0 0" />
-      <mass value="31.075" />
+      <mass value="131.075" />
       <inertia ixx="0.67537" ixy="-0.00030935" ixz="-0.0025852"
                iyy="0.61552" iyz="-0.0003748" izz="0.65918" />

File: robot_description/frida_description/urdf/gazebo.xacro (robot description, xacro)
@@ -58,11 +58,11 @@
     </gazebo>
 <gazebo reference="caster_wheel_right">
-      <mu1 value="0.001"/>
-      <mu2 value="0.001"/>
+      <mu1 value="0.1"/>
+      <mu2 value="0.1"/>
     <material>Gazebo/Black</material>
   </gazebo>
   <gazebo reference="caster_wheel_left">
-      <mu1 value="0.001"/>
-      <mu2 value="0.001"/>
+      <mu1 value="0.1"/>
+      <mu2 value="0.1"/>
     <material>Gazebo/Black</material>
   </gazebo>

Commit message: manip changed urdf

File: robot_description/frida_description/urdf/base.xacro (robot description, xacro)
@@ -32,5 +32,5 @@
   <link name="xarm_base" />
   <joint name="xarm_base_joint" type="fixed">
-    <origin xyz="0.0049756 0 0.34" rpy="0 0 1.57" />
+    <origin xyz="0.0049756 0 0.44" rpy="0 0 1.57" />
     <parent link="base_link" />
     <child link="xarm_base" />
