Commit message: Finished new robot and gripper URDF

File: robot_description/frida_description/urdf/newFrida/NewFrida.urdf.xacro (robot description, xacro)
@@ -44,5 +44,5 @@
   <xacro:arg name="default_gripper_baud" default="2000000"/>
   <xacro:arg name="attach_to" default="base_link"/>
-  <xacro:arg name="attach_xyz" default="0.0049756 0 0.34"/>
+  <xacro:arg name="attach_xyz" default="0.036255 0 0.44028"/>
   <xacro:arg name="attach_rpy" default="0 0 1.57"/>
   <xacro:arg name="mesh_suffix" default="stl"/>
@@ -71,60 +71,7 @@
   <!-- Gripper -->
   <xacro:include filename="gripper.xacro" />
-    <xacro:load_gripper attach_to="link_eef" xyz="0 0 0" rpy="2.3562 -1.5708 0" />
+    <xacro:load_gripper attach_to="link_eef" xyz="0 0 0" rpy="0 0 1.5708" />
    <!-- ZED MACRO -->
     <xacro:include filename="zed.xacro" />
-  <xacro:load_zed attach_to="gripper" xyz="0.030461 0 -0.050649" rpy="0 0.81804 0" />
-  <link
-    name="xArm">
-    <inertial>
-      <origin
-        xyz="9.0513E-05 0.0014973 0.073511"
-        rpy="0 0 0" />
-      <mass
-        value="1.7836" />
-      <inertia
-        ixx="0.0049951"
-        ixy="-1.1431E-05"
-        ixz="7.4909E-06"
-        iyy="0.004841"
-        iyz="0.0001237"
-        izz="0.0022894" />
-    </inertial>
-    <visual>
-      <origin
-        xyz="0 0 0"
-        rpy="0 0 0" />
-      <geometry>
-        <mesh
-          filename="package://NewFridaURDF/meshes/xArm.STL" />
-      </geometry>
-      <material
-        name="">
-        <color
-          rgba="0.86667 0.86667 0.8902 1" />
-      </material>
-    </visual>
-    <collision>
-      <origin
-        xyz="0 0 0"
-        rpy="0 0 0" />
-      <geometry>
-        <mesh
-          filename="package://NewFridaURDF/meshes/xArm.STL" />
-      </geometry>
-    </collision>
-  </link>
-  <joint
-    name="xarm"
-    type="fixed">
-    <origin
-      xyz="0.036255 0 0.44028"
-      rpy="0 0 0" />
-    <parent
-      link="base_link" />
-    <child
-      link="xArm" />
-    <axis
-      xyz="0 0 0" />
-  </joint>
+  <xacro:load_zed attach_to="base_gripper" xyz="-0.0045 -0.063576 0.033519" rpy="0 -0.7854 -1.5708" />
 </robot>

File: robot_description/frida_description/urdf/newFrida/castwheel.xacro (robot description, xacro)
@@ -67,13 +67,8 @@
   </link>
   <joint name="rightcastwheel" type="continuous">
-    <origin
-      xyz="0 0 0"
-      rpy="1.5708 0 0" />
-    <parent
-      link="right_castwheel_bracket" />
-    <child
-      link="right_cast_wheel" />
-    <axis
-      xyz="0 0 1" />
+    <origin xyz="0 0 0" rpy="1.5708 0 0" />
+    <parent link="right_castwheel_bracket" />
+    <child link="right_cast_wheel" />
+    <axis xyz="0 0 1" />
   </joint>
   <!--LEFT-->
@@ -99,5 +94,5 @@
       <geometry>
         <mesh
-          filename="package://NewFridaURDF/meshes/left_castwheel_bracket.STL" />
+          filename="${mesh_path}left_castwheel_bracket.STL" />
       </geometry>
       <material
@@ -113,18 +108,14 @@
       <geometry>
         <mesh
-          filename="package://NewFridaURDF/meshes/left_castwheel_bracket.STL" />
+          filename="${mesh_path}left_castwheel_bracket.STL" />
       </geometry>
     </collision>
   </link>
   <joint name="leftcastwheelbracket" type="continuous">
-    <origin
-      xyz="0.11226 0.09 -0.11242"
-      rpy="3.1416 0 0" />
+    <origin xyz="0.11226 0.09 -0.11242" rpy="3.1416 0 0" />
     <parent
       link="base_link" />
-    <child
-      link="left_castwheel_bracket" />
-    <axis
-      xyz="0 0 -1" />
+    <child link="left_castwheel_bracket" />
+    <axis xyz="0 0 -1" />
   </joint>
   <link name="left_cast_wheel">
@@ -148,6 +139,5 @@
         rpy="0 0 0" />
       <geometry>
-        <mesh
-          filename="package://NewFridaURDF/meshes/left_cast_wheel.STL" />
+        <mesh filename="${mesh_path}left_cast_wheel.STL" />
       </geometry>
       <material
@@ -163,18 +153,13 @@
       <geometry>
         <mesh
-          filename="package://NewFridaURDF/meshes/left_cast_wheel.STL" />
+          filename="${mesh_path}left_cast_wheel.STL" />
       </geometry>
     </collision>
   </link>
   <joint name="leftcastwheel" type="continuous">
-    <origin
-      xyz="0 0 0"
-      rpy="1.5708 0 0" />
-    <parent
-      link="left_castwheel_bracket" />
-    <child
-      link="left_cast_wheel" />
-    <axis
-      xyz="0 0 1" />
+    <origin xyz="0 0 0" rpy="1.5708 0 0" />
+    <parent link="left_castwheel_bracket" />
+    <child link="left_cast_wheel" />
+    <axis xyz="0 0 1" />
   </joint>
 </robot>
