Commit message: 2.0 version

File: robot_description/frida_description/urdf/Gripper/Commercial/gripper.xacro (robot description, xacro)
@@ -48,5 +48,5 @@
       </geometry>
       <material name="">
-        <color rgba="${lidar_rgba}" />
+        <color rgba="0.79216 0.81961 0.93333 1" />
       </material>
     </visual>

File: robot_description/frida_description/urdf/TMR2025/FRIDA_Real.urdf.xacro (robot description, xacro)
@@ -64,10 +64,18 @@
     model1300="$(arg model1300)" attach_to="$(arg attach_to)" attach_xyz="$(arg attach_xyz)" attach_rpy="$(arg attach_rpy)"
     robot_sn="$(arg robot_sn)" use_gazebo_camera="$(arg use_gazebo_camera)" mesh_suffix="$(arg mesh_suffix)" kinematics_suffix="$(arg kinematics_suffix)" />
+  <!-- OLD GRIPPER    -->
   <!-- Gripper -->
-  <xacro:include filename="$(find frida_description)/urdf/Gripper/Custom/gripper.xacro" />
-  <xacro:load_gripper attach_to="link_eef" xyz="0 0 0.046" rpy="0 0 1.57" />
+  <xacro:include filename="$(find frida_description)/urdf/Gripper/Commercial/gripper.xacro" />
+    <xacro:load_gripper attach_to="link_eef" xyz="0 0 0" rpy="2.3562 -1.5708 0" />
    <!-- ZED MACRO -->
-  <xacro:include filename="$(find frida_description)/urdf/RoboCup2024/zed.xacro" />
-  <xacro:load_zed attach_to="zed" xyz="0 0 0" rpy="0 0 0" />
+    <xacro:include filename="$(find frida_description)/urdf/RoboCup2024/zed.xacro" />
+  <xacro:load_zed attach_to="gripper" xyz="0.030461 0 -0.050649" rpy="0 0.81804 0" />
+  <!-- NEW GRIPPER MACRO   -->
+  <!-- Gripper -->
+  <!-- <xacro:include filename="$(find frida_description)/urdf/Gripper/Custom/gripper.xacro" />
+  <xacro:load_gripper attach_to="link_eef" xyz="0 0 0.046" rpy="0 0 1.57" /> -->
+   <!-- ZED MACRO -->
+  <!-- <xacro:include filename="$(find frida_description)/urdf/RoboCup2024/zed.xacro" />
+  <xacro:load_zed attach_to="zed" xyz="0 0 0" rpy="0 0 0" /> -->
   <!-- <joint name="base_footprint_joint" type="fixed">
       <origin xyz="0 0 ${base_length/2 + caster_radius*2}" rpy="0 0 0" />

File: robot_description/frida_description/urdf/TMR2025/base.xacro (robot description, xacro)
@@ -32,5 +32,5 @@
   <link name="xarm_base" />
   <joint name="xarm_base_joint" type="fixed">
-    <origin xyz="0.036105613000001 0 0.441000000000001" rpy="0 0 1.57" />
+    <origin xyz="0.036105613000001 0 0.401000000000001" rpy="0 0 1.57" />
     <parent link="base_link" />
     <child link="xarm_base" />

File: robot_description/frida_description/urdf/TMR2025/lidar.xacro (robot description, xacro)
@@ -25,5 +25,5 @@
   </link>
   <joint name="lidar" type="fixed">
-    <origin xyz="0.15026 0 0.002" rpy="3.1416 0 0" />
+    <origin xyz="0.15026 0 0.002" rpy="3.1416 3.1416 1.57" />
     <parent link="base_link" />
     <child link="laser" />
