Commit message: URDF patched to get zed position

File: robot_description/frida_description/srdf/_xarm6_macro.srdf.sim.xacro (robot description, xacro)
@@ -55,4 +55,11 @@
       <joint name="${prefix}joint6" value="0" />
     </group_state>
+    <disable_collisions link1="zed_camera_link" link2="link_eef" reason="Never"/>
+    <disable_collisions link1="zed_camera_link" link2="gripper" reason="Never"/>
+    <disable_collisions link1="zed_camera_link" link2="left_finger" reason="Never"/>
+    <disable_collisions link1="zed_camera_link" link2="link3" reason="Never"/>
+    <disable_collisions link1="zed_camera_link" link2="link5" reason="Never"/>
+    <disable_collisions link1="zed_camera_link" link2="link6" reason="Never"/>
+    <disable_collisions link1="zed_camera_link" link2="right_finger" reason="Never"/>
     <!-- gripper -->
     <xacro:if value="${add_gripper}">
@@ -138,10 +145,4 @@
       <disable_collisions link1="LIDAR" link2="link4" reason="Never"/>
       <disable_collisions link1="LIDAR" link2="link_base" reason="Never"/>
-      <disable_collisions link1="ZED" link2="gripper" reason="Adjacent"/>
-      <disable_collisions link1="ZED" link2="left_finger" reason="Never"/>
-      <disable_collisions link1="ZED" link2="link3" reason="Never"/>
-      <disable_collisions link1="ZED" link2="link5" reason="Never"/>
-      <disable_collisions link1="ZED" link2="link6" reason="Never"/>
-      <disable_collisions link1="ZED" link2="right_finger" reason="Never"/>
       <disable_collisions link1="base_link" link2="intel_realsense" reason="Adjacent"/>
       <disable_collisions link1="base_link" link2="left_finger" reason="Default"/>

File: robot_description/frida_description/srdf/_xarm6_macro.srdf.xacro (robot description, xacro)
@@ -55,4 +55,11 @@
       <joint name="${prefix}joint6" value="0" />
     </group_state>
+    <disable_collisions link1="zed_camera_link" link2="link_eef" reason="Never"/>
+    <disable_collisions link1="zed_camera_link" link2="gripper" reason="Never"/>
+    <disable_collisions link1="zed_camera_link" link2="left_finger" reason="Never"/>
+    <disable_collisions link1="zed_camera_link" link2="link3" reason="Never"/>
+    <disable_collisions link1="zed_camera_link" link2="link5" reason="Never"/>
+    <disable_collisions link1="zed_camera_link" link2="link6" reason="Never"/>
+    <disable_collisions link1="zed_camera_link" link2="right_finger" reason="Never"/>
     <!-- gripper -->
     <xacro:if value="${add_gripper}">
@@ -138,10 +145,4 @@
       <disable_collisions link1="LIDAR" link2="link4" reason="Never"/>
       <disable_collisions link1="LIDAR" link2="link_base" reason="Never"/>
-      <disable_collisions link1="ZED" link2="gripper" reason="Adjacent"/>
-      <disable_collisions link1="ZED" link2="left_finger" reason="Never"/>
-      <disable_collisions link1="ZED" link2="link3" reason="Never"/>
-      <disable_collisions link1="ZED" link2="link5" reason="Never"/>
-      <disable_collisions link1="ZED" link2="link6" reason="Never"/>
-      <disable_collisions link1="ZED" link2="right_finger" reason="Never"/>
       <disable_collisions link1="base_link" link2="intel_realsense" reason="Adjacent"/>
       <disable_collisions link1="base_link" link2="left_finger" reason="Default"/>

File: robot_description/frida_description/srdf/xarm_macro.srdf.xacro (robot description, xacro)
@@ -4,5 +4,5 @@
     add_gripper:='false' add_vacuum_gripper:='false' add_bio_gripper:='false' add_other_geometry:='false' ">
     <xacro:if value="${dof == 5}">
-      <xacro:include filename="$(find xarm_moveit_config)/srdf/_xarm5_macro.srdf.xacro" />
+      <xacro:include filename="$(find frida_description)/srdf/_xarm5_macro.srdf.xacro" />
       <xacro:xarm5_macro_srdf prefix="${prefix}"
         add_gripper="${add_gripper}" add_vacuum_gripper="${add_vacuum_gripper}" add_bio_gripper="${add_bio_gripper}" add_other_geometry="${add_other_geometry}" />
@@ -10,10 +10,10 @@
     <xacro:if value="${dof == 6}">
       <xacro:if value="${robot_type == 'uf850'}">
-        <xacro:include filename="$(find xarm_moveit_config)/srdf/_uf850_macro.srdf.xacro" />
+        <xacro:include filename="$(find frida_description)/srdf/_uf850_macro.srdf.xacro" />
         <xacro:uf850_macro_srdf prefix="${prefix}"
           add_gripper="${add_gripper}" add_vacuum_gripper="${add_vacuum_gripper}" add_bio_gripper="${add_bio_gripper}" add_other_geometry="${add_other_geometry}"  />
       </xacro:if>
       <xacro:if value="${robot_type == 'lite'}">
-        <xacro:include filename="$(find xarm_moveit_config)/srdf/_lite6_macro.srdf.xacro" />
+        <xacro:include filename="$(find frida_description)/srdf/_lite6_macro.srdf.xacro" />
         <xacro:lite6_macro_srdf prefix="${prefix}"
           add_gripper="${add_gripper}" add_vacuum_gripper="${add_vacuum_gripper}" add_other_geometry="${add_other_geometry}"  />
@@ -27,10 +27,10 @@
     <xacro:unless value="${dof == 5 or dof == 6}">
       <xacro:if value="${robot_type == 'xarm7_mirror'}">
-        <xacro:include filename="$(find xarm_moveit_config)/srdf/_xarm7_mirror_macro.srdf.xacro" />
+        <xacro:include filename="$(find frida_description)/srdf/_xarm7_mirror_macro.srdf.xacro" />
         <xacro:xarm7_mirror_macro_srdf prefix="${prefix}"
           add_gripper="${add_gripper}" add_vacuum_gripper="${add_vacuum_gripper}" add_bio_gripper="${add_bio_gripper}" add_other_geometry="${add_other_geometry}"  />
       </xacro:if>
       <xacro:unless value="${robot_type == 'xarm7_mirror'}">
-        <xacro:include filename="$(find xarm_moveit_config)/srdf/_xarm7_macro.srdf.xacro" />
+        <xacro:include filename="$(find frida_description)/srdf/_xarm7_macro.srdf.xacro" />
         <xacro:xarm7_macro_srdf prefix="${prefix}"
           add_gripper="${add_gripper}" add_vacuum_gripper="${add_vacuum_gripper}" add_bio_gripper="${add_bio_gripper}" add_other_geometry="${add_other_geometry}"  />

File: robot_description/frida_description/urdf/TMR2025/FRIDA_Real.urdf.xacro (robot description, xacro)
@@ -70,5 +70,5 @@
    <!-- ZED MACRO -->
     <xacro:include filename="$(find frida_description)/urdf/RoboCup2024/zed.xacro" />
-  <xacro:load_zed attach_to="gripper" xyz="0.030461 0 -0.050649" rpy="0 0.81804 0" />
+  <xacro:load_zed attach_to="gripper" xyz="0.046461 0 -0.075649" rpy="0 0.81804 0" />
   <!-- NEW GRIPPER MACRO   -->
   <!-- Gripper -->

File: robot_description/frida_description/urdf/TMR2025/base.xacro (robot description, xacro)
@@ -32,5 +32,5 @@
   <link name="xarm_base" />
   <joint name="xarm_base_joint" type="fixed">
-    <origin xyz="0.036105613000001 0 0.401000000000001" rpy="0 0 1.57" />
+    <origin xyz="0.036105613000001 0 0.441000000000001" rpy="0 0 1.57" />
     <parent link="base_link" />
     <child link="xarm_base" />
