Commit message: I want to move it, but I dont have MoveIt
Status:
       - Launch now adds the rviz config, as well as all the move it Config by the moveit sim builder. However it still dont answer the pick_and_place.launch a.k.a the manipulation core

File: robot_description/frida_description/srdf/xarm.srdf.xacro (robot description, xacro)
@@ -1,4 +1,4 @@
 <?xml version="1.0" encoding="UTF-8"?>
-<robot xmlns:xacro="http://wiki.ros.org/xacro" name="UF_ROBOT">
+<robot xmlns:xacro="http://wiki.ros.org/xacro" name="FRIDA">
   <!-- parameters -->
   <xacro:arg name="prefix" default="" />

File: robot_description/frida_description/urdf/TMR2025/FRIDA_Real.urdf.xacro (robot description, xacro)
@@ -49,12 +49,11 @@
       <compiler angle="radian" balanceinertia="true" autolimits="true"/>
     </mujoco>
-    <!-- Important in order to add additional files in the spawn -->
-    <link name="world" />
-    <joint name="world_to_base" type="fixed">
-      <parent link="world" />
-      <child link="base_link" />
-      <origin rpy="0 0 0" xyz="0 0 0.3" />
-    </joint>
   </xacro:if>
+  <link name="world" />
+  <joint name="world_to_base" type="fixed">
+    <parent link="world" />
+    <child link="base_link" />
+    <origin rpy="0 0 0" xyz="0 0 0.3" />
+  </joint>
   <!-- XARM MACRO -->
   <xacro:include filename="$(find frida_description)/urdf/xarm/xarm_device_macro.xacro" />
