Commit message: added poses to rviz

File: robot_description/frida_description/srdf/_xarm6_macro.srdf.xacro (robot description, xacro)
@@ -39,19 +39,59 @@
     </group>
     <!-- GROUP STATES, Purpose, Define a named state for a particular group, in terms of joint values. This is useful to define states like 'folded arms' -->
-    <group_state name="home" group="${prefix}xarm6">
-      <joint name="${prefix}joint1" value="0" />
-      <joint name="${prefix}joint2" value="0" />
-      <joint name="${prefix}joint3" value="0" />
-      <joint name="${prefix}joint4" value="0" />
-      <joint name="${prefix}joint5" value="0" />
-      <joint name="${prefix}joint6" value="0" />
-    </group_state>
-    <group_state name="hold-up" group="${prefix}xarm6">
-      <joint name="${prefix}joint1" value="0" />
-      <joint name="${prefix}joint2" value="0" />
-      <joint name="${prefix}joint3" value="0" />
-      <joint name="${prefix}joint4" value="0" />
-      <joint name="${prefix}joint5" value="-1.5708" />
-      <joint name="${prefix}joint6" value="0" />
+    <group_state name="front_stare" group="${prefix}xarm6">
+      <joint name="${prefix}joint1" value="-1.5708" />
+      <joint name="${prefix}joint2" value="-0.7854" />
+      <joint name="${prefix}joint3" value="-1.5708" />
+      <joint name="${prefix}joint4" value="0.0" />
+      <joint name="${prefix}joint5" value="0.0" />
+      <joint name="${prefix}joint6" value="0.7854" />
+    </group_state>
+    <group_state name="front_low_stare" group="${prefix}xarm6">
+      <joint name="${prefix}joint1" value="-1.5708" />
+      <joint name="${prefix}joint2" value="-0.7854" />
+      <joint name="${prefix}joint3" value="-1.5708" />
+      <joint name="${prefix}joint4" value="0.0" />
+      <joint name="${prefix}joint5" value="0.3491" />
+      <joint name="${prefix}joint6" value="0.7854" />
+    </group_state>
+    <group_state name="table_stare" group="${prefix}xarm6">
+      <joint name="${prefix}joint1" value="-1.5708" />
+      <joint name="${prefix}joint2" value="-1.3963" />
+      <joint name="${prefix}joint3" value="-1.2217" />
+      <joint name="${prefix}joint4" value="0.0" />
+      <joint name="${prefix}joint5" value="1.0472" />
+      <joint name="${prefix}joint6" value="0.7854" />
+    </group_state>
+    <group_state name="receive_object" group="${prefix}xarm6">
+      <joint name="${prefix}joint1" value="-1.6047" />
+      <joint name="${prefix}joint2" value="-1.1695" />
+      <joint name="${prefix}joint3" value="-0.5476" />
+      <joint name="${prefix}joint4" value="0.0139" />
+      <joint name="${prefix}joint5" value="0.0473" />
+      <joint name="${prefix}joint6" value="0.7352" />
+    </group_state>
+    <group_state name="pick_stare_at_table" group="${prefix}xarm6">
+      <joint name="${prefix}joint1" value="-1.5708" />
+      <joint name="${prefix}joint2" value="-0.1745" />
+      <joint name="${prefix}joint3" value="-2.9671" />
+      <joint name="${prefix}joint4" value="0.0" />
+      <joint name="${prefix}joint5" value="1.7453" />
+      <joint name="${prefix}joint6" value="0.7854" />
+    </group_state>
+    <group_state name="nav_pose" group="${prefix}xarm6">
+      <joint name="${prefix}joint1" value="-1.5708" />
+      <joint name="${prefix}joint2" value="-1.0472" />
+      <joint name="${prefix}joint3" value="-0.9599" />
+      <joint name="${prefix}joint4" value="0.0" />
+      <joint name="${prefix}joint5" value="0.4363" />
+      <joint name="${prefix}joint6" value="0.7854" />
+    </group_state>
+    <group_state name="carry_pose" group="${prefix}xarm6">
+      <joint name="${prefix}joint1" value="-1.5708" />
+      <joint name="${prefix}joint2" value="-1.2217" />
+      <joint name="${prefix}joint3" value="-0.8203" />
+      <joint name="${prefix}joint4" value="0.0" />
+      <joint name="${prefix}joint5" value="-0.2094" />
+      <joint name="${prefix}joint6" value="-0.7854" />
     </group_state>
     <disable_collisions link1="zed_camera_link" link2="link_eef" reason="Never"/>

Commit message: fix sign

File: robot_description/frida_description/srdf/_xarm6_macro.srdf.xacro (robot description, xacro)
@@ -93,5 +93,5 @@
       <joint name="${prefix}joint4" value="0.0" />
       <joint name="${prefix}joint5" value="-0.2094" />
-      <joint name="${prefix}joint6" value="-0.7854" />
+      <joint name="${prefix}joint6" value="0.7854" />
     </group_state>
     <disable_collisions link1="zed_camera_link" link2="link_eef" reason="Never"/>

Commit message: added poses to rviz (#534)
* added poses to rviz

* fix sign

File: robot_description/frida_description/srdf/_xarm6_macro.srdf.xacro (robot description, xacro)
@@ -39,19 +39,59 @@
     </group>
     <!-- GROUP STATES, Purpose, Define a named state for a particular group, in terms of joint values. This is useful to define states like 'folded arms' -->
-    <group_state name="home" group="${prefix}xarm6">
-      <joint name="${prefix}joint1" value="0" />
-      <joint name="${prefix}joint2" value="0" />
-      <joint name="${prefix}joint3" value="0" />
-      <joint name="${prefix}joint4" value="0" />
-      <joint name="${prefix}joint5" value="0" />
-      <joint name="${prefix}joint6" value="0" />
-    </group_state>
-    <group_state name="hold-up" group="${prefix}xarm6">
-      <joint name="${prefix}joint1" value="0" />
-      <joint name="${prefix}joint2" value="0" />
-      <joint name="${prefix}joint3" value="0" />
-      <joint name="${prefix}joint4" value="0" />
-      <joint name="${prefix}joint5" value="-1.5708" />
-      <joint name="${prefix}joint6" value="0" />
+    <group_state name="front_stare" group="${prefix}xarm6">
+      <joint name="${prefix}joint1" value="-1.5708" />
+      <joint name="${prefix}joint2" value="-0.7854" />
+      <joint name="${prefix}joint3" value="-1.5708" />
+      <joint name="${prefix}joint4" value="0.0" />
+      <joint name="${prefix}joint5" value="0.0" />
+      <joint name="${prefix}joint6" value="0.7854" />
+    </group_state>
+    <group_state name="front_low_stare" group="${prefix}xarm6">
+      <joint name="${prefix}joint1" value="-1.5708" />
+      <joint name="${prefix}joint2" value="-0.7854" />
+      <joint name="${prefix}joint3" value="-1.5708" />
+      <joint name="${prefix}joint4" value="0.0" />
+      <joint name="${prefix}joint5" value="0.3491" />
+      <joint name="${prefix}joint6" value="0.7854" />
+    </group_state>
+    <group_state name="table_stare" group="${prefix}xarm6">
+      <joint name="${prefix}joint1" value="-1.5708" />
+      <joint name="${prefix}joint2" value="-1.3963" />
+      <joint name="${prefix}joint3" value="-1.2217" />
+      <joint name="${prefix}joint4" value="0.0" />
+      <joint name="${prefix}joint5" value="1.0472" />
+      <joint name="${prefix}joint6" value="0.7854" />
+    </group_state>
+    <group_state name="receive_object" group="${prefix}xarm6">
+      <joint name="${prefix}joint1" value="-1.6047" />
+      <joint name="${prefix}joint2" value="-1.1695" />
+      <joint name="${prefix}joint3" value="-0.5476" />
+      <joint name="${prefix}joint4" value="0.0139" />
+      <joint name="${prefix}joint5" value="0.0473" />
+      <joint name="${prefix}joint6" value="0.7352" />
+    </group_state>
+    <group_state name="pick_stare_at_table" group="${prefix}xarm6">
+      <joint name="${prefix}joint1" value="-1.5708" />
+      <joint name="${prefix}joint2" value="-0.1745" />
+      <joint name="${prefix}joint3" value="-2.9671" />
+      <joint name="${prefix}joint4" value="0.0" />
+      <joint name="${prefix}joint5" value="1.7453" />
+      <joint name="${prefix}joint6" value="0.7854" />
+    </group_state>
+    <group_state name="nav_pose" group="${prefix}xarm6">
+      <joint name="${prefix}joint1" value="-1.5708" />
+      <joint name="${prefix}joint2" value="-1.0472" />
+      <joint name="${prefix}joint3" value="-0.9599" />
+      <joint name="${prefix}joint4" value="0.0" />
+      <joint name="${prefix}joint5" value="0.4363" />
+      <joint name="${prefix}joint6" value="0.7854" />
+    </group_state>
+    <group_state name="carry_pose" group="${prefix}xarm6">
+      <joint name="${prefix}joint1" value="-1.5708" />
+      <joint name="${prefix}joint2" value="-1.2217" />
+      <joint name="${prefix}joint3" value="-0.8203" />
+      <joint name="${prefix}joint4" value="0.0" />
+      <joint name="${prefix}joint5" value="-0.2094" />
+      <joint name="${prefix}joint6" value="0.7854" />
     </group_state>
     <disable_collisions link1="zed_camera_link" link2="link_eef" reason="Never"/>

Commit message: onsite tests

File: robot_description/frida_description/srdf/_xarm6_macro.srdf.xacro (robot description, xacro)
@@ -81,8 +81,8 @@
     <group_state name="nav_pose" group="${prefix}xarm6">
       <joint name="${prefix}joint1" value="-1.5708" />
-      <joint name="${prefix}joint2" value="-1.0472" />
-      <joint name="${prefix}joint3" value="-0.9599" />
-      <joint name="${prefix}joint4" value="0.0" />
-      <joint name="${prefix}joint5" value="0.4363" />
+      <joint name="${prefix}joint2" value="-1.22173048" />
+      <joint name="${prefix}joint3" value="-0.78539816" />
+      <joint name="${prefix}joint4" value="0.0" />
+      <joint name="${prefix}joint5" value="0.17453293" />
       <joint name="${prefix}joint6" value="0.7854" />
     </group_state>

File: robot_description/frida_description/urdf/TMR2025/lidar.xacro (robot description, xacro)
@@ -25,5 +25,5 @@
   </link>
   <joint name="lidar" type="fixed">
-    <origin xyz="0.15026 0 0.002" rpy="3.1416 3.1416 1.57" />
+    <origin xyz="0.15026 0 0.002" rpy="0 0 1.57" />
     <parent link="base_link" />
     <child link="laser" />

Commit message: Integrar gripper paralelo en el robot real + SRDF (#944)
FRIDA_Real usa gripper_assem (gripper nuevo): orientacion de la ZED (giro de 180 en load_zed, camara fisicamente derecha) y pedestal world->base_link a 0.145 m por medicion fisica. SRDF (_xarm6_macro) con la matriz de colision del gripper+ZED nuevos para poder planear. La simulacion (FRIDA.urdf.xacro) sigue usando gripper.xacro.

File: robot_description/frida_description/srdf/_xarm6_macro.srdf.xacro (robot description, xacro)
@@ -95,11 +95,36 @@
       <joint name="${prefix}joint6" value="0.7854" />
     </group_state>
+    <!-- ZED + gripper custom (parallel mount, #944): el ensamble
+         (base_gripper, leftFinger, rightFinger, zed, zed_camera_link) va rigido
+         sobre link_eef, por eso se deshabilitan entre si y contra la muneca. -->
+    <!-- ensamble interno -->
+    <disable_collisions link1="base_gripper" link2="zed" reason="Adjacent"/>
+    <disable_collisions link1="base_gripper" link2="zed_camera_link" reason="Never"/>
+    <disable_collisions link1="base_gripper" link2="leftFinger" reason="Adjacent"/>
+    <disable_collisions link1="base_gripper" link2="rightFinger" reason="Adjacent"/>
+    <disable_collisions link1="leftFinger" link2="rightFinger" reason="Never"/>
+    <disable_collisions link1="leftFinger" link2="zed" reason="Never"/>
+    <disable_collisions link1="leftFinger" link2="zed_camera_link" reason="Never"/>
+    <disable_collisions link1="rightFinger" link2="zed" reason="Never"/>
+    <disable_collisions link1="rightFinger" link2="zed_camera_link" reason="Never"/>
+    <disable_collisions link1="zed" link2="zed_camera_link" reason="Adjacent"/>
+    <!-- ensamble vs muneca -->
+    <disable_collisions link1="base_gripper" link2="link_eef" reason="Adjacent"/>
+    <disable_collisions link1="base_gripper" link2="link6" reason="Never"/>
+    <disable_collisions link1="base_gripper" link2="link5" reason="Never"/>
+    <disable_collisions link1="leftFinger" link2="link_eef" reason="Never"/>
+    <disable_collisions link1="leftFinger" link2="link6" reason="Never"/>
+    <disable_collisions link1="rightFinger" link2="link_eef" reason="Never"/>
+    <disable_collisions link1="rightFinger" link2="link6" reason="Never"/>
+    <disable_collisions link1="zed" link2="link_eef" reason="Never"/>
+    <disable_collisions link1="zed" link2="link6" reason="Never"/>
+    <disable_collisions link1="zed" link2="link5" reason="Never"/>
+    <disable_collisions link1="zed" link2="link4" reason="Never"/>
+    <disable_collisions link1="zed" link2="link3" reason="Never"/>
     <disable_collisions link1="zed_camera_link" link2="link_eef" reason="Never"/>
-    <disable_collisions link1="zed_camera_link" link2="gripper" reason="Never"/>
-    <disable_collisions link1="zed_camera_link" link2="left_finger" reason="Never"/>
+    <disable_collisions link1="zed_camera_link" link2="link6" reason="Never"/>
+    <disable_collisions link1="zed_camera_link" link2="link5" reason="Never"/>
+    <disable_collisions link1="zed_camera_link" link2="link4" reason="Never"/>
     <disable_collisions link1="zed_camera_link" link2="link3" reason="Never"/>
-    <disable_collisions link1="zed_camera_link" link2="link5" reason="Never"/>
-    <disable_collisions link1="zed_camera_link" link2="link6" reason="Never"/>
-    <disable_collisions link1="zed_camera_link" link2="right_finger" reason="Never"/>
     <!-- gripper -->
     <xacro:if value="${add_gripper}">
@@ -186,18 +211,18 @@
       <disable_collisions link1="LIDAR" link2="link_base" reason="Never"/>
       <disable_collisions link1="base_link" link2="intel_realsense" reason="Adjacent"/>
-      <disable_collisions link1="base_link" link2="left_finger" reason="Default"/>
+      <disable_collisions link1="base_link" link2="leftFinger" reason="Default"/>
       <disable_collisions link1="base_link" link2="link1" reason="Never"/>
       <disable_collisions link1="base_link" link2="link_base" reason="Adjacent"/>
-      <disable_collisions link1="base_link" link2="right_finger" reason="Default"/>
-      <disable_collisions link1="gripper" link2="left_finger" reason="Adjacent"/>
-      <disable_collisions link1="gripper" link2="link5" reason="Never"/>
-      <disable_collisions link1="gripper" link2="link6" reason="Never"/>
-      <disable_collisions link1="gripper" link2="right_finger" reason="Adjacent"/>
+      <disable_collisions link1="base_link" link2="rightFinger" reason="Default"/>
+      <disable_collisions link1="base_gripper" link2="leftFinger" reason="Adjacent"/>
+      <disable_collisions link1="base_gripper" link2="link5" reason="Never"/>
+      <disable_collisions link1="base_gripper" link2="link6" reason="Never"/>
+      <disable_collisions link1="base_gripper" link2="rightFinger" reason="Adjacent"/>
       <disable_collisions link1="intel_realsense" link2="link1" reason="Never"/>
       <disable_collisions link1="intel_realsense" link2="link2" reason="Never"/>
       <disable_collisions link1="intel_realsense" link2="link_base" reason="Never"/>
-      <disable_collisions link1="left_finger" link2="link5" reason="Never"/>
-      <disable_collisions link1="left_finger" link2="link6" reason="Never"/>
-      <disable_collisions link1="left_finger" link2="right_finger" reason="Never"/>
+      <disable_collisions link1="leftFinger" link2="link5" reason="Never"/>
+      <disable_collisions link1="leftFinger" link2="link6" reason="Never"/>
+      <disable_collisions link1="leftFinger" link2="rightFinger" reason="Never"/>
       <disable_collisions link1="link1" link2="link2" reason="Adjacent"/>
       <disable_collisions link1="link1" link2="link3" reason="Never"/>
@@ -211,6 +236,6 @@
       <disable_collisions link1="link4" link2="link6" reason="Never"/>
       <disable_collisions link1="link5" link2="link6" reason="Adjacent"/>
-      <disable_collisions link1="link5" link2="right_finger" reason="Never"/>
-      <disable_collisions link1="link6" link2="right_finger" reason="Never"/>
+      <disable_collisions link1="link5" link2="rightFinger" reason="Never"/>
+      <disable_collisions link1="link6" link2="rightFinger" reason="Never"/>
     </xacro:if>
     <!-- bio gripper -->
@@ -288,12 +313,12 @@
     <disable_collisions link1="base_link" link2="intel_realsense" reason="Adjacent"/>
     <disable_collisions link1="base_link" link2="laser" reason="Adjacent"/>
-    <disable_collisions link1="base_link" link2="left_finger" reason="Default"/>
+    <disable_collisions link1="base_link" link2="leftFinger" reason="Default"/>
     <disable_collisions link1="base_link" link2="link1" reason="Never"/>
     <disable_collisions link1="base_link" link2="link_base" reason="Adjacent"/>
-    <disable_collisions link1="gripper" link2="left_finger" reason="Adjacent"/>
-    <disable_collisions link1="gripper" link2="link5" reason="Never"/>
-    <disable_collisions link1="gripper" link2="link6" reason="Adjacent"/>
-    <disable_collisions link1="gripper" link2="right_finger" reason="Adjacent"/>
-    <disable_collisions link1="gripper" link2="zed_camera_center" reason="Adjacent"/>
+    <disable_collisions link1="base_gripper" link2="leftFinger" reason="Adjacent"/>
+    <disable_collisions link1="base_gripper" link2="link5" reason="Never"/>
+    <disable_collisions link1="base_gripper" link2="link6" reason="Adjacent"/>
+    <disable_collisions link1="base_gripper" link2="rightFinger" reason="Adjacent"/>
+    <disable_collisions link1="base_gripper" link2="zed_camera_center" reason="Adjacent"/>
     <disable_collisions link1="intel_realsense" link2="laser" reason="Never"/>
     <disable_collisions link1="intel_realsense" link2="link1" reason="Never"/>
@@ -305,8 +330,8 @@
     <disable_collisions link1="laser" link2="link4" reason="Never"/>
     <disable_collisions link1="laser" link2="link_base" reason="Never"/>
-    <disable_collisions link1="left_finger" link2="link5" reason="Never"/>
-    <disable_collisions link1="left_finger" link2="link6" reason="Never"/>
-    <disable_collisions link1="left_finger" link2="right_finger" reason="Default"/>
-    <disable_collisions link1="left_finger" link2="zed_camera_center" reason="Never"/>
+    <disable_collisions link1="leftFinger" link2="link5" reason="Never"/>
+    <disable_collisions link1="leftFinger" link2="link6" reason="Never"/>
+    <disable_collisions link1="leftFinger" link2="rightFinger" reason="Default"/>
+    <disable_collisions link1="leftFinger" link2="zed_camera_center" reason="Never"/>
     <disable_collisions link1="link1" link2="link2" reason="Adjacent"/>
     <disable_collisions link1="link1" link2="link3" reason="Never"/>
@@ -321,9 +346,9 @@
     <disable_collisions link1="link4" link2="link6" reason="Never"/>
     <disable_collisions link1="link5" link2="link6" reason="Adjacent"/>
-    <disable_collisions link1="link5" link2="right_finger" reason="Never"/>
+    <disable_collisions link1="link5" link2="rightFinger" reason="Never"/>
     <disable_collisions link1="link5" link2="zed_camera_center" reason="Never"/>
-    <disable_collisions link1="link6" link2="right_finger" reason="Never"/>
+    <disable_collisions link1="link6" link2="rightFinger" reason="Never"/>
     <disable_collisions link1="link6" link2="zed_camera_center" reason="Never"/>
-    <disable_collisions link1="right_finger" link2="zed_camera_center" reason="Never"/>
+    <disable_collisions link1="rightFinger" link2="zed_camera_center" reason="Never"/>
   </xacro:macro>
 </robot>

File: robot_description/frida_description/urdf/TMR2025/FRIDA_Real.urdf.xacro (robot description, xacro)
@@ -100,5 +100,5 @@
       <parent link="world" />
       <child link="base_link" />
-      <origin rpy="0 0 0" xyz="0 0 0.3" />
+      <origin rpy="0 0 0" xyz="0 0 0.145" />
     </joint>
   </xacro:unless>
@@ -140,9 +140,9 @@
   <!-- NEW GRIPPER MACRO   -->
   <!-- Gripper -->
-  <xacro:include filename="$(find frida_description)/urdf/Gripper/Custom/gripper.xacro" />
+  <xacro:include filename="$(find frida_description)/urdf/Gripper/Custom/gripper_assem.xacro" />
   <xacro:load_gripper attach_to="link_eef" xyz="0 0 0.046" rpy="0 0 3.926" fixed_joints="false" mujoco_plugin="$(arg mujoco_plugin)"/>
    <!-- ZED MACRO -->
   <xacro:include filename="$(find frida_description)/urdf/zed/zed.xacro" />
-  <xacro:load_zed attach_to="zed" xyz="0.0 0 0.0" rpy="0 0 0"  mujoco_plugin="$(arg mujoco_plugin)" />
+  <xacro:load_zed attach_to="zed" xyz="0.0 0 0.0" rpy="3.14159265358979 0 0"  mujoco_plugin="$(arg mujoco_plugin)" />
   <!-- <joint name="base_footprint_joint" type="fixed">
       <origin xyz="0 0 ${base_length/2 + caster_radius*2}" rpy="0 0 0" />
