Commit message: URDF sim stable

File: robot_description/frida_description/urdf/RoboCup2024/base.xacro (robot description, xacro)
@@ -4,5 +4,5 @@
     <inertial>
       <origin xyz="-0.017897 -0.0059216 0.12557" rpy="0 0 0" />
-      <mass value="131.075" />
+      <mass value="1000.075" />
       <inertia ixx="0.67537" ixy="-0.00030935" ixz="-0.0025852"
                iyy="0.61552" iyz="-0.0003748" izz="0.65918" />

File: robot_description/frida_description/urdf/RoboCup2024/wheels.xacro (robot description, xacro)
@@ -5,5 +5,5 @@
       <inertial>
         <origin xyz="-1.3878E-17 0 2.7756E-17" rpy="0 0 0" />
-        <mass value="100.52892" />
+        <mass value="0.52892" />
         <inertia ixx="0.00063131" ixy="${ixy}" ixz="${ixz}"
                  iyy="0.00063131" iyz="${iyz}" izz="0.0011216" />

File: robot_description/frida_description/urdf/TMR2025/base.xacro (robot description, xacro)
@@ -4,5 +4,5 @@
     <inertial>
       <origin xyz="0.031681 -0.0052694 0.10165" rpy="0 0 0" />
-      <mass value="131.075" />
+      <mass value="500.075" />
       <inertia ixx="0.44959" ixy="-0.005113" ixz="0.017804"
                iyy="0.46194" iyz="-0.00061969" izz="0.78515" />

File: robot_description/frida_description/urdf/TMR2025/castwheel.xacro (robot description, xacro)
@@ -1,82 +1,56 @@
 <?xml version="1.0" encoding="utf-8"?>
 <robot xmlns:xacro="http://www.ros.org/wiki/xacro">
-    <xacro:macro name="caster_wheel_bracket" params="prefix xyz ixy ixz iyz joint_origin">
-      <link name="${prefix}_castwheel_bracket">
-        <inertial>
-        <origin
-            xyz="${xyz}"
-            rpy="0 0 0" />
-        <mass
-            value="0.451852451728102" />
-        <inertia
-            ixx="1.91437440179204E-05" ixy="${ixy}" ixz="${ixz}"
-            iyy="2.03620552975365E-05" iyz="${iyz}" izz="1.58126328123224E-05" />
-        </inertial>
+<material name="black">
+        <color rgba="0 0 0 1"/>
+    </material>
+<joint name="caster_wheel_joint_left" type="fixed">
+        <parent link="base_link"/>
+        <child link="caster_wheel_left"/>
+        <origin xyz="0.11 0.1 -0.09"/>
+    </joint>
+    <link name="caster_wheel_left">
         <visual>
-        <origin xyz="0 0 0" rpy="0 0 0" />
-        <geometry>
-            <mesh filename="${mesh_path}${prefix}_castwheel_bracket.STL" />
-        </geometry>
-        <material name="">
-            <color rgba="${black_rgba}" />
-        </material>
+            <geometry>
+                <sphere radius="0.05"/>
+            </geometry>
+            <material name="black"/>
         </visual>
         <collision>
-        <origin xyz="0 0 0" rpy="0 0 0" />
-        <geometry>
-            <mesh filename="${mesh_path}${prefix}_castwheel_bracket.STL" />
-        </geometry>
+            <geometry>
+                <sphere radius="0.05"/>
+            </geometry>
         </collision>
+        <inertial>
+            <origin xyz="0 0 0" rpy="0 0 0"/>
+            <mass value="0.1" />
+            <inertia ixx="${(2/5) * 0.1 * (0.05*0.05)}" ixy="0.0" ixz="0.0"
+                    iyy="${(2/5) * 0.1 * (0.05*0.05)}" iyz="0.0"
+                    izz="${(2/5) * 0.1 * (0.05*0.05)}" />
+        </inertial>
     </link>
-    <joint name="${prefix}castwheelbracket" type="continuous">
-        <origin xyz="${joint_origin}" rpy="3.1416 0 0" />
-        <parent link="base_link" />
-        <child link="${prefix}_castwheel_bracket" />
-        <axis xyz="0 0 -1" />
+  <joint name="caster_wheel_joint_right" type="fixed">
+        <parent link="base_link"/>
+        <child link="caster_wheel_right"/>
+        <origin xyz="0.11 -0.1 -0.09"/>
     </joint>
-    </xacro:macro>
-    <xacro:caster_wheel_bracket prefix="right" xyz="2.77555756156289E-17 -2.08166817117217E-16 -0.0319709734767012" ixy="5.65290697905272E-21" ixz="-6.79719081628809E-21" iyz="-1.18762790839083E-20" joint_origin="0.112255613 -0.09 -0.112416320504547"/>
-    <xacro:caster_wheel_bracket prefix="left" xyz="-1.11022302462516E-16 4.16333634234434E-17 -0.0319709734767013" ixy="9.03249326780732E-22" ixz="-4.43903476297829E-22" iyz="-9.72493121445985E-21" joint_origin="0.112255613 0.09 -0.112416320504547"/>
-    <xacro:macro name="caster_wheel" params="prefix xyz ixy ixz iyz">
-      <link
-        name="${prefix}_cast_wheel">
-        <inertial>
-        <origin
-            xyz="xyz"
-            rpy="0 0 0" />
-        <mass
-            value="0.694291976443345" />
-        <inertia ixx="1.95153903045283E-05" ixy="${ixy}" ixz="${ixz}"
-                 iyy="1.95153903045283E-05" iyz="${iyz}" izz="3.17985725211052E-05" />
-        </inertial>
+    <link name="caster_wheel_right">
         <visual>
-        <origin
-            xyz="0 0 0"
-            rpy="0 0 0" />
-        <geometry>
-            <mesh
-            filename="${mesh_path}${prefix}_cast_wheel.STL" />
-        </geometry>
-        <material name="">
-            <color rgba="${black_rgba}" />
-        </material>
+            <geometry>
+                <sphere radius="0.05"/>
+            </geometry>
+            <material name="black"/>
         </visual>
         <collision>
-        <origin
-            xyz="0 0 0"
-            rpy="0 0 0" />
-        <geometry>
-            <mesh filename="${mesh_path}${prefix}_cast_wheel.STL" />
-        </geometry>
+            <geometry>
+                <sphere radius="0.05"/>
+            </geometry>
         </collision>
-      </link>
-      <joint name="${prefix}castwheel" type="continuous">
-        <origin xyz="0 0 0" rpy="1.5707963267949 0 0" />
-        <parent link="${prefix}_castwheel_bracket" />
-        <child link="${prefix}_cast_wheel" />
-        <axis xyz="0 0 1" />
-      </joint>
-    </xacro:macro>
-    <xacro:caster_wheel prefix="right" xyz="4.16333634234434E-17 -1.34441069388203E-17 1.38777878078145E-17" ixy="-7.05128389877886E-22" ixz="-3.30872245021211E-22" iyz="-3.41901319855252E-22"/>
-    <xacro:caster_wheel prefix="left" xyz="0 8.67361737988404E-19 2.77555756156289E-17" ixy="-7.4724136116802E-22" ixz="-3.29900618130813E-21" iyz="-3.03150518992427E-21"/>
+        <inertial>
+            <origin xyz="0 0 0" rpy="0 0 0"/>
+            <mass value="0.1" />
+            <inertia ixx="${(2/5) * 0.1 * (0.05*0.05)}" ixy="0.0" ixz="0.0"
+                    iyy="${(2/5) * 0.1 * (0.05*0.05)}" iyz="0.0"
+                    izz="${(2/5) * 0.1 * (0.05*0.05)}" />
+        </inertial>
+    </link>
 </robot>

File: robot_description/frida_description/urdf/TMR2025/wheels.xacro (robot description, xacro)
@@ -5,5 +5,5 @@
       <inertial>
         <origin xyz="${xyz}" rpy="0 0 0" />
-        <mass value="0.528918539158378" />
+        <mass value="100.528918539158378" />
         <inertia ixx="0.00063131" ixy="6.14301607073899E-41" ixz="-1.72050413075699E-18"
                  iyy="0.00063131" iyz="1.33885585873066E-36" izz="0.0011216" />
