Commit message: Fixed simulation URDF, needs weight? fixes

File: robot_description/frida_description/urdf/RoboCup2024/FRIDA.urdf.xacro (robot description, xacro)
@@ -67,5 +67,5 @@
       <xacro:load_gripper attach_to="link_eef" xyz="0 0 0" rpy="2.3562 -1.5708 0" fixed_joints="true"/>
       <!-- ZED MACRO -->
-      <xacro:include filename="$(find frida_description)/urdf/RoboCup2024/zed_macro.urdf.xacro" />
+      <xacro:include filename="$(find frida_description)/urdf/zed/zed_macro.urdf.xacro" />
       <xacro:zed_camera name="zed" model="zed2" custom_baseline="0" enable_gnss="false" simulation="true" attach_to="gripper" xyz="0.030461 0 -0.050649" rpy="0 0.81804 0">
           <origin xyz="0 0 0" rpy="0 0 0"/>

File: robot_description/frida_description/urdf/RoboCup2024/FRIDA_Real.urdf.xacro (robot description, xacro)
@@ -68,5 +68,5 @@
     <xacro:load_gripper attach_to="link_eef" xyz="0 0 0" rpy="2.3562 -1.5708 0" />
    <!-- ZED MACRO -->
-    <xacro:include filename="zed.xacro" />
+    <xacro:include filename="$(find frida_description)/urdf/zed/zed.xacro" />
   <xacro:load_zed attach_to="gripper" xyz="0.030461 0 -0.050649" rpy="0 0.81804 0" />
   <!-- <joint name="base_footprint_joint" type="fixed">

File: robot_description/frida_description/urdf/TMR2025/FRIDA.urdf.xacro (robot description, xacro)
@@ -63,10 +63,19 @@
     model1300="$(arg model1300)" attach_to="$(arg attach_to)" attach_xyz="$(arg attach_xyz)" attach_rpy="$(arg attach_rpy)"
     robot_sn="$(arg robot_sn)" use_gazebo_camera="$(arg use_gazebo_camera)" mesh_suffix="$(arg mesh_suffix)" kinematics_suffix="$(arg kinematics_suffix)" />
+    <!-- <xacro:if value="$(arg load_zed)"> -->
+      <!-- <xacro:include filename="$(find frida_description)/urdf/Gripper/Custom/gripper.xacro" /> -->
+      <!-- <xacro:load_gripper attach_to="link_eef" xyz="0 0 0.046" rpy="0 0 1.57" fixed_joints="true"/> -->
+      <!-- ZED MACRO -->
+      <!-- <xacro:include filename="$(find frida_description)/urdf/zed/zed_macro.urdf.xacro" /> -->
+      <!-- <xacro:zed_camera name="zed" model="zed2" custom_baseline="0" enable_gnss="false" simulation="true" attach_to="zed" xyz="0 0 0" rpy="0 0 0"> -->
+          <!-- <origin xyz="0 0 0" rpy="0 0 0"/> -->
+      <!-- </xacro:zed_camera> -->
+    <!-- </xacro:if> -->
     <xacro:if value="$(arg load_zed)">
-      <xacro:include filename="$(find frida_description)/urdf/Gripper/Custom/gripper.xacro" />
-      <xacro:load_gripper attach_to="link_eef" xyz="0 0 0.046" rpy="0 0 1.57" fixed_joints="true"/>
+      <xacro:include filename="$(find frida_description)/urdf/Gripper/Commercial/gripper.xacro" />
+      <xacro:load_gripper attach_to="link_eef" xyz="0 0 0" rpy="2.3562 -1.5708 0" fixed_joints="true"/>
       <!-- ZED MACRO -->
-      <xacro:include filename="$(find frida_description)/urdf/RoboCup2024/zed_macro.urdf.xacro" />
-      <xacro:zed_camera name="zed" model="zed2" custom_baseline="0" enable_gnss="false" simulation="true" attach_to="zed" xyz="0 0 0" rpy="0 0 0">
+      <xacro:include filename="$(find frida_description)/urdf/zed/zed_macro.urdf.xacro" />
+      <xacro:zed_camera name="zed" model="zed2" custom_baseline="0" enable_gnss="false" simulation="true" attach_to="gripper" xyz="0.030461 0 -0.050649" rpy="0 0.81804 0">
           <origin xyz="0 0 0" rpy="0 0 0"/>
       </xacro:zed_camera>

File: robot_description/frida_description/urdf/TMR2025/FRIDA_Real.urdf.xacro (robot description, xacro)
@@ -69,5 +69,5 @@
     <xacro:load_gripper attach_to="link_eef" xyz="0 0 0" rpy="2.3562 -1.5708 0" />
    <!-- ZED MACRO -->
-    <xacro:include filename="$(find frida_description)/urdf/RoboCup2024/zed.xacro" />
+    <xacro:include filename="$(find frida_description)/urdf/zed/zed.xacro" />
   <xacro:load_zed attach_to="gripper" xyz="0.046461 0 -0.075649" rpy="0 0.81804 0" />
   <!-- NEW GRIPPER MACRO   -->

File: robot_description/frida_description/urdf/zed/zed_macro.urdf.xacro (robot description, xacro)
@@ -241,5 +241,5 @@
     </xacro:if>
     <xacro:if value="${simulation}">
-      <xacro:include filename="$(find frida_description)/urdf/zed_gazebo.xacro"/>
+      <xacro:include filename="$(find frida_description)/urdf/zed/zed_gazebo.xacro"/>
       <xacro:zed_gazebo prefix="${name}" />
     </xacro:if>

Commit message: close

File: robot_description/frida_description/urdf/RoboCup2024/FRIDA.urdf.xacro (robot description, xacro)
@@ -68,5 +68,5 @@
       <!-- ZED MACRO -->
       <xacro:include filename="$(find frida_description)/urdf/zed/zed_macro.urdf.xacro" />
-      <xacro:zed_camera name="zed" model="zed2" custom_baseline="0" enable_gnss="false" simulation="true" attach_to="gripper" xyz="0.030461 0 -0.050649" rpy="0 0.81804 0">
+  <xacro:zed_camera name="zed" model="zed2" custom_baseline="0" enable_gnss="false" simulation="true" attach_to="gripper" xyz="0.030461 0 -0.050649" rpy="0 0.81804 0">
           <origin xyz="0 0 0" rpy="0 0 0"/>
       </xacro:zed_camera>

File: robot_description/frida_description/urdf/TMR2025/FRIDA.urdf.xacro (robot description, xacro)
@@ -63,7 +63,13 @@
     model1300="$(arg model1300)" attach_to="$(arg attach_to)" attach_xyz="$(arg attach_xyz)" attach_rpy="$(arg attach_rpy)"
     robot_sn="$(arg robot_sn)" use_gazebo_camera="$(arg use_gazebo_camera)" mesh_suffix="$(arg mesh_suffix)" kinematics_suffix="$(arg kinematics_suffix)" />
+    <joint name="gripper_grasp_joint" type="fixed">
+      <parent link="link_eef"/>
+      <child link="gripper_grasp_frame"/>
+      <origin xyz="0 0 0" rpy="0 0 -0.7854"/>
+    </joint>
+    <link name="gripper_grasp_frame"> </link>
     <xacro:if value="$(arg load_zed)">
       <xacro:include filename="$(find frida_description)/urdf/Gripper/Custom/gripper.xacro" />
-      <xacro:load_gripper attach_to="link_eef" xyz="0 0 0.046" rpy="0 0 3.14" fixed_joints="true"/>
+      <xacro:load_gripper attach_to="link_eef" xyz="0 0 0.046" rpy="0 0 3.926"/>
       <!-- ZED MACRO -->
       <xacro:include filename="$(find frida_description)/urdf/zed/zed_macro.urdf.xacro" />

File: robot_description/frida_description/urdf/zed/zed_gazebo.xacro (robot description, xacro)
@@ -3,5 +3,5 @@
   <xacro:macro name="zed_gazebo" params="prefix:='zed' ">
     <!-- Depth camera sensor -->
-    <gazebo reference="${prefix}_left_camera_frame">
+    <gazebo reference="zed_left_camera_frame">
       <sensor name="zed" type="depth">
         <update_rate>20</update_rate>

Commit message: Revert "Merge branch 'fix-zed-offset' of https://github.com/RoBorregos/home2 into fix-zed-offset"
This reverts commit 6847e1a802d434215e6df3f668b19ed807935466, reversing
changes made to d17f606ed2fa344e73ff07488f55b9e8515981f2.

File: robot_description/frida_description/urdf/RoboCup2024/FRIDA.urdf.xacro (robot description, xacro)
@@ -34,5 +34,5 @@
   <xacro:arg name="baud_checkset" default="true"/>
   <xacro:arg name="default_gripper_baud" default="2000000"/>
-  <xacro:arg name="attach_to" default="_base_link"/>
+  <xacro:arg name="attach_to" default="base_link"/>
   <xacro:arg name="attach_xyz" default="0.0049756 0 0.34"/>
   <xacro:arg name="attach_rpy" default="0 0 1.57"/>
@@ -42,5 +42,5 @@
   <xacro:arg name="load_zed" default="false"/>
   <xacro:arg name="simulation" default="false"/>
-  <xacro:include filename="$(find home_custom_base_description)/urdf/robot.xacro"/>
+  <xacro:include filename="robot.xacro"/>
   <xacro:include filename="$(find frida_description)/urdf/xarm/xarm_device_macro.xacro" />
     <xacro:xarm_device prefix="$(arg prefix)" hw_ns="$(arg hw_ns)" limited="$(arg limited)"

File: robot_description/frida_description/urdf/TMR2025/FRIDA_Real.urdf.xacro (robot description, xacro)
@@ -38,10 +38,10 @@
   <xacro:arg name="attach_to" default="xarm_base"/>
   <xacro:arg name="attach_xyz" default="0 0 0"/>
-  <xacro:arg name="attach_rpy" default="0 0 1.5707963267948966"/>
+  <xacro:arg name="attach_rpy" default="0 0 0"/>
   <xacro:arg name="mesh_suffix" default="stl"/>
   <xacro:arg name="kinematics_suffix" default=""/>
   <!-- ZED ARGUMENTS -->
   <!-- ROBOT COMPONENTS -->
-  <xacro:include filename="$(find frida_description)/urdf/omnibase/robot.xacro"/>
+  <xacro:include filename="robot_real.xacro"/>
   <!-- MUJOCO PARAMS -->
   <!-- gravcomp mirrors the xarm6 firmware's internal gravity compensation:
@@ -92,5 +92,5 @@
     <joint name="world_to_base" type="fixed">
       <parent link="world" />
-      <child link="_base_footprint" />
+      <child link="base_link" />
       <origin rpy="0 0 0" xyz="0 0 0" />
     </joint>
@@ -99,5 +99,5 @@
     <joint name="world_to_base" type="fixed">
       <parent link="world" />
-      <child link="_base_footprint" />
+      <child link="base_link" />
       <origin rpy="0 0 0" xyz="0 0 0.3" />
     </joint>
