Commit message: urdf with all spheres

File: robot_description/frida_description/urdf/TMR2025/frida_real.urdf (robot description, URDF)
Before this commit: robot FRIDA, 15 links, 13 joints
Links:
- link base_link: geometry collision sphere radius=0.02; collision sphere radius=0.02
- link gripper: geometry visual mesh filename=meshes/gripper/gripper.stl
- link left_finger: geometry collision sphere radius=0.01766; collision sphere radius=0.01861
- link link1: geometry collision sphere radius=0.03582; collision sphere radius=0.04113
- link link2: geometry collision sphere radius=0.03; collision sphere radius=0.03
- link link3: geometry collision sphere radius=0.02522; collision sphere radius=0.02641
- link link4: geometry collision sphere radius=0.02011; collision sphere radius=0.02061
- link link5: geometry collision sphere radius=0.03511; collision sphere radius=0.03591
- link link6: geometry collision sphere radius=0.02111; collision sphere radius=0.02111
- link link_base: geometry visual mesh filename=meshes/xarm/link_base.stl
- link right_finger: geometry collision sphere radius=0.01766; collision sphere radius=0.01861
- link zed_camera_link: geometry visual mesh filename=meshes/gripper/zed.stl
