Commit message: nav files

File: robot_description/frida_description/urdf/TMR2025/lidar.xacro (robot description, xacro)
@@ -30,3 +30,26 @@
     <axis xyz="0 0 0" />
   </joint>
+<link name="imu_base">
+    <inertial>
+      <origin xyz="-1.3878E-17 3.3818E-34 -0.0125" rpy="0 0 0" />
+      <mass value="0.096211" />
+      <inertia ixx="3.4476E-05" ixy="-1.3255E-52" ixz="6.0099E-37"
+               iyy="3.4476E-05" iyz="8.1342E-38" izz="5.8929E-05" />
+    </inertial>
+    <visual>
+      <origin xyz="0 0 0" rpy="0 0 0" />
+      <material name="">
+        <color rgba="${black_rgba}" />
+      </material>
+    </visual>
+    <collision>
+      <origin xyz="0 0 0" rpy="0 0 0" />
+    </collision>
+  </link>
+  <joint name="imu_base_joint" type="fixed">
+    <origin xyz="0.15026 0 0.002" rpy="3.1416 3.1416 1.57" />
+    <parent link="base_link" />
+    <child link="imu_base" />
+    <axis xyz="0 0 0" />
+  </joint>
 </robot>

Commit message: Mujoco Interface Start
 - Added mujoco_ros2 controller from DFKI that seems pretty usefull\n - Modified xacros to be able to spawn the robot in the simulation : [lidar]\n - Modified the base_link.stl to have less vertex\n -Added a trial launch file in a new package 'mujoco_spawn' to test the controller from DFKI

File: robot_description/frida_description/urdf/TMR2025/lidar.xacro (robot description, xacro)
@@ -42,7 +42,13 @@
         <color rgba="${black_rgba}" />
       </material>
+      <geometry>
+        <box size="0.01 0.01 0.01"/>
+      </geometry>
     </visual>
     <collision>
       <origin xyz="0 0 0" rpy="0 0 0" />
+      <geometry>
+        <box size="0.001 0.001 0.001"/>
+      </geometry>
     </collision>
   </link>

Commit message: Fix lidar position

File: robot_description/frida_description/urdf/TMR2025/lidar.xacro (robot description, xacro)
@@ -25,5 +25,5 @@
   </link>
   <joint name="lidar" type="fixed">
-    <origin xyz="0.15026 0 0.002" rpy="0 0 1.57" />
+    <origin xyz="0.15026 0 0.002" rpy="0 0 3.14" />
     <parent link="base_link" />
     <child link="laser" />

Commit message: Lidar updated position and noise

File: robot_description/frida_description/urdf/TMR2025/lidar.xacro (robot description, xacro)
@@ -25,5 +25,5 @@
   </link>
   <joint name="lidar" type="fixed">
-    <origin xyz="0.15026 0 0.002" rpy="0 0 3.14" />
+    <origin xyz="0.16 0 0.002" rpy="0 0 3.14" />
     <parent link="base_link" />
     <child link="laser" />
