Commit message: manipulation changes

File: robot_description/frida_description/urdf/TMR2025/base.xacro (robot description, xacro)
@@ -32,5 +32,5 @@
   <link name="xarm_base" />
   <joint name="xarm_base_joint" type="fixed">
-    <origin xyz="0.036105613000001 0 0.401000000000001" rpy="0 0 1.57" />
+    <origin xyz="0.036105613000001 0 0.341000000000001" rpy="0 0 1.57" />
     <parent link="base_link" />
     <child link="xarm_base" />

Commit message: changes_general

File: robot_description/frida_description/urdf/TMR2025/base.xacro (robot description, xacro)
@@ -32,5 +32,5 @@
   <link name="xarm_base" />
   <joint name="xarm_base_joint" type="fixed">
-    <origin xyz="0.036105613000001 0 0.341000000000001" rpy="0 0 1.57" />
+    <origin xyz="0.036105613000001 0 0.301000000000001" rpy="0 0 1.57" />
     <parent link="base_link" />
     <child link="xarm_base" />

Commit message: fixed_things

File: robot_description/frida_description/urdf/TMR2025/base.xacro (robot description, xacro)
@@ -32,5 +32,5 @@
   <link name="xarm_base" />
   <joint name="xarm_base_joint" type="fixed">
-    <origin xyz="0.036105613000001 0 0.301000000000001" rpy="0 0 1.57" />
+    <origin xyz="0.036105613000001 0 0.401000000000001" rpy="0 0 1.57" />
     <parent link="base_link" />
     <child link="xarm_base" />

Commit message: add speaker collision

File: robot_description/frida_description/urdf/TMR2025/base.xacro (robot description, xacro)
@@ -23,4 +23,10 @@
       </geometry>
     </collision>
+        <collision>
+      <origin xyz=".09 -0.12 .49" rpy="0 0 0"/>
+      <geometry>
+        <sphere radius="0.063"/>
+      </geometry>
+    </collision>
   </link>
   <link name="base_footprint" />

Commit message: Pick and place build now builds everything needed to run pipeline

File: robot_description/frida_description/urdf/TMR2025/base.xacro (robot description, xacro)
@@ -4,5 +4,5 @@
     <inertial>
       <origin xyz="0.031681 -0.0052694 0.10165" rpy="0 0 0" />
-      <mass value="500.075" />
+      <mass value="5000.075" />
       <inertia ixx="0.44959" ixy="-0.005113" ixz="0.017804"
                iyy="0.46194" iyz="-0.00061969" izz="0.78515" />

Commit message: sim update

File: robot_description/frida_description/urdf/TMR2025/base.xacro (robot description, xacro)
@@ -4,5 +4,5 @@
     <inertial>
       <origin xyz="0.031681 -0.0052694 0.10165" rpy="0 0 0" />
-      <mass value="5000.075" />
+      <mass value="200.075" />
       <inertia ixx="0.44959" ixy="-0.005113" ixz="0.017804"
                iyy="0.46194" iyz="-0.00061969" izz="0.78515" />

Commit message: robocup 2025

File: robot_description/frida_description/urdf/TMR2025/base.xacro (robot description, xacro)
@@ -23,5 +23,5 @@
       </geometry>
     </collision>
-        <collision>
+    <collision>
       <origin xyz=".09 -0.12 .49" rpy="0 0 0"/>
       <geometry>

Commit message: quit past speaker collision

File: robot_description/frida_description/urdf/TMR2025/base.xacro (robot description, xacro)
@@ -23,10 +23,4 @@
       </geometry>
     </collision>
-    <collision>
-      <origin xyz=".09 -0.12 .49" rpy="0 0 0"/>
-      <geometry>
-        <sphere radius="0.063"/>
-      </geometry>
-    </collision>
   </link>
   <link name="base_footprint" />

Commit message: added simplify mesh for base link

File: robot_description/frida_description/urdf/TMR2025/base.xacro (robot description, xacro)
@@ -20,5 +20,5 @@
       <origin xyz="0 0 0" rpy="0 0 0" />
       <geometry>
-        <mesh filename="${mesh_path}base_link.STL" />
+        <mesh filename="${mesh_path}base_link_simplified.stl" scale="0.1 0.1 0.1"/>
       </geometry>
     </collision>

Commit message: change stl collision for base link due to changes in speaker and screen

File: robot_description/frida_description/urdf/TMR2025/base.xacro (robot description, xacro)
@@ -20,5 +20,5 @@
       <origin xyz="0 0 0" rpy="0 0 0" />
       <geometry>
-        <mesh filename="${mesh_path}base_link.STL" />
+        <mesh filename="${mesh_path}base_link_collision.stl" />
       </geometry>
     </collision>
