Commit message: Wire sim ZED through object_detector_2d and make the test cube easier to detect
- Bump mujoco_ros2_control submodule: color frames now published as
  rgb8 (was the un-convertible '8UC3'), so cv_bridge consumers and the
  detector don't crash on the first frame.
- object_detector_2d/config/parameters.yaml:
  * point YOLO_MODEL_PATH at tmr2025.pt (the actual file shipped);
    tmr_30classes_v2.pt doesn't exist in the package.
  * change the params-file top-level key from 'object_detector_node' to
    '/**' so the values apply when launch renames the node to
    ObjectDetect2D.
  * fix the '//visiondetections_image' double-slash typo that crashed
    node startup with InvalidTopicNameException.
  * lower MIN_SCORE_THRESH from 0.75 to 0.3 -- the simulated objects
    have a larger domain gap so confidence scores are lower.
- table_and_object.xacro: grow the pickable cube from 5 cm to 10 cm so
  there are enough pixels in the ZED frame for the detector to work
  with, and update its inertia + start height accordingly.

File: robot_description/frida_description/urdf/TMR2025/table_and_object.xacro (robot description, xacro)
@@ -46,5 +46,5 @@
       <origin xyz="0 0 0" rpy="0 0 0"/>
       <geometry>
-        <box size="0.05 0.05 0.05"/>
+        <box size="0.10 0.10 0.10"/>
       </geometry>
       <material name="cube_green">
@@ -55,5 +55,5 @@
       <origin xyz="0 0 0" rpy="0 0 0"/>
       <geometry>
-        <box size="0.05 0.05 0.05"/>
+        <box size="0.10 0.10 0.10"/>
       </geometry>
     </collision>
@@ -61,6 +61,6 @@
       <mass value="0.1"/>
       <origin xyz="0 0 0" rpy="0 0 0"/>
-      <!-- Solid cube inertia: (1/12)*m*(a^2 + b^2) = (1/12)*0.1*0.005 = 4.17e-5 -->
-      <inertia ixx="4.17e-5" ixy="0" ixz="0" iyy="4.17e-5" iyz="0" izz="4.17e-5"/>
+      <!-- Solid cube inertia: (1/12)*m*(a^2 + b^2) = (1/12)*0.1*0.02 = 1.67e-4 -->
+      <inertia ixx="1.67e-4" ixy="0" ixz="0" iyy="1.67e-4" iyz="0" izz="1.67e-4"/>
     </inertial>
   </link>
@@ -68,7 +68,6 @@
     <parent link="world"/>
     <child link="cube_link"/>
-    <!-- Start sitting on the table top (0.7 m) + half the cube (0.025 m).
-         Tiny forward bias so the cube isn't exactly at the table center. -->
-    <origin xyz="0.55 0 0.73" rpy="0 0 0"/>
+    <!-- Start sitting on the table top (0.7 m) + half the cube (0.05 m). -->
+    <origin xyz="0.55 0 0.75" rpy="0 0 0"/>
   </joint>
 </robot>

Commit message: Shape the sim cube for the real xarm custom gripper + drop house.xacro
Keep pick_and_place / place / pour with the same parameters they use on
the real robot (no sim-only overrides). Adjust the environment instead:

- table_and_object.xacro: cube goes from 10 cm cube to 4 x 4 x 12 cm.
  Custom gripper opens up to ~5.6 cm, so 4 cm fits cleanly; the 12 cm
  height gives GPD a proper vertical surface to find side grasps on.
- mujoco_sim_init.launch.py:
  * stop loading house.xacro. Its walls saturated the ZED pointcloud
    so perception_3d's plane segmenter kept latching onto a wall at
    base_link z=0.70 instead of our 0.40 m table top, which made the
    real-robot PICK_MIN_HEIGHT=0.1 reject every valid grasp.
  * drop the pick_min_height launch override; the sim now uses the
    same 0.1 m default as the real robot.

Pick pipeline status: detection -> cluster -> GPD -> grasps all work
end to end; the last remaining gap is the plane segmenter picking up
the robot's own meshes (gripper/ZED) because there is no self-filter
on /point_cloud yet.

File: robot_description/frida_description/urdf/TMR2025/table_and_object.xacro (robot description, xacro)
@@ -46,5 +46,5 @@
       <origin xyz="0 0 0" rpy="0 0 0"/>
       <geometry>
-        <box size="0.10 0.10 0.10"/>
+        <box size="0.04 0.04 0.12"/>
       </geometry>
       <material name="cube_green">
@@ -55,5 +55,5 @@
       <origin xyz="0 0 0" rpy="0 0 0"/>
       <geometry>
-        <box size="0.10 0.10 0.10"/>
+        <box size="0.04 0.04 0.12"/>
       </geometry>
     </collision>
@@ -61,6 +61,8 @@
       <mass value="0.1"/>
       <origin xyz="0 0 0" rpy="0 0 0"/>
-      <!-- Solid cube inertia: (1/12)*m*(a^2 + b^2) = (1/12)*0.1*0.02 = 1.67e-4 -->
-      <inertia ixx="1.67e-4" ixy="0" ixz="0" iyy="1.67e-4" iyz="0" izz="1.67e-4"/>
+      <!-- Cuboid inertia for 4 x 4 x 12 cm, 100 g.
+           Ixx = Iyy = (1/12)*m*(a^2 + c^2) = (1/12)*0.1*(0.0016 + 0.0144) = 1.33e-4
+           Izz = (1/12)*m*(a^2 + b^2)       = (1/12)*0.1*(0.0016 + 0.0016) = 2.67e-5 -->
+      <inertia ixx="1.33e-4" ixy="0" ixz="0" iyy="1.33e-4" iyz="0" izz="2.67e-5"/>
     </inertial>
   </link>
@@ -68,6 +70,6 @@
     <parent link="world"/>
     <child link="cube_link"/>
-    <!-- Start sitting on the table top (0.7 m) + half the cube (0.05 m). -->
-    <origin xyz="0.55 0 0.75" rpy="0 0 0"/>
+    <!-- Start sitting on the table top (0.7 m) + half the cube height (0.06 m). -->
+    <origin xyz="0.55 0 0.76" rpy="0 0 0"/>
   </joint>
 </robot>
