Commit message: set new gripper for real and sim robot

File: robot_description/frida_description/urdf/TMR2025/FRIDA.urdf.xacro (robot description, xacro)
@@ -63,21 +63,21 @@
     model1300="$(arg model1300)" attach_to="$(arg attach_to)" attach_xyz="$(arg attach_xyz)" attach_rpy="$(arg attach_rpy)"
     robot_sn="$(arg robot_sn)" use_gazebo_camera="$(arg use_gazebo_camera)" mesh_suffix="$(arg mesh_suffix)" kinematics_suffix="$(arg kinematics_suffix)" />
+    <xacro:if value="$(arg load_zed)">
+      <xacro:include filename="$(find frida_description)/urdf/Gripper/Custom/gripper.xacro" />
+      <xacro:load_gripper attach_to="link_eef" xyz="0 0 0.046" rpy="0 0 3.14" fixed_joints="true"/>
+      <!-- ZED MACRO -->
+      <xacro:include filename="$(find frida_description)/urdf/zed/zed_macro.urdf.xacro" />
+      <xacro:zed_camera name="zed" model="zed2" custom_baseline="0" enable_gnss="false" simulation="true" attach_to="zed" xyz="0 0 0" rpy="0 0 0">
+          <origin xyz="0 0 0" rpy="0 0 0"/>
+      </xacro:zed_camera>
+    </xacro:if>
     <!-- <xacro:if value="$(arg load_zed)"> -->
-      <!-- <xacro:include filename="$(find frida_description)/urdf/Gripper/Custom/gripper.xacro" /> -->
-      <!-- <xacro:load_gripper attach_to="link_eef" xyz="0 0 0.046" rpy="0 0 1.57" fixed_joints="true"/> -->
+      <!-- <xacro:include filename="$(find frida_description)/urdf/Gripper/Commercial/gripper.xacro" /> -->
+      <!-- <xacro:load_gripper attach_to="link_eef" xyz="0 0 0" rpy="2.3562 -1.5708 0" fixed_joints="true"/> -->
       <!-- ZED MACRO -->
       <!-- <xacro:include filename="$(find frida_description)/urdf/zed/zed_macro.urdf.xacro" /> -->
-      <!-- <xacro:zed_camera name="zed" model="zed2" custom_baseline="0" enable_gnss="false" simulation="true" attach_to="zed" xyz="0 0 0" rpy="0 0 0"> -->
+      <!-- <xacro:zed_camera name="zed" model="zed2" custom_baseline="0" enable_gnss="false" simulation="true" attach_to="gripper" xyz="0.030461 0 -0.050649" rpy="0 0.81804 0"> -->
           <!-- <origin xyz="0 0 0" rpy="0 0 0"/> -->
       <!-- </xacro:zed_camera> -->
     <!-- </xacro:if> -->
-    <xacro:if value="$(arg load_zed)">
-      <xacro:include filename="$(find frida_description)/urdf/Gripper/Commercial/gripper.xacro" />
-      <xacro:load_gripper attach_to="link_eef" xyz="0 0 0" rpy="2.3562 -1.5708 0" fixed_joints="true"/>
-      <!-- ZED MACRO -->
-      <xacro:include filename="$(find frida_description)/urdf/zed/zed_macro.urdf.xacro" />
-      <xacro:zed_camera name="zed" model="zed2" custom_baseline="0" enable_gnss="false" simulation="true" attach_to="gripper" xyz="0.030461 0 -0.050649" rpy="0 0.81804 0">
-          <origin xyz="0 0 0" rpy="0 0 0"/>
-      </xacro:zed_camera>
-    </xacro:if>
 </robot>

File: robot_description/frida_description/urdf/TMR2025/FRIDA_Real.urdf.xacro (robot description, xacro)
@@ -66,16 +66,16 @@
   <!-- OLD GRIPPER    -->
   <!-- Gripper -->
-  <xacro:include filename="$(find frida_description)/urdf/Gripper/Commercial/gripper.xacro" />
-    <xacro:load_gripper attach_to="link_eef" xyz="0 0 0" rpy="2.3562 -1.5708 0" />
+  <!-- <xacro:include filename="$(find frida_description)/urdf/Gripper/Commercial/gripper.xacro" />
+    <xacro:load_gripper attach_to="link_eef" xyz="0 0 0" rpy="2.3562 -1.5708 0" /> -->
    <!-- ZED MACRO -->
-    <xacro:include filename="$(find frida_description)/urdf/zed/zed.xacro" />
-  <xacro:load_zed attach_to="gripper" xyz="0.046461 0 -0.075649" rpy="0 0.81804 0" />
+  <!-- <xacro:include filename="$(find frida_description)/urdf/zed/zed.xacro" />
+  <xacro:load_zed attach_to="gripper" xyz="0.046461 0 -0.075649" rpy="0 0.81804 0" /> -->
   <!-- NEW GRIPPER MACRO   -->
   <!-- Gripper -->
-  <!-- <xacro:include filename="$(find frida_description)/urdf/Gripper/Custom/gripper.xacro" />
-  <xacro:load_gripper attach_to="link_eef" xyz="0 0 0.046" rpy="0 0 1.57" /> -->
+  <xacro:include filename="$(find frida_description)/urdf/Gripper/Custom/gripper.xacro" />
+  <xacro:load_gripper attach_to="link_eef" xyz="0 0 0.046" rpy="0 0 1.57" fixed_joints="true"/>
    <!-- ZED MACRO -->
-  <!-- <xacro:include filename="$(find frida_description)/urdf/RoboCup2024/zed.xacro" />
-  <xacro:load_zed attach_to="zed" xyz="0 0 0" rpy="0 0 0" /> -->
+  <xacro:include filename="$(find frida_description)/urdf/zed/zed.xacro" />
+  <xacro:load_zed attach_to="zed" xyz="0 0 0" rpy="0 0 0" />
   <!-- <joint name="base_footprint_joint" type="fixed">
       <origin xyz="0 0 ${base_length/2 + caster_radius*2}" rpy="0 0 0" />

Commit message: PourManager skeleton and fix urdf and joint limits

File: robot_description/frida_description/urdf/TMR2025/FRIDA.urdf.xacro (robot description, xacro)
@@ -63,7 +63,13 @@
     model1300="$(arg model1300)" attach_to="$(arg attach_to)" attach_xyz="$(arg attach_xyz)" attach_rpy="$(arg attach_rpy)"
     robot_sn="$(arg robot_sn)" use_gazebo_camera="$(arg use_gazebo_camera)" mesh_suffix="$(arg mesh_suffix)" kinematics_suffix="$(arg kinematics_suffix)" />
+    <joint name="gripper_grasp_joint" type="fixed">
+      <parent link="link_eef"/>
+      <child link="gripper_grasp_frame"/>
+      <origin xyz="0 0 0" rpy="0 0 -0.7854"/>
+    </joint>
+    <link name="gripper_grasp_frame"> </link>
     <xacro:if value="$(arg load_zed)">
       <xacro:include filename="$(find frida_description)/urdf/Gripper/Custom/gripper.xacro" />
-      <xacro:load_gripper attach_to="link_eef" xyz="0 0 0.046" rpy="0 0 3.14" fixed_joints="true"/>
+      <xacro:load_gripper attach_to="link_eef" xyz="0 0 0.046" rpy="0 0 3.926" fixed_joints="true"/>
       <!-- ZED MACRO -->
       <xacro:include filename="$(find frida_description)/urdf/zed/zed_macro.urdf.xacro" />

Commit message: urdf on sim missing a link

File: robot_description/frida_description/urdf/TMR2025/FRIDA.urdf.xacro (robot description, xacro)
@@ -63,4 +63,10 @@
     model1300="$(arg model1300)" attach_to="$(arg attach_to)" attach_xyz="$(arg attach_xyz)" attach_rpy="$(arg attach_rpy)"
     robot_sn="$(arg robot_sn)" use_gazebo_camera="$(arg use_gazebo_camera)" mesh_suffix="$(arg mesh_suffix)" kinematics_suffix="$(arg kinematics_suffix)" />
+    <joint name="gripper_grasp_joint" type="fixed">
+      <parent link="link_eef"/>
+      <child link="gripper_grasp_frame"/>
+      <origin xyz="0 0 0" rpy="0 0 -0.7854"/>
+    </joint>
+    <link name="gripper_grasp_frame"> </link>
     <xacro:if value="$(arg load_zed)">
       <xacro:include filename="$(find frida_description)/urdf/Gripper/Custom/gripper.xacro" />

Commit message: Functional actuators added, solve problem with additional_files
Added actuators for FRIDA in the xarm
Actuators controlled by the ros2_control interfaces
Need check on parameters of this actuators
Need final fix on the gripper joint and actuators

File: robot_description/frida_description/urdf/TMR2025/FRIDA.urdf.xacro (robot description, xacro)
@@ -44,4 +44,17 @@
   <xacro:arg name="simulation" default="false"/>
   <xacro:include filename="robot.xacro"/>
+      <!-- Mujoco Config -->
+    <xacro:if value="$(arg mujoco_plugin)">
+      <mujoco>
+        <compiler angle="radian" balanceinertia="true" />
+      </mujoco>
+      <!-- Important to add additional files in the spawn -->
+      <link name="world" />
+      <joint name="world_to_base" type="floating">
+        <parent link="world" />
+        <child link="base_link" />
+        <origin rpy="0 0 0" xyz="0 0 0.5" />
+      </joint>
+    </xacro:if>
   <xacro:include filename="$(find frida_description)/urdf/xarm/xarm_device_macro.xacro" />
     <xacro:xarm_device prefix="$(arg prefix)" hw_ns="$(arg hw_ns)" limited="$(arg limited)"
@@ -51,5 +64,5 @@
     ros2_control_plugin="$(arg ros2_control_plugin)" robot_type="$(arg robot_type)"
     mujoco_plugin="$(arg mujoco_plugin)"
-    load_gazebo_plugin="true" ros2_control_params="$(arg ros2_control_params)"
+    load_gazebo_plugin="false" ros2_control_params="$(arg ros2_control_params)"
     add_realsense_d435i="$(arg add_realsense_d435i)"
     add_d435i_links="$(arg add_d435i_links)"
@@ -65,10 +78,4 @@
     model1300="$(arg model1300)" attach_to="$(arg attach_to)" attach_xyz="$(arg attach_xyz)" attach_rpy="$(arg attach_rpy)"
     robot_sn="$(arg robot_sn)" use_gazebo_camera="$(arg use_gazebo_camera)" mesh_suffix="$(arg mesh_suffix)" kinematics_suffix="$(arg kinematics_suffix)" />
-        <!-- Mujoco Config -->
-    <xacro:if value="$(arg mujoco_plugin)">
-      <mujoco>
-        <compiler angle="radian" />
-      </mujoco>
-    </xacro:if>
 <joint name="gripper_grasp_joint" type="fixed">
       <parent link="link_eef"/>

File: robot_description/frida_description/urdf/xarm/xarm6/xarm6_robot_macro.xacro (robot description, xacro)
@@ -16,5 +16,6 @@
     inertial_params_filename:=''
     kinematics_params_filename:=''
-    hard_interface:='PositionJointInterface' "
+    hard_interface:='PositionJointInterface'
+    mujoco_plugin:=false "
     >
     <!-- include xarm6 relative macros: -->
@@ -67,4 +68,10 @@
     <xacro:xarm6_transmission prefix="${prefix}" hard_interface="${hard_interface}" />
     <xacro:xarm6_gazebo prefix="${prefix}" />
+    <xacro:if value="${mujoco_plugin}">
+      <xacro:include filename="$(find frida_description)/urdf/xarm/xarm6/xarm6.mujoco_actuators.xacro"/>
+      <mujoco>
+        <xacro:create_xarm_mujoco_actuators/>
+      </mujoco>
+    </xacro:if>
   </xacro:macro>
 </robot>

File: robot_description/frida_description/urdf/xarm/xarm_device_macro.xacro (robot description, xacro)
@@ -42,5 +42,5 @@
     mesh_suffix:='stl'
     kinematics_suffix:=''
-    mujoco_plugin:=true
+    mujoco_plugin:=false
     "
     >
@@ -166,5 +166,6 @@
           inertial_params_filename="${inertial_params_filename}"
           kinematics_params_filename="${kinematics_params_filename}"
-          hard_interface="${hard_interface}" />
+          hard_interface="${hard_interface}"
+          mujoco_plugin = "${mujoco_plugin}" />
       </xacro:unless>
     </xacro:if>

File: robot_description/frida_description/urdf/zed/zed_macro.urdf.xacro (robot description, xacro)
@@ -174,4 +174,12 @@
           </collision>
         </xacro:if>
+        <xacro:unless value="${model=='virtual'}">
+          <visual>
+            <origin xyz="0 0 0" rpy="0 0 0"/>
+            <geometry>
+              <box size="0.001 0.001 0.001"/>
+            </geometry>
+          </visual>
+        </xacro:unless>
       </link>
       <mujoco>

Commit message: switch frida_real for new package

File: robot_description/frida_description/urdf/TMR2025/FRIDA.urdf.xacro (robot description, xacro)
@@ -43,5 +43,5 @@
   <xacro:arg name="load_zed" default="false"/>
   <xacro:arg name="simulation" default="false"/>
-  <xacro:include filename="robot.xacro"/>
+  <xacro:include filename="$(find home_custom_base_description)/urdf/robot.xacro"/>
       <!-- Mujoco Config -->
     <xacro:if value="$(arg mujoco_plugin)">

File: robot_description/frida_description/urdf/TMR2025/FRIDA_Real.urdf.xacro (robot description, xacro)
@@ -43,5 +43,5 @@
   <!-- ZED ARGUMENTS -->
   <!-- ROBOT COMPONENTS -->
-  <xacro:include filename="robot_real.xacro"/>
+  <xacro:include filename="../../../home_custom_base_description/urdf/robot.xacro"/>
   <!-- MUJOCO PARAMS -->
   <!-- gravcomp mirrors the xarm6 firmware's internal gravity compensation:

File: robot_description/frida_description/urdf/zed/zed.xacro (robot description, xacro)
@@ -2,4 +2,5 @@
 <robot xmlns:xacro="http://www.ros.org/wiki/xacro">
 <xacro:property name="mesh_path" value="file://$(find frida_description)/urdf/meshes/Gripper/Commercial/" />
+<xacro:property name="black_rgba" value="0.102 0.102 0.102 1" />
 <xacro:macro name="load_zed" params="attach_to:='' xyz:='0 0 0' rpy:='0 0 0' mujoco_plugin:=false" >
     <xacro:unless value="${attach_to == ''}">

File: robot_description/home_custom_base_description/urdf/robot.xacro (robot description, xacro)
@@ -10,5 +10,5 @@
   <!-- Conditionally include simulation files -->
   <xacro:if value="${use_sim_time}">
-    <xacro:include filename="$(find home_custom_base_description)/urdf/home_base_ros2_control.xacro"/>
+    <xacro:include filename="home_base_ros2_control.xacro"/>
   </xacro:if>
   <material name="home_base_gray">

Commit message: fix the urdf of the omnibase

File: robot_description/frida_description/urdf/TMR2025/FRIDA.urdf.xacro (robot description, xacro)
@@ -1,4 +1,4 @@
 <?xml version="1.0" encoding="utf-8"?>
-<robot name="FRIDA" xmlns:xacro="http://www.ros.org/wiki/xacro">
+<robot name="FRIDA" xmlns:xacro="http://www.ros.org/wiki/xacro" xmlns:gz="http://gazebosim.org/schema">
   <xacro:arg name="prefix" default=""/>
   <xacro:arg name="hw_ns" default="xarm"/>

File: robot_description/frida_description/urdf/TMR2025/FRIDA_Real.urdf.xacro (robot description, xacro)
@@ -1,4 +1,4 @@
 <?xml version="1.0" encoding="utf-8"?>
-<robot name="FRIDA" xmlns:xacro="http://www.ros.org/wiki/xacro">
+<robot name="FRIDA" xmlns:xacro="http://www.ros.org/wiki/xacro" xmlns:gz="http://gazebosim.org/schema">
 <!-- XARM ARGUMENTS -->
   <xacro:arg name="prefix" default=""/>
@@ -92,5 +92,5 @@
     <joint name="world_to_base" type="fixed">
       <parent link="world" />
-      <child link="base_link" />
+      <child link="_base_footprint" />
       <origin rpy="0 0 0" xyz="0 0 0" />
     </joint>
@@ -99,5 +99,5 @@
     <joint name="world_to_base" type="fixed">
       <parent link="world" />
-      <child link="base_link" />
+      <child link="_base_footprint" />
       <origin rpy="0 0 0" xyz="0 0 0.3" />
     </joint>

Commit message: Updated modular omni

File: robot_description/frida_description/urdf/TMR2025/FRIDA.urdf.xacro (robot description, xacro)
@@ -43,5 +43,5 @@
   <xacro:arg name="load_zed" default="false"/>
   <xacro:arg name="simulation" default="false"/>
-  <xacro:include filename="$(find home_custom_base_description)/urdf/robot.xacro"/>
+  <xacro:include filename="robot.xacro"/>
       <!-- Mujoco Config -->
     <xacro:if value="$(arg mujoco_plugin)">

File: robot_description/frida_description/urdf/zed/zed.xacro (robot description, xacro)
@@ -2,5 +2,4 @@
 <robot xmlns:xacro="http://www.ros.org/wiki/xacro">
 <xacro:property name="mesh_path" value="file://$(find frida_description)/urdf/meshes/Gripper/Commercial/" />
-<xacro:property name="black_rgba" value="0.102 0.102 0.102 1" />
 <xacro:macro name="load_zed" params="attach_to:='' xyz:='0 0 0' rpy:='0 0 0' mujoco_plugin:=false" >
     <xacro:unless value="${attach_to == ''}">
