Commit message: Remove MuJoCo/gazebo xacro blocks and plumbing

File: robot_description/frida_description/urdf/TMR2025/FRIDA.urdf.xacro (robot description, xacro)
@@ -17,5 +17,4 @@
   <xacro:arg name="ros2_control_plugin" default="uf_robot_hardware/UFRobotSystemHardware"/>
   <xacro:arg name="ros2_control_params" default=""/>
-  <xacro:arg name="mujoco_plugin" default="false"/>
   <xacro:arg name="add_realsense_d435i" default="false"/>
   <xacro:arg name="add_d435i_links" default="true"/>
@@ -44,17 +43,4 @@
   <xacro:arg name="simulation" default="false"/>
   <xacro:include filename="robot.xacro"/>
-      <!-- Mujoco Config -->
-    <xacro:if value="$(arg mujoco_plugin)">
-      <mujoco>
-        <compiler angle="radian" balanceinertia="true" autolimits="true"/>
-      </mujoco>
-      <!-- Important in order to add additional files in the spawn -->
-      <link name="world" />
-      <joint name="world_to_base" type="floating">
-        <parent link="world" />
-        <child link="base_link" />
-        <origin rpy="0 0 0" xyz="0 0 0.5" />
-      </joint>
-    </xacro:if>
   <xacro:include filename="$(find frida_description)/urdf/xarm/xarm_device_macro.xacro" />
     <xacro:xarm_device prefix="$(arg prefix)" hw_ns="$(arg hw_ns)" limited="$(arg limited)"
@@ -63,5 +49,4 @@
     add_bio_gripper="$(arg add_bio_gripper)" dof="$(arg dof)"
     ros2_control_plugin="$(arg ros2_control_plugin)" robot_type="$(arg robot_type)"
-    mujoco_plugin="$(arg mujoco_plugin)"
     load_gazebo_plugin="false" ros2_control_params="$(arg ros2_control_params)"
     add_realsense_d435i="$(arg add_realsense_d435i)"
@@ -87,7 +72,7 @@
     <xacro:if value="$(arg load_zed)">
       <xacro:include filename="$(find frida_description)/urdf/Gripper/Custom/gripper.xacro" />
-      <xacro:load_gripper attach_to="link_eef" xyz="0 0 0.046" rpy="0 0 3.926" fixed_joints="false" mujoco_plugin="$(arg mujoco_plugin)" />
+      <xacro:load_gripper attach_to="link_eef" xyz="0 0 0.046" rpy="0 0 3.926" fixed_joints="false" />
       <xacro:include filename="$(find frida_description)/urdf/zed/zed.xacro" />
-      <xacro:load_zed attach_to="zed" xyz="0 0 0" rpy="0 0 0" mujoco_plugin="$(arg mujoco_plugin)" />
+      <xacro:load_zed attach_to="zed" xyz="0 0 0" rpy="0 0 0" />
     </xacro:if>
     <!-- <xacro:if value="$(arg load_zed)"> -->

File: robot_description/frida_description/urdf/TMR2025/FRIDA_Real.urdf.xacro (robot description, xacro)
@@ -34,5 +34,4 @@
   <xacro:arg name="geometry_mesh_tcp_rpy" default="0 0 0"/>
   <xacro:arg name="baud_checkset" default="true"/>
-  <xacro:arg name="mujoco_plugin" default="false"/>
   <xacro:arg name="default_gripper_baud" default="2000000"/>
   <xacro:arg name="attach_to" default="xarm_base"/>
@@ -44,63 +43,15 @@
   <!-- ROBOT COMPONENTS -->
   <xacro:include filename="robot_real.xacro"/>
-  <!-- MUJOCO PARAMS -->
-  <!-- gravcomp mirrors the xarm6 firmware's internal gravity compensation:
-       the real servos hold pose against gravity on their own, so the sim does the same.
-       Applied only on arm+gripper bodies so world objects still fall realistically. -->
-  <xacro:if value="$(arg mujoco_plugin)">
-    <mujoco>
-      <compiler angle="radian" balanceinertia="true" autolimits="true"/>
-      <!-- Sim-only solver tuning for reliable physics-based grasping.
-           The combination below keeps the cheap defaults where they work
-           (PGS is fine for articulated dynamics) but adds the two knobs
-           that matter for grasping stability:
-             impratio=10: tightens the friction cone so the tangential
-                friction ceiling stays proportional to normal force under
-                rapid normal-force changes.
-             noslip_iterations=5: post-solve pass that explicitly enforces
-                no-tangential-slip at each contact point.
-           The more aggressive integrator=implicit + solver=Newton +
-           cone=elliptic combo was tested but tripled the physics cost
-           and stalled the sim well below realtime so ros2_control timed
-           out, which looks externally like the pick freezing in place. -->
-      <option impratio="10"
-              noslip_iterations="5"/>
-      <reference name="link1"><body gravcomp="1"/></reference>
-      <reference name="link2"><body gravcomp="1"/></reference>
-      <reference name="link3"><body gravcomp="1"/></reference>
-      <reference name="link4"><body gravcomp="1"/></reference>
-      <reference name="link5"><body gravcomp="1"/></reference>
-      <reference name="link6"><body gravcomp="1"/></reference>
-      <reference name="link_eef"><body gravcomp="1"/></reference>
-      <reference name="gripper"><body gravcomp="1"/></reference>
-      <reference name="right_finger"><body gravcomp="1"/></reference>
-      <reference name="left_finger"><body gravcomp="1"/></reference>
-      <reference name="zed"><body gravcomp="1"/></reference>
-      <reference name="zed_camera_link"><body gravcomp="1"/></reference>
-    </mujoco>
-  </xacro:if>
   <!-- The world<->base_link offset matters for MoveIt because "world" is the
        planning frame: the plane-collision-object added by perception_3d in
        "base_link" gets stored by MoveIt in "world", and pick_server.check_
        feasibility compares its z against the grasp pose (in "base_link").
-       Any non-zero offset becomes a silent frame mismatch that fails every
-       pick.  On the real robot the 0.3 m pedestal is the physical mounting;
-       in MuJoCo the arm is attached directly to world and there is no
-       pedestal, so pin world<->base_link at identity for sim only. -->
+       The 0.3 m pedestal is the physical mounting. -->
   <link name="world" />
-  <xacro:if value="$(arg mujoco_plugin)">
-    <joint name="world_to_base" type="fixed">
-      <parent link="world" />
-      <child link="base_link" />
-      <origin rpy="0 0 0" xyz="0 0 0" />
-    </joint>
-  </xacro:if>
-  <xacro:unless value="$(arg mujoco_plugin)">
-    <joint name="world_to_base" type="fixed">
-      <parent link="world" />
-      <child link="base_link" />
-      <origin rpy="0 0 0" xyz="0 0 0.3" />
-    </joint>
-  </xacro:unless>
+  <joint name="world_to_base" type="fixed">
+    <parent link="world" />
+    <child link="base_link" />
+    <origin rpy="0 0 0" xyz="0 0 0.3" />
+  </joint>
   <!-- XARM MACRO -->
   <xacro:include filename="$(find frida_description)/urdf/xarm/xarm_device_macro.xacro" />
@@ -110,5 +61,4 @@
     add_bio_gripper="$(arg add_bio_gripper)" dof="$(arg dof)"
     ros2_control_plugin="$(arg ros2_control_plugin)" robot_type="$(arg robot_type)"
-    mujoco_plugin="$(arg mujoco_plugin)"
     load_gazebo_plugin="false" ros2_control_params="$(arg ros2_control_params)"
     add_realsense_d435i="$(arg add_realsense_d435i)"
@@ -141,8 +91,8 @@
   <!-- Gripper -->
   <xacro:include filename="$(find frida_description)/urdf/Gripper/Custom/gripper.xacro" />
-  <xacro:load_gripper attach_to="link_eef" xyz="0 0 0.046" rpy="0 0 3.926" fixed_joints="false" mujoco_plugin="$(arg mujoco_plugin)" ros2_control_plugin="$(arg ros2_control_plugin)"/>
+  <xacro:load_gripper attach_to="link_eef" xyz="0 0 0.046" rpy="0 0 3.926" fixed_joints="false" ros2_control_plugin="$(arg ros2_control_plugin)"/>
    <!-- ZED MACRO -->
   <xacro:include filename="$(find frida_description)/urdf/zed/zed.xacro" />
-  <xacro:load_zed attach_to="zed" xyz="0.0 0 0.0" rpy="0 0 0"  mujoco_plugin="$(arg mujoco_plugin)" />
+  <xacro:load_zed attach_to="zed" xyz="0.0 0 0.0" rpy="0 0 0" />
   <!-- <joint name="base_footprint_joint" type="fixed">
       <origin xyz="0 0 ${base_length/2 + caster_radius*2}" rpy="0 0 0" />

File: robot_description/frida_description/urdf/omnibase/FRIDA_Real.urdf.xacro (robot description, xacro)
@@ -34,5 +34,4 @@
   <xacro:arg name="geometry_mesh_tcp_rpy" default="0 0 0"/>
   <xacro:arg name="baud_checkset" default="true"/>
-  <xacro:arg name="mujoco_plugin" default="false"/>
   <xacro:arg name="default_gripper_baud" default="2000000"/>
   <xacro:arg name="attach_to" default="xarm_base"/>
@@ -44,48 +43,11 @@
   <!-- ROBOT COMPONENTS -->
   <xacro:include filename="$(find frida_description)/urdf/omnibase/robot.xacro"/>
-  <!-- MUJOCO PARAMS -->
-  <!-- gravcomp mirrors the xarm6 firmware's internal gravity compensation:
-       the real servos hold pose against gravity on their own, so the sim does the same.
-       Applied only on arm+gripper bodies so world objects still fall realistically. -->
-  <xacro:if value="$(arg mujoco_plugin)">
-    <mujoco>
-      <compiler angle="radian" balanceinertia="true" autolimits="true"/>
-      <!-- Sim-only solver tuning for reliable physics-based grasping.
-           The combination below keeps the cheap defaults where they work
-           (PGS is fine for articulated dynamics) but adds the two knobs
-           that matter for grasping stability:
-             impratio=10: tightens the friction cone so the tangential
-                friction ceiling stays proportional to normal force under
-                rapid normal-force changes.
-             noslip_iterations=5: post-solve pass that explicitly enforces
-                no-tangential-slip at each contact point.
-           The more aggressive integrator=implicit + solver=Newton +
-           cone=elliptic combo was tested but tripled the physics cost
-           and stalled the sim well below realtime so ros2_control timed
-           out, which looks externally like the pick freezing in place. -->
-      <option impratio="10"
-              noslip_iterations="5"/>
-      <reference name="link1"><body gravcomp="1"/></reference>
-      <reference name="link2"><body gravcomp="1"/></reference>
-      <reference name="link3"><body gravcomp="1"/></reference>
-      <reference name="link4"><body gravcomp="1"/></reference>
-      <reference name="link5"><body gravcomp="1"/></reference>
-      <reference name="link6"><body gravcomp="1"/></reference>
-      <reference name="link_eef"><body gravcomp="1"/></reference>
-      <reference name="gripper"><body gravcomp="1"/></reference>
-      <reference name="right_finger"><body gravcomp="1"/></reference>
-      <reference name="left_finger"><body gravcomp="1"/></reference>
-      <reference name="zed"><body gravcomp="1"/></reference>
-      <reference name="zed_camera_link"><body gravcomp="1"/></reference>
-    </mujoco>
-  </xacro:if>
-  <xacro:if value="$(arg mujoco_plugin)">
-    <link name="world" />
-    <joint name="world_to_base" type="fixed">
-      <parent link="world" />
-      <child link="base_footprint" />
-      <origin rpy="0 0 0" xyz="0 0 0" />
-    </joint>
-  </xacro:if>
+  <!-- World link and static transform for real hardware/planning frame -->
+  <link name="world" />
+  <joint name="world_to_base" type="fixed">
+    <parent link="world" />
+    <child link="base_link" />
+    <origin rpy="0 0 0" xyz="0 0 0" />
+  </joint>
   <!-- XARM MACRO -->
   <xacro:include filename="$(find frida_description)/urdf/xarm/xarm_device_macro.xacro" />
@@ -95,5 +57,4 @@
     add_bio_gripper="$(arg add_bio_gripper)" dof="$(arg dof)"
     ros2_control_plugin="$(arg ros2_control_plugin)" robot_type="$(arg robot_type)"
-    mujoco_plugin="$(arg mujoco_plugin)"
     load_gazebo_plugin="false" ros2_control_params="$(arg ros2_control_params)"
     add_realsense_d435i="$(arg add_realsense_d435i)"
@@ -126,8 +87,8 @@
   <!-- Gripper -->
   <xacro:include filename="$(find frida_description)/urdf/Gripper/Custom/gripper.xacro" />
-  <xacro:load_gripper attach_to="link_eef" xyz="0 0 0.046" rpy="0 0 3.926" fixed_joints="false" mujoco_plugin="$(arg mujoco_plugin)" ros2_control_plugin="$(arg ros2_control_plugin)"/>
+  <xacro:load_gripper attach_to="link_eef" xyz="0 0 0.046" rpy="0 0 3.926" fixed_joints="false" ros2_control_plugin="$(arg ros2_control_plugin)"/>
    <!-- ZED MACRO -->
   <xacro:include filename="$(find frida_description)/urdf/zed/zed.xacro" />
-  <xacro:load_zed attach_to="zed" xyz="0.0 0 0.0" rpy="0 0 0"  mujoco_plugin="$(arg mujoco_plugin)" />
+  <xacro:load_zed attach_to="zed" xyz="0.0 0 0.0" rpy="0 0 0" />
   <!-- <joint name="base_footprint_joint" type="fixed">
       <origin xyz="0 0 ${base_length/2 + caster_radius*2}" rpy="0 0 0" />
