Commit message: added a grasp frame to correct 45degree rotation

File: robot_description/frida_description/urdf/TMR2025/FRIDA_Real.urdf.xacro (robot description, xacro)
@@ -71,4 +71,10 @@
   <!-- <xacro:include filename="$(find frida_description)/urdf/zed/zed.xacro" />
   <xacro:load_zed attach_to="gripper" xyz="0.046461 0 -0.075649" rpy="0 0.81804 0" /> -->
+  <joint name="gripper_grasp_joint" type="fixed">
+    <parent link="link_eef"/>
+    <child link="gripper_grasp_frame"/>
+    <origin xyz="0 0 0" rpy="0 0 -0.7854"/>
+  </joint>
+  <link name="gripper_grasp_frame"> </link>
   <!-- NEW GRIPPER MACRO   -->
   <!-- Gripper -->

Commit message: New Gripper Pick and Place (#337) -> Big one
* set new gripper for real and sim robot

* Working pick and place on new gripper, somewhat stable

* new params, adjust zed position

* Reliability stuff, try pick alternatives and check feasibility  to discard poses immediately if needed

* wait grasp service

* fixes

* added a grasp frame to correct 45degree rotation

* Somwhat stable new gripper pick and place

* Stable pick and place with place on shelves

---------

Co-authored-by: Ivan Romero <i.wells.ar@gmail.com>

File: robot_description/frida_description/urdf/TMR2025/FRIDA_Real.urdf.xacro (robot description, xacro)
@@ -66,16 +66,22 @@
   <!-- OLD GRIPPER    -->
   <!-- Gripper -->
-  <xacro:include filename="$(find frida_description)/urdf/Gripper/Commercial/gripper.xacro" />
-    <xacro:load_gripper attach_to="link_eef" xyz="0 0 0" rpy="2.3562 -1.5708 0" />
+  <!-- <xacro:include filename="$(find frida_description)/urdf/Gripper/Commercial/gripper.xacro" />
+    <xacro:load_gripper attach_to="link_eef" xyz="0 0 0" rpy="2.3562 -1.5708 0" /> -->
    <!-- ZED MACRO -->
-    <xacro:include filename="$(find frida_description)/urdf/zed/zed.xacro" />
-  <xacro:load_zed attach_to="gripper" xyz="0.046461 0 -0.075649" rpy="0 0.81804 0" />
+  <!-- <xacro:include filename="$(find frida_description)/urdf/zed/zed.xacro" />
+  <xacro:load_zed attach_to="gripper" xyz="0.046461 0 -0.075649" rpy="0 0.81804 0" /> -->
+  <joint name="gripper_grasp_joint" type="fixed">
+    <parent link="link_eef"/>
+    <child link="gripper_grasp_frame"/>
+    <origin xyz="0 0 0" rpy="0 0 -0.7854"/>
+  </joint>
+  <link name="gripper_grasp_frame"> </link>
   <!-- NEW GRIPPER MACRO   -->
   <!-- Gripper -->
-  <!-- <xacro:include filename="$(find frida_description)/urdf/Gripper/Custom/gripper.xacro" />
-  <xacro:load_gripper attach_to="link_eef" xyz="0 0 0.046" rpy="0 0 1.57" /> -->
+  <xacro:include filename="$(find frida_description)/urdf/Gripper/Custom/gripper.xacro" />
+  <xacro:load_gripper attach_to="link_eef" xyz="0 0 0.046" rpy="0 0 3.926" fixed_joints="true"/>
    <!-- ZED MACRO -->
-  <!-- <xacro:include filename="$(find frida_description)/urdf/RoboCup2024/zed.xacro" />
-  <xacro:load_zed attach_to="zed" xyz="0 0 0" rpy="0 0 0" /> -->
+  <xacro:include filename="$(find frida_description)/urdf/zed/zed.xacro" />
+  <xacro:load_zed attach_to="zed" xyz="0.0 0 0.0" rpy="0 0 0" />
   <!-- <joint name="base_footprint_joint" type="fixed">
       <origin xyz="0 0 ${base_length/2 + caster_radius*2}" rpy="0 0 0" />

Commit message: finish yml with all spheres

File: robot_description/frida_description/urdf/TMR2025/FRIDA_Real.urdf.xacro (robot description, xacro)
@@ -80,5 +80,5 @@
   <!-- Gripper -->
   <xacro:include filename="$(find frida_description)/urdf/Gripper/Custom/gripper.xacro" />
-  <xacro:load_gripper attach_to="link_eef" xyz="0 0 0.046" rpy="0 0 3.926" fixed_joints="true"/>
+  <xacro:load_gripper attach_to="link_eef" xyz="0 0 0.046" rpy="0 0 3.926" fixed_joints="false"/>
    <!-- ZED MACRO -->
   <xacro:include filename="$(find frida_description)/urdf/zed/zed.xacro" />

File: robot_description/frida_description/urdf/TMR2025/base.xacro (robot description, xacro)
@@ -20,5 +20,5 @@
       <origin xyz="0 0 0" rpy="0 0 0" />
       <geometry>
-        <mesh filename="${mesh_path}base_link_simplified.stl" scale="0.1 0.1 0.1"/>
+        <mesh filename="${mesh_path}base_link_simplified.stl"/>
       </geometry>
     </collision>

File: robot_description/frida_description/urdf/TMR2025/frida_real.urdf (robot description, URDF)
Before this commit: robot FRIDA, 15 links, 13 joints
Links:
- link base_link: geometry collision mesh filename=meshes/base_link_simplified.stl; visual mesh filename=meshes/base_link.stl

Commit message: Move it addition

File: robot_description/frida_description/urdf/TMR2025/FRIDA_Real.urdf.xacro (robot description, xacro)
@@ -34,4 +34,5 @@
   <xacro:arg name="geometry_mesh_tcp_rpy" default="0 0 0"/>
   <xacro:arg name="baud_checkset" default="true"/>
+  <xacro:arg name="mujoco_plugin" default="false"/>
   <xacro:arg name="default_gripper_baud" default="2000000"/>
   <xacro:arg name="attach_to" default="xarm_base"/>
@@ -43,4 +44,17 @@
   <!-- ROBOT COMPONENTS -->
   <xacro:include filename="robot_real.xacro"/>
+  <!-- MUJOCO PARAMS -->
+  <xacro:if value="$(arg mujoco_plugin)">
+    <mujoco>
+      <compiler angle="radian" balanceinertia="true" autolimits="true"/>
+    </mujoco>
+    <!-- Important in order to add additional files in the spawn -->
+    <link name="world" />
+    <joint name="world_to_base" type="fixed">
+      <parent link="world" />
+      <child link="base_link" />
+      <origin rpy="0 0 0" xyz="0 0 0.3" />
+    </joint>
+  </xacro:if>
   <!-- XARM MACRO -->
   <xacro:include filename="$(find frida_description)/urdf/xarm/xarm_device_macro.xacro" />
@@ -50,5 +64,6 @@
     add_bio_gripper="$(arg add_bio_gripper)" dof="$(arg dof)"
     ros2_control_plugin="$(arg ros2_control_plugin)" robot_type="$(arg robot_type)"
-    load_gazebo_plugin="true" ros2_control_params="$(arg ros2_control_params)"
+    mujoco_plugin="$(arg mujoco_plugin)"
+    load_gazebo_plugin="false" ros2_control_params="$(arg ros2_control_params)"
     add_realsense_d435i="$(arg add_realsense_d435i)"
     add_d435i_links="$(arg add_d435i_links)"
@@ -80,8 +95,8 @@
   <!-- Gripper -->
   <xacro:include filename="$(find frida_description)/urdf/Gripper/Custom/gripper.xacro" />
-  <xacro:load_gripper attach_to="link_eef" xyz="0 0 0.046" rpy="0 0 3.926" fixed_joints="true"/>
+  <xacro:load_gripper attach_to="link_eef" xyz="0 0 0.046" rpy="0 0 3.926" fixed_joints="false" mujoco_plugin="$(arg mujoco_plugin)"/>
    <!-- ZED MACRO -->
   <xacro:include filename="$(find frida_description)/urdf/zed/zed.xacro" />
-  <xacro:load_zed attach_to="zed" xyz="0.0 0 0.0" rpy="0 0 0" />
+  <xacro:load_zed attach_to="zed" xyz="0.0 0 0.0" rpy="0 0 0"  mujoco_plugin="$(arg mujoco_plugin)" />
   <!-- <joint name="base_footprint_joint" type="fixed">
       <origin xyz="0 0 ${base_length/2 + caster_radius*2}" rpy="0 0 0" />

File: robot_description/frida_description/urdf/zed/zed.xacro (robot description, xacro)
@@ -2,5 +2,5 @@
 <robot xmlns:xacro="http://www.ros.org/wiki/xacro">
 <xacro:property name="mesh_path" value="file://$(find frida_description)/urdf/meshes/Gripper/Commercial/" />
-<xacro:macro name="load_zed" params="attach_to:='' xyz:='0 0 0' rpy:='0 0 0'">
+<xacro:macro name="load_zed" params="attach_to:='' xyz:='0 0 0' rpy:='0 0 0' mujoco_plugin:=false" >
     <xacro:unless value="${attach_to == ''}">
       <joint name="zed" type="fixed">
@@ -33,4 +33,11 @@
     </collision>
   </link>
+  <xacro:if value="${mujoco_plugin}">
+    <mujoco>
+      <reference name="${attach_to}">
+        <camera name="zed_mujoco_camera_link" mode="fixed" fovy="45" quat="-0.5 -0.5 0.5 0.5 "/>
+        </reference>
+    </mujoco>
+  </xacro:if>
 </xacro:macro>
 </robot>

Commit message: feat: integrate URDF components for FRIDA robot and add MoveIt launch configuration

File: robot_description/frida_description/urdf/TMR2025/FRIDA_Real.urdf.xacro (robot description, xacro)
@@ -88,6 +88,6 @@
        in MuJoCo the arm is attached directly to world and there is no
        pedestal, so pin world<->base_link at identity for sim only. -->
-  <link name="world" />
   <xacro:if value="$(arg mujoco_plugin)">
+    <link name="world" />
     <joint name="world_to_base" type="fixed">
       <parent link="world" />
@@ -96,11 +96,4 @@
     </joint>
   </xacro:if>
-  <xacro:unless value="$(arg mujoco_plugin)">
-    <joint name="world_to_base" type="fixed">
-      <parent link="world" />
-      <child link="base_link" />
-      <origin rpy="0 0 0" xyz="0 0 0.3" />
-    </joint>
-  </xacro:unless>
   <!-- XARM MACRO -->
   <xacro:include filename="$(find frida_description)/urdf/xarm/xarm_device_macro.xacro" />

File: robot_description/frida_description/urdf/TMR2025/base.xacro (robot description, xacro)
@@ -26,6 +26,6 @@
   <link name="base_footprint" />
   <joint name = "base_footprint_joint" type="fixed">
-    <parent link="base_link"/>
-    <child link="base_footprint"/>
+    <parent link="base_footprint"/>
+    <child link="base_link"/>
     <origin xyz="0 0 0" rpy="0 0 0 "/>
     <axis xyz="0 0 1"/>

Commit message: Revert "feat: integrate URDF components for FRIDA robot and add MoveIt launch configuration"
This reverts commit bc89a8f717e97a0c678689fe08d8c58ea7cb5a66.

File: robot_description/frida_description/urdf/TMR2025/FRIDA_Real.urdf.xacro (robot description, xacro)
@@ -88,6 +88,6 @@
        in MuJoCo the arm is attached directly to world and there is no
        pedestal, so pin world<->base_link at identity for sim only. -->
+  <link name="world" />
   <xacro:if value="$(arg mujoco_plugin)">
-    <link name="world" />
     <joint name="world_to_base" type="fixed">
       <parent link="world" />
@@ -96,4 +96,11 @@
     </joint>
   </xacro:if>
+  <xacro:unless value="$(arg mujoco_plugin)">
+    <joint name="world_to_base" type="fixed">
+      <parent link="world" />
+      <child link="base_link" />
+      <origin rpy="0 0 0" xyz="0 0 0.3" />
+    </joint>
+  </xacro:unless>
   <!-- XARM MACRO -->
   <xacro:include filename="$(find frida_description)/urdf/xarm/xarm_device_macro.xacro" />

File: robot_description/frida_description/urdf/TMR2025/base.xacro (robot description, xacro)
@@ -26,6 +26,6 @@
   <link name="base_footprint" />
   <joint name = "base_footprint_joint" type="fixed">
-    <parent link="base_footprint"/>
-    <child link="base_link"/>
+    <parent link="base_link"/>
+    <child link="base_footprint"/>
     <origin xyz="0 0 0" rpy="0 0 0 "/>
     <axis xyz="0 0 1"/>

Commit message: feat: add navigation support to MoveIt configuration and related launch files

File: robot_description/frida_description/urdf/TMR2025/FRIDA_Real.urdf.xacro (robot description, xacro)
@@ -36,4 +36,5 @@
   <xacro:arg name="mujoco_plugin" default="false"/>
   <xacro:arg name="default_gripper_baud" default="2000000"/>
+  <xacro:arg name="use_nav" default="false"/>
   <xacro:arg name="attach_to" default="xarm_base"/>
   <xacro:arg name="attach_xyz" default="0 0 0"/>
@@ -89,18 +90,29 @@
        pedestal, so pin world<->base_link at identity for sim only. -->
   <link name="world" />
-  <xacro:if value="$(arg mujoco_plugin)">
-    <joint name="world_to_base" type="fixed">
-      <parent link="world" />
-      <child link="base_link" />
-      <origin rpy="0 0 0" xyz="0 0 0" />
+  <!-- use_nav=false (default): world is root; standalone manipulation or sim -->
+  <xacro:unless value="$(arg use_nav)">
+    <xacro:if value="$(arg mujoco_plugin)">
+      <joint name="world_to_base" type="fixed">
+        <parent link="world" />
+        <child link="base_link" />
+        <origin rpy="0 0 0" xyz="0 0 0" />
+      </joint>
+    </xacro:if>
+    <xacro:unless value="$(arg mujoco_plugin)">
+      <joint name="world_to_base" type="fixed">
+        <parent link="world" />
+        <child link="base_link" />
+        <origin rpy="0 0 0" xyz="0 0 0.3" />
+      </joint>
+    </xacro:unless>
+  </xacro:unless>
+  <!-- use_nav=true: nav owns base_link; world becomes child at -0.3m Z (same offset, nav-safe) -->
+  <xacro:if value="$(arg use_nav)">
+    <joint name="base_to_world" type="fixed">
+      <parent link="base_link" />
+      <child link="world" />
+      <origin rpy="0 0 0" xyz="0 0 -0.3" />
     </joint>
   </xacro:if>
-  <xacro:unless value="$(arg mujoco_plugin)">
-    <joint name="world_to_base" type="fixed">
-      <parent link="world" />
-      <child link="base_link" />
-      <origin rpy="0 0 0" xyz="0 0 0.3" />
-    </joint>
-  </xacro:unless>
   <!-- XARM MACRO -->
   <xacro:include filename="$(find frida_description)/urdf/xarm/xarm_device_macro.xacro" />

Commit message: offset

File: robot_description/frida_description/urdf/TMR2025/FRIDA_Real.urdf.xacro (robot description, xacro)
@@ -144,5 +144,5 @@
    <!-- ZED MACRO -->
   <xacro:include filename="$(find frida_description)/urdf/zed/zed.xacro" />
-  <xacro:load_zed attach_to="zed" xyz="0.0 0 0.0" rpy="0 0 0"  mujoco_plugin="$(arg mujoco_plugin)" />
+  <xacro:load_zed attach_to="zed" xyz="-0.03 0 0.01404" rpy="0 0 0"  mujoco_plugin="$(arg mujoco_plugin)" />
   <!-- <joint name="base_footprint_joint" type="fixed">
       <origin xyz="0 0 ${base_length/2 + caster_radius*2}" rpy="0 0 0" />

File: robot_description/frida_description/urdf/zed/zed_macro.urdf.xacro (robot description, xacro)
@@ -31,5 +31,5 @@
       <xacro:property name="screw_offset_x" value="0.0" />
       <xacro:property name="screw_offset_z" value="0.0" />
-      <xacro:property name="optical_offset_x" value="-0.01" />
+      <xacro:property name="optical_offset_x" value="0.0" />
       <xacro:property name="mono" value="false" />
     </xacro:if>
@@ -49,5 +49,5 @@
       <xacro:property name="screw_offset_x" value="0.0" />
       <xacro:property name="screw_offset_z" value="0.0" />
-      <xacro:property name="optical_offset_x" value="-0.01" />
+      <xacro:property name="optical_offset_x" value="0.0" />
       <xacro:property name="mono" value="false" />
     </xacro:if>
@@ -56,7 +56,7 @@
       <xacro:property name="height" value="0.03" />
       <xacro:property name="bottom_slope" value="0.0" />
-      <xacro:property name="screw_offset_x" value="-0.01" />
-      <xacro:property name="screw_offset_z" value="0.0" />
-      <xacro:property name="optical_offset_x" value="-0.01" />
+      <xacro:property name="screw_offset_x" value="0.0" />
+      <xacro:property name="screw_offset_z" value="0.0" />
+      <xacro:property name="optical_offset_x" value="0.0" />
       <xacro:property name="mono" value="false" />
     </xacro:if>
@@ -66,6 +66,6 @@
       <xacro:property name="bottom_slope" value="0.0" />
       <xacro:property name="screw_offset_x" value="0.0" />
-      <xacro:property name="screw_offset_z" value="-0.016" />
-      <xacro:property name="optical_offset_x" value="-0.01" />
+      <xacro:property name="screw_offset_z" value="0.0" />
+      <xacro:property name="optical_offset_x" value="0.0" />
       <xacro:property name="mono" value="false" />
     </xacro:if>
@@ -75,6 +75,6 @@
       <xacro:property name="bottom_slope" value="0.0" />
       <xacro:property name="screw_offset_x" value="0.0" />
-      <xacro:property name="screw_offset_z" value="-0.016" />
-      <xacro:property name="optical_offset_x" value="-0.01" />
+      <xacro:property name="screw_offset_z" value="0.0" />
+      <xacro:property name="optical_offset_x" value="0.0" />
       <xacro:property name="mono" value="false" />
     </xacro:if>
@@ -84,5 +84,5 @@
       <xacro:property name="bottom_slope" value="0.0" />
       <xacro:property name="screw_offset_x" value="0.00" />
-      <xacro:property name="screw_offset_z" value="-0.0155" />
+      <xacro:property name="screw_offset_z" value="0.0" />
       <xacro:property name="optical_offset_x" value="0.0" />
       <xacro:property name="mono" value="false" />
@@ -93,5 +93,5 @@
       <xacro:property name="bottom_slope" value="0.0" />
       <xacro:property name="screw_offset_x" value="0.0" />
-      <xacro:property name="screw_offset_z" value="-0.0155" />
+      <xacro:property name="screw_offset_z" value="0.0" />
       <xacro:property name="optical_offset_x" value="0.0" />
       <xacro:property name="mono" value="true" />
@@ -102,5 +102,5 @@
       <xacro:property name="bottom_slope" value="0.0" />
       <xacro:property name="screw_offset_x" value="0.00" />
-      <xacro:property name="screw_offset_z" value="-0.0155" />
+      <xacro:property name="screw_offset_z" value="0.0" />
       <xacro:property name="optical_offset_x" value="0.0" />
       <xacro:property name="mono" value="true" />

Commit message: floor

File: robot_description/frida_description/urdf/TMR2025/FRIDA_Real.urdf.xacro (robot description, xacro)
@@ -100,5 +100,5 @@
       <parent link="world" />
       <child link="base_link" />
-      <origin rpy="0 0 0" xyz="0 0 0.3" />
+      <origin rpy="0 0 0" xyz="0 0 0.144" />
     </joint>
   </xacro:unless>

Commit message: not floor

File: robot_description/frida_description/urdf/TMR2025/FRIDA_Real.urdf.xacro (robot description, xacro)
@@ -100,5 +100,5 @@
       <parent link="world" />
       <child link="base_link" />
-      <origin rpy="0 0 0" xyz="0 0 0.144" />
+      <origin rpy="0 0 0" xyz="0 0 0.3" />
     </joint>
   </xacro:unless>

Commit message: original point cloud pos no offset

File: robot_description/frida_description/urdf/TMR2025/FRIDA_Real.urdf.xacro (robot description, xacro)
@@ -144,5 +144,5 @@
    <!-- ZED MACRO -->
   <xacro:include filename="$(find frida_description)/urdf/zed/zed.xacro" />
-  <xacro:load_zed attach_to="zed" xyz="-0.03 0 0.01404" rpy="0 0 0"  mujoco_plugin="$(arg mujoco_plugin)" />
+  <xacro:load_zed attach_to="zed" xyz="0 0 0" rpy="0 0 0"  mujoco_plugin="$(arg mujoco_plugin)" />
   <!-- <joint name="base_footprint_joint" type="fixed">
       <origin xyz="0 0 ${base_length/2 + caster_radius*2}" rpy="0 0 0" />

File: robot_description/frida_description/urdf/zed/zed_macro.urdf.xacro (robot description, xacro)
@@ -131,5 +131,5 @@
       <xacro:unless value="${model == 'virtual'}">
         <visual>
-          <origin xyz="${screw_offset_x} 0 ${screw_offset_z}" rpy="0 0 0"/>
+          <origin xyz="-0.03 0 0.01404" rpy="0 0 0"/>
           <geometry>
 <mesh filename="file://$(find zed_msgs)/meshes/${model}.stl"/>
@@ -138,5 +138,5 @@
         </visual>
         <collision>
-          <origin xyz="${screw_offset_x} 0 ${screw_offset_z}" rpy="0 0 0"/>
+          <origin xyz="-0.03 0 0.01404" rpy="0 0 0"/>
           <geometry>
 <mesh filename="file://$(find zed_msgs)/meshes/${model}.stl"/>
@@ -161,5 +161,5 @@
         <xacro:if value="${model == 'virtual' and not simulation}">
           <visual>
-            <origin xyz="0 0 0" rpy="0 0 0"/>
+            <origin xyz="-0.03 0 0.01404" rpy="0 0 0"/>
             <geometry>
   <mesh filename="file://$(find zed_msgs)/meshes/${model}.stl"/>
@@ -168,5 +168,5 @@
           </visual>
           <collision>
-            <origin xyz="0 0 0" rpy="0 0 0"/>
+            <origin xyz="-0.03 0 0.01404" rpy="0 0 0"/>
             <geometry>
   <mesh filename="file://$(find zed_msgs)/meshes/${model}.stl"/>
@@ -211,5 +211,5 @@
         <xacro:if value="${model == 'virtual' and not simulation}">
           <visual>
-            <origin xyz="0 0 0" rpy="0 0 0"/>
+            <origin xyz="-0.03 0 0.01404" rpy="0 0 0"/>
             <geometry>
   <mesh filename="file://$(find zed_msgs)/meshes/${model}.stl"/>
@@ -218,5 +218,5 @@
           </visual>
           <collision>
-            <origin xyz="0 0 0" rpy="0 0 0"/>
+            <origin xyz="-0.03 0 0.01404" rpy="0 0 0"/>
             <geometry>
   <mesh filename="file://$(find zed_msgs)/meshes/${model}.stl"/>

Commit message: fix error "package not found"

File: robot_description/frida_description/urdf/TMR2025/FRIDA_Real.urdf.xacro (robot description, xacro)
@@ -43,5 +43,5 @@
   <!-- ZED ARGUMENTS -->
   <!-- ROBOT COMPONENTS -->
-  <xacro:include filename="$(find home_custom_base_description)/urdf/robot.xacro"/>
+  <xacro:include filename="$(find frida_description)/urdf/TMR2025/robot_real.xacro"/>
   <!-- MUJOCO PARAMS -->
   <!-- gravcomp mirrors the xarm6 firmware's internal gravity compensation:
@@ -92,5 +92,5 @@
     <joint name="world_to_base" type="fixed">
       <parent link="world" />
-      <child link="_base_footprint" />
+      <child link="base_link" />
       <origin rpy="0 0 0" xyz="0 0 0" />
     </joint>
@@ -99,5 +99,5 @@
     <joint name="world_to_base" type="fixed">
       <parent link="world" />
-      <child link="_base_footprint" />
+      <child link="base_link" />
       <origin rpy="0 0 0" xyz="0 0 0.3" />
     </joint>

File: xacro_output.urdf (robot description, URDF)
Before this commit: robot FRIDA, 24 links, 23 joints
Links:
- removed link _base_footprint
- removed link _base_link
- removed link _lidar_front
- removed link _lidar_rear
- removed link _wheel_FL
- removed link _wheel_FR
- removed link _wheel_RL
- removed link _wheel_RR
- added link base_footprint
- added link base_link, mass 200.075; collision mesh filename=file:///home/jeremy/home2/install/frida_description/share/f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; visual mesh filename=file:///home/jeremy/home2/install/frida_description/share/f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
- added link imu_base, mass 0.096211; collision box size=0.001 0.001 0.001; visual box size=0.01 0.01 0.01
- added link intel_realsense, mass 0.048201; collision mesh filename=file:///home/jeremy/home2/install/frida_description/share/f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; visual mesh filename=file:///home/jeremy/home2/install/frida_description/share/f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
- added link laser, mass 0.096211; collision mesh filename=file:///home/jeremy/home2/install/frida_description/share/f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; visual mesh filename=file:///home/jeremy/home2/install/frida_description/share/f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
Joints:
- removed joint _base_footprint_joint
- removed joint _lidar_front_joint
- removed joint _lidar_rear_joint
- removed joint _wheel_FL_joint
- removed joint _wheel_FR_joint
- removed joint _wheel_RL_joint
- removed joint _wheel_RR_joint
- removed joint xarm_joint
- added joint base_footprint_joint: type fixed, parent base_link, child base_footprint, origin xyz=0 0 0 rpy=0 0 0 , axis 0 0 1
- added joint imu_base_joint: type fixed, parent base_link, child imu_base, origin xyz=0.15026 0 0.002 rpy=3.1416 3.1416 1.57, axis 0 0 1
- added joint intelrealsense: type fixed, parent base_link, child intel_realsense, origin xyz=0.140953490988428 0 0.428947355746093 rpy=0 0 0, axis 0 0 1
- added joint lidar: type fixed, parent base_link, child laser, origin xyz=0.16 0 0.002 rpy=0 0 3.14, axis 0 0 1
- added joint xarm_base_joint: type fixed, parent base_link, child xarm_base, origin xyz=0.036105613000001 0 0.441000000000001 rpy=0 0 1.57, axis 0 0 1
- joint world_to_base: child _base_footprint -> base_link

Commit message: done

File: robot_description/frida_description/urdf/TMR2025/FRIDA_Real.urdf.xacro (robot description, xacro)
@@ -92,5 +92,5 @@
     <joint name="world_to_base" type="fixed">
       <parent link="world" />
-      <child link="base_link" />
+      <child link="_base_footprint" />
       <origin rpy="0 0 0" xyz="0 0 0" />
     </joint>
@@ -99,5 +99,5 @@
     <joint name="world_to_base" type="fixed">
       <parent link="world" />
-      <child link="base_link" />
+      <child link="_base_footprint" />
       <origin rpy="0 0 0" xyz="0 0 0.3" />
     </joint>
