Commit message: 90

File: robot_description/frida_description/urdf/TMR2025/FRIDA_Real.urdf.xacro (robot description, xacro)
@@ -38,5 +38,5 @@
   <xacro:arg name="attach_to" default="xarm_base"/>
   <xacro:arg name="attach_xyz" default="0 0 0"/>
-  <xacro:arg name="attach_rpy" default="0 0 1.5707963267948966"/>
+  <xacro:arg name="attach_rpy" default="0 0 0"/>
   <xacro:arg name="mesh_suffix" default="stl"/>
   <xacro:arg name="kinematics_suffix" default=""/>
@@ -93,5 +93,5 @@
       <parent link="world" />
       <child link="_base_footprint" />
-      <origin rpy="0 0 0" xyz="0 0 0" />
+      <origin rpy="0 0 1.5707963267948966" xyz="0 0 0" />
     </joint>
   </xacro:if>
@@ -100,5 +100,5 @@
       <parent link="world" />
       <child link="_base_footprint" />
-      <origin rpy="0 0 0" xyz="0 0 0.3" />
+      <origin rpy="0 0 1.5707963267948966" xyz="0 0 0.3" />
     </joint>
   </xacro:unless>

File: robot_description/frida_description/urdf/omnibase/robot.xacro (robot description, xacro)
@@ -21,5 +21,5 @@
   <link name="${prefix}_base_footprint"/>
   <joint name="${prefix}_base_footprint_joint" type="fixed">
-    <origin xyz="0 0 0.0385" rpy="0 0 0"/>
+    <origin xyz="0 0 0.0385" rpy="0 0 90"/>
     <parent link="${prefix}_base_footprint"/>
     <child link="${prefix}_base_link"/>

Commit message: 2pi

File: robot_description/frida_description/urdf/TMR2025/FRIDA_Real.urdf.xacro (robot description, xacro)
@@ -38,5 +38,5 @@
   <xacro:arg name="attach_to" default="xarm_base"/>
   <xacro:arg name="attach_xyz" default="0 0 0"/>
-  <xacro:arg name="attach_rpy" default="0 0 0"/>
+  <xacro:arg name="attach_rpy" default="0 0 1.5707963267948966"/>
   <xacro:arg name="mesh_suffix" default="stl"/>
   <xacro:arg name="kinematics_suffix" default=""/>
@@ -93,5 +93,5 @@
       <parent link="world" />
       <child link="_base_footprint" />
-      <origin rpy="0 0 1.5707963267948966" xyz="0 0 0" />
+      <origin rpy="0 0 0" xyz="0 0 0" />
     </joint>
   </xacro:if>
@@ -100,5 +100,5 @@
       <parent link="world" />
       <child link="_base_footprint" />
-      <origin rpy="0 0 1.5707963267948966" xyz="0 0 0.3" />
+      <origin rpy="0 0 0" xyz="0 0 0.3" />
     </joint>
   </xacro:unless>

Commit message: prefix changes

File: robot_description/frida_description/urdf/TMR2025/FRIDA_Real.urdf.xacro (robot description, xacro)
@@ -92,5 +92,5 @@
     <joint name="world_to_base" type="fixed">
       <parent link="world" />
-      <child link="_base_footprint" />
+      <child link="base_footprint" />
       <origin rpy="0 0 0" xyz="0 0 0" />
     </joint>
@@ -99,5 +99,5 @@
     <joint name="world_to_base" type="fixed">
       <parent link="world" />
-      <child link="_base_footprint" />
+      <child link="base_footprint" />
       <origin rpy="0 0 0" xyz="0 0 0.3" />
     </joint>

File: robot_description/frida_description/urdf/omnibase/home_base_ros2_control.xacro (robot description, xacro)
@@ -1,5 +1,5 @@
 <?xml version="1.0"?>
 <robot xmlns:xacro="http://ros.org/wiki/xacro">
-  <xacro:macro name="home_base_ros2_control" params="name prefix use_sim_time"
+  <xacro:macro name="home_base_ros2_control" params="name use_sim_time"
     xmlns:gz="http://gazebosim.org/schema">
     <!-- ROS 2 Control Setup - only for Gazebo simulation -->
@@ -9,5 +9,5 @@
           <plugin>gz_ros2_control/GazeboSimSystem</plugin>
         </hardware>
-        <joint name="${prefix}_wheel_FL_joint">
+        <joint name="wheel_FL_joint">
           <command_interface name="velocity">
             <param name="min">-10</param>
@@ -17,5 +17,5 @@
           <state_interface name="position"/>
         </joint>
-        <joint name="${prefix}_wheel_FR_joint">
+        <joint name="wheel_FR_joint">
           <command_interface name="velocity">
             <param name="min">-10</param>
@@ -25,5 +25,5 @@
           <state_interface name="position"/>
         </joint>
-        <joint name="${prefix}_wheel_RL_joint">
+        <joint name="wheel_RL_joint">
           <command_interface name="velocity">
             <param name="min">-10</param>
@@ -33,5 +33,5 @@
           <state_interface name="position"/>
         </joint>
-        <joint name="${prefix}_wheel_RR_joint">
+        <joint name="wheel_RR_joint">
           <command_interface name="velocity">
             <param name="min">-10</param>
@@ -45,5 +45,5 @@
   requires a custom friction model so the vehicle can strafe left to right -->
       <!-- Wheel friction properties -->
-      <gazebo reference="${prefix}_wheel_RL">
+      <gazebo reference="wheel_RL">
         <collision>
           <surface>
@@ -58,5 +58,5 @@
         </collision>
       </gazebo>
-      <gazebo reference="${prefix}_wheel_RR">
+      <gazebo reference="wheel_RR">
         <collision>
           <surface>
@@ -71,5 +71,5 @@
         </collision>
       </gazebo>
-      <gazebo reference="${prefix}_wheel_FL">
+      <gazebo reference="wheel_FL">
         <collision>
           <surface>
@@ -84,5 +84,5 @@
         </collision>
       </gazebo>
-      <gazebo reference="${prefix}_wheel_FR">
+      <gazebo reference="wheel_FR">
         <collision>
           <surface>

File: robot_description/frida_description/urdf/omnibase/robot.xacro (robot description, xacro)
@@ -4,6 +4,4 @@
   <xacro:arg name="use_sim_time" default="false"/>
   <xacro:arg name="robot_type" default="real"/>
-  <xacro:arg name="prefix" default="home_base"/>
-  <xacro:property name="prefix" value="$(arg prefix)"/>
   <xacro:property name="use_sim_time" value="$(arg use_sim_time)"/>
   <xacro:property name="mesh_dir" value="file://$(find frida_description)/urdf/meshes/omnibase"/>
@@ -19,12 +17,12 @@
   </material>
   <!-- =================== base_footprint (root) =================== -->
-  <link name="${prefix}_base_footprint"/>
-  <joint name="${prefix}_base_footprint_joint" type="fixed">
+  <link name="base_footprint"/>
+  <joint name="base_footprint_joint" type="fixed">
     <origin xyz="0 0 0.0385" rpy="0 0 0"/>
-    <parent link="${prefix}_base_footprint"/>
-    <child link="${prefix}_base_link"/>
+    <parent link="base_footprint"/>
+    <child link="base_link"/>
   </joint>
   <!-- =================== base_link =================== -->
-  <link name="${prefix}_base_link">
+  <link name="base_link">
     <inertial>
       <origin xyz="0.0035289 4.9532E-05 0.18881" rpy="0 0 0"/>
@@ -48,5 +46,5 @@
   </link>
   <!-- =================== wheel_FL =================== -->
-  <link name="${prefix}_wheel_FL">
+  <link name="wheel_FL">
     <inertial>
       <origin xyz="-2.01760275153617E-11 -1.2648801422932E-08 -0.000225751978378957" rpy="0 0 0"/>
@@ -69,12 +67,12 @@
     </collision>
   </link>
-  <joint name="${prefix}_wheel_FL_joint" type="continuous">
+  <joint name="wheel_FL_joint" type="continuous">
     <origin xyz="0.184790699909997 0.219394995052441 0.0376959841787657" rpy="-1.5707963267949 0 0"/>
-    <parent link="${prefix}_base_link"/>
-    <child link="${prefix}_wheel_FL"/>
+    <parent link="base_link"/>
+    <child link="wheel_FL"/>
     <axis xyz="0 0 1"/>
   </joint>
   <!-- =================== wheel_FR =================== -->
-  <link name="${prefix}_wheel_FR">
+  <link name="wheel_FR">
     <inertial>
       <origin xyz="1.08346649985158E-08 2.62530414074647E-09 -0.000243946115891319" rpy="0 0 0"/>
@@ -97,12 +95,12 @@
     </collision>
   </link>
-  <joint name="${prefix}_wheel_FR_joint" type="continuous">
+  <joint name="wheel_FR_joint" type="continuous">
     <origin xyz="0.184790699909996 -0.219395004947559 0.0376959841787653" rpy="-1.5707963267949 0 0"/>
-    <parent link="${prefix}_base_link"/>
-    <child link="${prefix}_wheel_FR"/>
+    <parent link="base_link"/>
+    <child link="wheel_FR"/>
     <axis xyz="0 0 1"/>
   </joint>
   <!-- =================== wheel_RL =================== -->
-  <link name="${prefix}_wheel_RL">
+  <link name="wheel_RL">
     <inertial>
       <origin xyz="6.27955468179842E-09 -8.84368271322766E-09 -0.000243945799877326" rpy="0 0 0"/>
@@ -125,12 +123,12 @@
     </collision>
   </link>
-  <joint name="${prefix}_wheel_RL_joint" type="continuous">
+  <joint name="wheel_RL_joint" type="continuous">
     <origin xyz="-0.184790699909991 0.219394995052441 0.0376959841787652" rpy="-1.5707963267949 0 0"/>
-    <parent link="${prefix}_base_link"/>
-    <child link="${prefix}_wheel_RL"/>
+    <parent link="base_link"/>
+    <child link="wheel_RL"/>
     <axis xyz="0 0 1"/>
   </joint>
   <!-- =================== wheel_RR =================== -->
-  <link name="${prefix}_wheel_RR">
+  <link name="wheel_RR">
     <inertial>
       <origin xyz="1.54742141322828E-09 1.26432938458987E-08 -0.000225751989580358" rpy="0 0 0"/>
@@ -153,12 +151,12 @@
     </collision>
   </link>
-  <joint name="${prefix}_wheel_RR_joint" type="continuous">
+  <joint name="wheel_RR_joint" type="continuous">
     <origin xyz="-0.184790699909991 -0.219395004947559 0.0376959841787661" rpy="-1.5707963267949 0 0"/>
-    <parent link="${prefix}_base_link"/>
-    <child link="${prefix}_wheel_RR"/>
+    <parent link="base_link"/>
+    <child link="wheel_RR"/>
     <axis xyz="0 0 1"/>
   </joint>
   <!-- =================== lidar_front =================== -->
-  <link name="${prefix}_lidar_front">
+  <link name="lidar_front">
     <inertial>
       <origin xyz="-0.000159118177998852 3.36756577745678E-06 -0.00515345431268351" rpy="0 0 0"/>
@@ -181,11 +179,11 @@
     </collision>
   </link>
-  <joint name="${prefix}_lidar_front_joint" type="fixed">
+  <joint name="lidar_front_joint" type="fixed">
     <origin xyz="0.287749512711774 -0.207249957761446 0.135795984178765" rpy="0 0 -1.5707963267949"/>
-    <parent link="${prefix}_base_link"/>
-    <child link="${prefix}_lidar_front"/>
+    <parent link="base_link"/>
+    <child link="lidar_front"/>
   </joint>
   <!-- =================== lidar_rear =================== -->
-  <link name="${prefix}_lidar_rear">
+  <link name="lidar_rear">
     <inertial>
       <origin xyz="-0.000159118177998907 3.36756577740127E-06 -0.00515345431268352" rpy="0 0 0"/>
@@ -208,13 +206,13 @@
     </collision>
   </link>
-  <joint name="${prefix}_lidar_rear_joint" type="fixed">
+  <joint name="lidar_rear_joint" type="fixed">
     <origin xyz="-0.287749512711767 0.207249947866326 0.135795984178765" rpy="0 0 1.5707963267949"/>
-    <parent link="${prefix}_base_link"/>
-    <child link="${prefix}_lidar_rear"/>
+    <parent link="base_link"/>
+    <child link="lidar_rear"/>
   </joint>
   <link name="xarm_base" />
   <joint name="xarm_joint" type="fixed">
     <origin xyz="0.0410000000000036 -0.00367166302995694 0.520695984178765" rpy="0 0 0" />
-    <parent link="${prefix}_base_link" />
+    <parent link="base_link" />
     <child link="xarm_base" />
     <axis xyz="0 0 0" />
@@ -222,5 +220,5 @@
   <!-- =================== Conditionally add simulation components =================== -->
   <xacro:if value="${use_sim_time}">
-    <xacro:home_base_ros2_control name="home_base" prefix="${prefix}" use_sim_time="${use_sim_time}"/>
+    <xacro:home_base_ros2_control name="home_base" use_sim_time="${use_sim_time}"/>
     <!-- Webots driver plugin configuration -->
     <webots>

Commit message: Updated frida_real

File: robot_description/frida_description/urdf/TMR2025/FRIDA_Real.urdf.xacro (robot description, xacro)
@@ -38,10 +38,10 @@
   <xacro:arg name="attach_to" default="xarm_base"/>
   <xacro:arg name="attach_xyz" default="0 0 0"/>
-  <xacro:arg name="attach_rpy" default="0 0 1.5707963267948966"/>
+  <xacro:arg name="attach_rpy" default="0 0 0"/>
   <xacro:arg name="mesh_suffix" default="stl"/>
   <xacro:arg name="kinematics_suffix" default=""/>
   <!-- ZED ARGUMENTS -->
   <!-- ROBOT COMPONENTS -->
-  <xacro:include filename="$(find frida_description)/urdf/omnibase/robot.xacro"/>
+  <xacro:include filename="robot_real.xacro"/>
   <!-- MUJOCO PARAMS -->
   <!-- gravcomp mirrors the xarm6 firmware's internal gravity compensation:
@@ -92,5 +92,5 @@
     <joint name="world_to_base" type="fixed">
       <parent link="world" />
-      <child link="base_footprint" />
+      <child link="base_link" />
       <origin rpy="0 0 0" xyz="0 0 0" />
     </joint>
@@ -99,5 +99,5 @@
     <joint name="world_to_base" type="fixed">
       <parent link="world" />
-      <child link="base_footprint" />
+      <child link="base_link" />
       <origin rpy="0 0 0" xyz="0 0 0.3" />
     </joint>
