Commit message: chore: clean up empty code change sections in the changes log

File: robot_description/frida_description/urdf/xarm/spherized_xarm/xarm6.urdf (robot description, URDF)
Before this commit: robot xarm6_urdf, 8 links, 7 joints
Links:
- link link1: geometry collision sphere radius=0.03582; collision sphere radius=0.04113
- link link2: geometry collision sphere radius=0.03; collision sphere radius=0.03
- link link3: geometry collision sphere radius=0.02522; collision sphere radius=0.02641
- link link4: geometry collision sphere radius=0.02011; collision sphere radius=0.02061
- link link5: geometry collision sphere radius=0.03511; collision sphere radius=0.03591
- link link6: geometry collision sphere radius=0.02111; collision sphere radius=0.02111
- link link_base: geometry visual mesh filename=meshes/xarm/link_base.stl
