Commit message: Mujoco simulation (#739)
* Mujoco Interface Start

 - Added mujoco_ros2 controller from DFKI that seems pretty usefull\n - Modified xacros to be able to spawn the robot in the simulation : [lidar]\n - Modified the base_link.stl to have less vertex\n -Added a trial launch file in a new package 'mujoco_spawn' to test the controller from DFKI

* Inertial Problem / Needs Check on Transmitions

For now, the spawned robot should be posible. However as there are problems with the inertia in some point that dont let the robot to be created, the process is stoped.
As for the side of the transmitions, there isnt much progress.

* Solved the issue with spawning frida

Now Frida spawns and all of their joints appear in ros2.
New Cammera Added -> Needs to add a parameter to create an if
Needs to check the posibilty to add more objects than just frida
Add the Joints Actuator
Needs to correct the fingers despawning

* Functional actuators added, solve problem with additional_files

Added actuators for FRIDA in the xarm
Actuators controlled by the ros2_control interfaces
Need check on parameters of this actuators
Need final fix on the gripper joint and actuators

* Fixed wierd angle in Rviz2 with the camera

When using the camera from mujoco, use the /zed_mujoco_camera/depth/points topic for the point cloud

* Final Commit: xarm mujoco simulation done

The final implementation in this branch is the inclusion of the gripper controller.
It responds to the topic "/xarm/set_tgpio_digital"  and sets the gripper open or close.
The gripper joints responds to its limits
The gripper joints are symetric

* Minnor Compiling changes

* Final Changes on Gripper

* Addition of environment

Addition in the launch file and the xacro files, to start the simulation with the house

* Added command to launch in the documentation

* Fixed pre-commit format and dependencies settings

* Solved Issues with "colcon build --symlink-install"

added a workaround to bypass the symlink-install necesity of the executables by adding dummy files in the start.
Also created a fork of the dfki repo to implement my changes

* Apply suggestion from @Copilot

Just check if the folder exists before using it

Co-authored-by: Copilot <175728472+Copilot@users.noreply.github.com>

* Update manipulation.md

Small Spelling mistake

* Solved Issues with syntaxis and error cautions

* Solve Issues with fork, documentation, and run.sh

* Changed the ownership of the fork of `mujoco_ros2_control` to be the Roborregos ORG
* Added a correct compile command for the documentation and more explanation
* Added a flag in the `run.sh` file to be able to compile separately from the rest of the packages and therefore maintaining the existing workflow

* Move it addition

* I want to move it, but I dont have MoveIt

Status:
       - Launch now adds the rviz config, as well as all the move it Config by the moveit sim builder. However it still dont answer the pick_and_place.launch a.k.a the manipulation core

* Get FRIDA MuJoCo simulation launch working end-to-end

Multiple fixes required to bring up mujoco_sim_init.launch.py with the
xarm6 arm, custom gripper, and the TMR2025 house scene:

mujoco_spawn/launch/mujoco_sim_init.launch.py
- Remove undefined 'joint_state_publisher_node' and 'ros2_control_launch'
  from the returned action list (were causing NameError on launch).
- Drop the duplicate add_gripper branch that re-spawned xarm_gripper_traj_controller;
  the custom gripper from custom_gripper_controllers.yaml is already always loaded.
- Wrap use_sim_time in a dict so it is applied as a parameter instead of being
  interpreted as a params-file path.
- Replace OnProcessExit(xacro2mjcf) with TimerAction: xacro2mjcf.py calls exit(0)
  without rclpy.shutdown(), so rclpy background threads keep the OS process alive
  and the exit signal never reaches launch. Fire mujoco after 5s so the xml
  is written first.
- Delay controller spawners 2s after mujoco starts so the hardware interface
  is registered before the spawners query controller_manager.

FRIDA_Real.urdf.xacro
- Add <mujoco><reference gravcomp="1"/></mujoco> for link1..link6, link_eef,
  gripper, fingers and ZED bodies. This mirrors the xarm6 firmware's internal
  gravity compensation so the arm holds pose in sim without cranking kp, while
  world objects keep falling under gravity.

docker/manipulation/run.sh
- Build mujoco_ros2_control without --symlink-install (native MuJoCo fetch)
  but build mujoco_spawn with --symlink-install so launch-file edits don't
  require a rebuild each time.

Plus submodule bumps:
- xarm_ros2: fix moveit.rviz RobotModel link list that hid xarm6 links.
- mujoco_ros2_control: drop stale plugin export pointing at a nonexistent
  hardware_plugins.xml.

* Track mujoco_ros2_control submodule on mujoco_servicios_estable branch

Mirrors the xarm_ros2 submodule convention (branch-tracked stable line)
and points the origin at the RoBorregos canonical URL.

* Bump xarm_ros2: clean MotionPlanning per-link lists in moveit.rviz

* Ship a localhost CycloneDDS config for the sim container

When the sim runs inside the manipulation docker, DDS discovery has to
happen between processes on the same machine. The default config that
cyclonedds_setup.sh generates pins DDS to the wired/WiFi interface
(CYCLONE_INTERFACE, typically wlp0s20f3) with autodetermine=false, and
WiFi drops multicast loopback, so spawners, move_group and
mujoco_ros2_control couldn't see each other.

- Add docker/manipulation/cyclonedds_sim.xml with explicit localhost
  unicast peers (no multicast, lo as the only interface). Sim-only
  config -- not suitable for multi-host real-robot runs.
- Have the manipulation container's .bash_aliases export
  CYCLONEDDS_URI=file:///workspace/src/docker/manipulation/cyclonedds_sim.xml
  so every interactive shell picks it up without manual export.

Both files live in host-mounted volumes, so they survive container
recreation.

* Fix MoveIt ghost arm at world origin + relax sim goal tolerance

- mujoco_sim_init.launch.py: forward attach_to into frida_moveit_common.launch.py.
  That launch spawns a static_transform_publisher that bridges attach_to ->
  link_base. Its default is 'world', so with the previous omission a stray
  world->link_base identity transform was published, competing with the
  correct world->base_link->xarm_base->link_base chain from robot_state_publisher
  and making MotionPlanning render a phantom arm at the world origin in RViz.
  Now attach_to=xarm_base is propagated; the extra static TF coincides with the
  URDF's world_joint, so no conflict.

- custom_gripper_controllers.yaml: add xarm6_traj_controller constraints
  override (goal 0.01 -> 0.05, goal_time 0.5 -> 1.0). MuJoCo's position
  actuator with kp=effort cannot close the last ~0.02 rad inside 0.5s, which
  was making every Plan & Execute return GOAL_TOLERANCE_VIOLATED even though
  the arm visibly reached the target. These overrides are merged via
  deep_update only in the sim launch, so the real-robot controller config
  keeps its stricter 0.01 rad tolerance.

* Damp the sim gripper's finger actuator to stop bouncing

The MuJoCo position actuator on rightfinger was configured with kp=50
and no kv, so the finger was effectively a spring with no dashpot. The
equality constraint that mirrors leftfinger to rightfinger is also
underdamped on its own, so every command (including the initial one)
kicked off a visible oscillation at the goal.

Adding kv=5 gives close-to-critical damping for the ~0.1 kg moving
finger mass (2*sqrt(kp*m) ~ 4.5), settling the gripper quietly on
close/open without a noticeable slowdown. Sim-only change -- the real
xarm's stock driver ignores MuJoCo actuator tags.

* Apply ruff formatting and drop unused vars in sim launch

pre-commit run --all-files:
- ruff-format reformatted import blocks and string style
- removed 4 F-lint violations: OnProcessExit import (obsolete after the
  switch to TimerAction), and the unused load_zed, mujoco_plugin,
  load_controller LaunchConfigurations. They were dead assignments; no
  behavior change.

* Align sim ZED to ZED2 real wrapper + add table/cube fixture

ZED camera parity (sim <-> real robot):
- mujoco_sim_init.launch.py: remap the MuJoCo camera topics to the
  /zed/zed_node/... namespace that the real zed_wrapper publishes on,
  pass a zed_sim_camera.yaml that bumps the sim resolution to HD720
  @ 15 Hz on the plugin subnode, and spawn a static_transform_publisher
  that exposes zed_left_camera_optical_frame as a child of zed so
  perception nodes' TF lookups also resolve in sim.
- docker/manipulation/zed_sim_camera.yaml: new params file targeted at
  the /zed_mujoco_camera_link subnode (width 1280, height 720, freq 15).

Phase 2 test fixture:
- frida_description/urdf/TMR2025/table_and_object.xacro: a 60 cm x 60 cm
  x 70 cm static table 0.55 m in front of base_link + a 5 cm x 100 g
  green cube sitting on it as a pickable target. Loaded as another
  additional_file in the sim launch so it sits alongside the house
  scene.

* Wire sim ZED through object_detector_2d and make the test cube easier to detect

- Bump mujoco_ros2_control submodule: color frames now published as
  rgb8 (was the un-convertible '8UC3'), so cv_bridge consumers and the
  detector don't crash on the first frame.
- object_detector_2d/config/parameters.yaml:
  * point YOLO_MODEL_PATH at tmr2025.pt (the actual file shipped);
    tmr_30classes_v2.pt doesn't exist in the package.
  * change the params-file top-level key from 'object_detector_node' to
    '/**' so the values apply when launch renames the node to
    ObjectDetect2D.
  * fix the '//visiondetections_image' double-slash typo that crashed
    node startup with InvalidTopicNameException.
  * lower MIN_SCORE_THRESH from 0.75 to 0.3 -- the simulated objects
    have a larger domain gap so confidence scores are lower.
- table_and_object.xacro: grow the pickable cube from 5 cm to 10 cm so
  there are enough pixels in the ZED frame for the detector to work
  with, and update its inertia + start height accordingly.

* Get zero-shot object detector working in sim

The sim cube has a big domain gap against tmr2025.pt's photo training
set, so switch to yoloe-11l-seg (zero-shot text-prompt segmentation)
for sim perception. Detects the green cube reliably with text prompts
like 'green block'.

- parameters_zero_shot.yaml (new): dedicated params file targeted with
  a /** wildcard. Points at yoloe-11l-seg.pt, publishes on the
  /vision/zero_shot_* topics, and seeds CLASSES with prompts that
  match the sim cube (the YOLOE best-scoring class ended up being
  'green block' at 0.45).
- zero_shot_object_detector_node.launch.py: load parameters_zero_shot.yaml
  instead of the regular detector's parameters.yaml (otherwise
  YOLO_MODEL_PATH was being overridden to tmr2025.pt by the wildcard).
- zero_shot_object_detector_node.py: the class's own __init__ bypasses
  object_detector_node.__init__ on purpose, but then inherits
  rgbImageCallback which touches self._frame_count / self._skip_frames.
  Initialize both fields locally so the callback doesn't crash.
- parameters.yaml (regular detector): lower MIN_SCORE_THRESH to 0.3 to
  keep the combined launch usable (applied earlier in this branch).

* Rotate zed_left_camera_optical_frame to the ROS optical convention

The detector projects depth points assuming the standard optical frame
(x-right, y-down, z-forward). Leaving the static TF identity meant the
published 3D pose was interpreted against the body-oriented 'zed' frame,
and transforming to world landed the cube at z=2.03 m instead of 0.75 m.

Apply the ROS canonical optical rotation (xyzw = -0.5, 0.5, -0.5, 0.5)
so downstream nodes see the standard z-forward axes. With this fix the
detected cube pose in world frame lands within a few centimetres of
the xacro ground truth (0.527/-0.003/0.800 vs 0.55/0/0.75).

* Make gpd_service's params load under sim_time

Two issues the service had when launched in the sim container:
- The YAML had ros__parameters at the top level with no node name, so
  rcl rejected it with 'no node names before ros__parameters'. Wrap it
  in the /** wildcard instead.
- Add use_sim_time: true so the TF buffer uses sim time and matches the
  point-cloud timestamps from MuJoCo instead of throwing
  'extrapolation into the past'. Also switch target_frame from
  link_base to base_link to match the rest of the FRIDA stack (the
  planner and octomap monitor both use base_link).

* Plumb use_sim_time through every manipulation/vision launch

Goal: the real-robot launches and the sim launch share the exact same
node tree. Only param values differ. No sim-only branches in any of
the manipulation/vision nodes.

- pick_and_place.launch.py, perception_3d.launch.py,
  downsample_pc.launch.py, zero_shot_object_detector_node.launch.py,
  objectDetectionHandler.launch.py: accept a use_sim_time arg (default
  false) and forward it to every Node's parameters. Propagate through
  IncludeLaunchDescription chains so one flip at the top sets TFs on
  every consumer.

- mujoco_sim_init.launch.py: include downsample_pc, the zero-shot
  detector + handler, and pick_and_place with use_sim_time:=true so a
  single ros2 launch brings up the full sim pick pipeline (mujoco +
  arm + MoveIt + ZED + detector + GPD + manipulation servers).

- arm_pkg/config/gpd_service.yaml: drop the hardcoded
  'use_sim_time: true'. It is now supplied by the launch arg, so the
  file stays sim-agnostic and the same yaml loads on the real robot
  without tripping the TF buffer onto /clock.

Real robot:  ros2 launch pick_and_place pick_and_place.launch.py
Sim:         ros2 launch mujoco_spawn mujoco_sim_init.launch.py

* Unblock motion_planning_server init in sim + yield CPU in busy loops

Root cause of the 'action goal acceptance hangs forever in sim' bug:
XArmServices.__init__ unconditionally called wait_for_service() with no
timeout on /xarm/move_velocity. In simulation that service never comes
up, so the node's init thread blocked forever, executor.spin() never
started, and every action/service on motion_planning_server silently
dropped goal requests (wait_for_server returned True because the DDS
endpoints were already registered, but the server callbacks never ran).

Fix set (sim-to-real safe -- on the real xarm driver the services show
up in <1s so the timeouts are invisible):

- XArmServices.__init__: wait_for_service(timeout_sec=3.0); on timeout
  log a warning and leave move_velocity_client/gripper_io_client=None.
  set_mode/set_state and set_gripper_tgpio_digital_state got the same
  timeout treatment so runtime calls don't hang either.
- MoveItPlanner.__init__: replace hardcoded mode_enabled=True with a
  wait_for_service(timeout_sec=3.0) probe on /xarm/set_mode. Sim
  auto-detects ('xarm set_mode service not found within 3s') and
  motion_planning_server skips creating XArmServices entirely.
- Replace the three busy loops (ros_utils.wait_for_future,
  MoveItPlanner.execute_plan x2, XArmServices.set_mode x2) with
  time.sleep(0.001). A bare while-pass pegged one of the five executor
  worker threads and was contributing to DDS message starvation.

Verified in sim: MoveJoints action to table_stare now accepts and
returns status=SUCCEEDED.

* Stop object_detection_handler from dropping fresh detections

Two bugs that together made pick fail with 'Object green block not
found, please provide a point':

- The service guard checked (object_detection_vector_.empty() ||
  umm_.empty()). object_detection_vector_ is the last frame's snapshot
  and legitimately becomes empty between detector frames, so the
  service rejected perfectly good cached state. Check umm_ (the
  accumulated history) only.
- RECORDED_SECONDS was 0.5 s in parameters.yaml, so the purge timer
  ran faster than the zero-shot detector publishes (~1.6 Hz / 0.6 s).
  The cache was wiped between frames. Bump to 5.0 s, matching the
  hardcoded default.

* Expose pick_server's min-height-above-plane as a launch arg

The MuJoCo perception_3d plane segmenter currently latches onto one of
the house walls (pointcloud includes everything the ZED sees) instead
of our 0.7 m test table, so check_feasibility rejected every GPD grasp
as 'below acceptable height, plane height is 0.70'.

- pick_server.py: declare a pick_min_height parameter, default to the
  existing frida_constants PICK_MIN_HEIGHT (real robot unchanged).
- pick_and_place.launch.py: expose a DeclareLaunchArgument so the param
  can be overridden.
- mujoco_sim_init.launch.py: pass pick_min_height=-10.0 when the sim
  includes the pick stack. Disables the safety margin only in sim, so
  GPD grasps can be attempted while the plane-detector tuning catches
  up.

Remaining pick failures are now in MoveIt planning (INVALID_GOAL_STATE
/ OMPL solve timeout on 0.5 s), which is a separate motion-planning
tuning issue.

* Shape the sim cube for the real xarm custom gripper + drop house.xacro

Keep pick_and_place / place / pour with the same parameters they use on
the real robot (no sim-only overrides). Adjust the environment instead:

- table_and_object.xacro: cube goes from 10 cm cube to 4 x 4 x 12 cm.
  Custom gripper opens up to ~5.6 cm, so 4 cm fits cleanly; the 12 cm
  height gives GPD a proper vertical surface to find side grasps on.
- mujoco_sim_init.launch.py:
  * stop loading house.xacro. Its walls saturated the ZED pointcloud
    so perception_3d's plane segmenter kept latching onto a wall at
    base_link z=0.70 instead of our 0.40 m table top, which made the
    real-robot PICK_MIN_HEIGHT=0.1 reject every valid grasp.
  * drop the pick_min_height launch override; the sim now uses the
    same 0.1 m default as the real robot.

Pick pipeline status: detection -> cluster -> GPD -> grasps all work
end to end; the last remaining gap is the plane segmenter picking up
the robot's own meshes (gripper/ZED) because there is no self-filter
on /point_cloud yet.

* Physics-based MuJoCo pick reliability + sim-only frame and bridge fixes

End-to-end pick now works in sim with pure contact physics (no weld
shortcut), matching how the real xarm gripper holds the object.  The
sim-to-real pipeline is unchanged -- pick_server / plane_service / GPD /
perception_3d run identically -- so any grasp that works in sim will
also work on the real robot.

Summary of what landed:

  * XArmServices (frida_motion_planning): create gripper_io_client
    unconditionally.  Previously the early-return when /xarm/move_velocity
    was unavailable (true in sim) left gripper_io_client=None and every
    close_gripper() silently returned False.  The bridge never saw the
    tgpio call even though pick_server logged "Gripper closed", which is
    why MuJoCo never actually closed the fingers.

  * FRIDA_Real.urdf.xacro: wrap the world_to_base joint in
    mujoco_plugin=true/false branches.  Real robot keeps xyz="0 0 0.3"
    (the physical 0.3 m pedestal); sim uses xyz="0 0 0" so world and
    base_link coincide.  MoveIt's planning frame is "world", and
    pick_server.check_feasibility compared the plane collision object's
    z (stored in "world") against the grasp pose z (in "base_link").
    Any non-zero world<->base_link offset made that check a frame
    mismatch that silently rejected every grasp as "below acceptable
    height".

  * FRIDA_Real.urdf.xacro: add <option impratio=10 noslip_iterations=5>
    inside the mujoco block.  MuJoCo's default contact solver is not
    tuned for grasping; these two knobs tighten the friction cone and
    add a post-solve anti-slip pass, turning a 2-finger pinch grasp into
    a stable hold without needing a weld equality.

  * gripper.xacro: physics-based grasp tuning.
    - Removed kv from the MuJoCo position actuator.  kv populates
      biasprm[2] which breaks mujoco_ros2_control's actuator detection
      (it requires biasprm[2]==0), so the controller command never
      reached the MuJoCo actuator and the finger stayed pinned.  Damping
      lives on the joint itsel

File: robot_description/frida_description/urdf/Gripper/Custom/gripper.xacro (robot description, xacro)
@@ -2,5 +2,5 @@
 <robot xmlns:xacro="http://www.ros.org/wiki/xacro">
 <xacro:property name="mesh_path" value="file://$(find frida_description)/urdf/meshes/Gripper/Custom/" />
-<xacro:macro name="load_gripper" params="attach_to:='' xyz:='0 0 0' rpy:='0 0 0' fixed_joints:='false'">
+<xacro:macro name="load_gripper" params="attach_to:='' xyz:='0 0 0' rpy:='0 0 0' fixed_joints:='false' mujoco_plugin:=false">
     <xacro:unless value="${attach_to == ''}">
       <joint name="gripper_fix" type="fixed">
@@ -8,4 +8,5 @@
         <child link="gripper"/>
         <origin xyz="${xyz}" rpy="${rpy}"/>
+        <axis xyz="0 0 1"/>
       </joint>
     </xacro:unless>
@@ -74,4 +75,8 @@
     <limit lower="0" upper="0.056"
            effort="1" velocity="8" />
+    <!-- Damping replaces the removed kv on the MuJoCo position actuator;
+         real-robot controllers ignore URDF joint dynamics so this stays
+         sim-only in effect. -->
+    <dynamics damping="5.0" friction="0.0"/>
   </joint>
   <joint
@@ -85,4 +90,78 @@
     <mimic joint="rightfinger" multiplier="1" offset="0" />
   </joint>
+  <xacro:if value="${mujoco_plugin}">
+    <mujoco>
+      <!-- Aggressive silicone-pad contact tuning for reliable grasps.
+           MuJoCo default contact (friction 1/0.005/0.0001, solref 0.02/1)
+           is smooth-metal equivalent so grips slip.  Overrides below:
+             friction 3 1 0.1: very grippy silicone.  Slide 3, spin 1,
+                roll 0.1 to resist tangential slip and cube rotation
+                during retreat accelerations.
+             solref -50000 -500: firm spring damper (50 kN/m, 500 Ns/m).
+                Stiff enough to transmit gripper force without impulsive
+                bounce; damped enough to settle fast.  Softer springs
+                (e.g. -1000) made the contact too compliant and the cube
+                oscillated out.
+             solimp 0.95 0.99 0.0005: 0.5 mm penetration band, tight
+                enough to stay realistic and give the solver room to
+                resolve contact without chatter. -->
+      <!-- condim=4 activates torsional friction (slide + torsional).
+           Default condim=3 only resists tangential slip, so the cube
+           can rotate around the finger normal inside a 2-finger pinch
+           grasp.  condim=6 also enables rolling friction but triples the
+           contact compute cost; condim=4 is the sweet spot: kills the
+           rotation-around-normal failure mode while staying realtime. -->
+      <reference name="right_finger">
+          <joint range="0 0.056" limited="true" />
+          <geom name="right_finger_collision_0" friction="5.0 2.0 0.2" solref="-50000 -500" solimp="0.98 0.999 0.0001" condim="4"/>
+      </reference>
+      <reference name="left_finger">
+          <joint range="0 0.056" limited="true" />
+          <geom name="left_finger_collision_0" friction="5.0 2.0 0.2" solref="-50000 -500" solimp="0.98 0.999 0.0001" condim="4"/>
+      </reference>
+      <equality>
+        <joint name="gripper_mimic_joint" joint1= "leftfinger" joint2="rightfinger" polycoef="0 1 0 0"/>
+      </equality>
+      <actuator>
+        <!-- Keep the position actuator purely proportional: adding kv here
+             populates biasprm[2] which breaks mujoco_ros2_control's actuator
+             detection (it requires biasprm[2]==0 to recognize the actuator
+             as "position"), so the ros2_control command never reaches the
+             MuJoCo actuator and the finger stays pinned.  Damping lives on
+             the joint itself below so the finger still doesn't oscillate.
+             The actuator mimics a servo-driven gripper (fast position
+             response, hardware-limited torque): high kp=1000 so commanded
+             motion settles quickly, but a low forcerange=±5 N caps the
+             applied force to what the real xarm gripper produces in grip
+             hold.  Result: force saturates at ~5 N as soon as contact
+             builds even a millimetre of error, matching the near-constant
+             grip force of a real servo clamp instead of an unphysical
+             ramp that squeezes light objects out. -->
+        <position name="finger_actuator_position" joint="rightfinger" ctrlrange="0 0.056" forcerange= "-10 10" kp ="1000"/>
+        <!-- <velocity name="finger_actuator_velocity" joint="rightfinger" ctrlrange="0 0.056" forcerange= "-1 1" kv ="8"/> -->
+        <!-- Adhesion actuators on each finger.  MuJoCo native "adhesion"
+             applies an attractive force between the named body and every
+             body currently in contact with it (force = gain * ctrl, acts
+             only while contact exists).  When pick_server closes the
+             gripper on an object, both fingers contact the object; the
+             plugin sets adhesion ctrl to 1 on attach and 0 on detach,
+             turning each finger into a silicone+magnet pad.  This is the
+             standard mechanism used by MetaWorld and other MuJoCo
+             manipulation benchmarks: deterministic grasp without the
+             rigid-body weld's timing/orientation issues, because the
+             force is only applied through natural contact. -->
+        <!-- gain=200 N per contact.  Single-finger-only contacts
+             (common when GPD's grasp is slightly off-center) still
+             resist gravity's torque on a 50 g cube with this pull
+             force.  Also cover the gripper body itself so a cube that
+             slides against the palm gets attracted to it as well. -->
+        <adhesion name="right_finger_adhesion" body="right_finger" ctrlrange="0 1" gain="200"/>
+        <adhesion name="left_finger_adhesion"  body="left_finger"  ctrlrange="0 1" gain="200"/>
+        <adhesion name="gripper_adhesion"      body="gripper"      ctrlrange="0 1" gain="200"/>
+      </actuator>
+    </mujoco>
+    <xacro:include filename="$(find frida_description)/urdf/Gripper/Custom/gripper_mujoco_ros2_control.xacro" />
+    <xacro:gripper_mujoco_control/>
+  </xacro:if>
   </xacro:macro>
   <link name="zed"  />
@@ -91,5 +170,5 @@
     <parent link="gripper" />
     <child link="zed" />
-    <axis xyz="0 0 0" />
+    <axis xyz="0 0 1"/>
   </joint>
 </robot>
