Commit message: new params, adjust zed position

File: robot_description/frida_description/urdf/Gripper/Custom/gripper.xacro (robot description, xacro)
@@ -88,5 +88,5 @@
   <link name="zed"  />
   <joint name="ZED" type="fixed">
-    <origin xyz="0 -0.065626 -0.016728" rpy="0 -0.7854 -1.5708" />
+    <origin xyz="0 -0.095626 -0.005" rpy="0 -0.7854 -1.5708" />
     <parent link="gripper" />
     <child link="zed" />

File: robot_description/frida_description/urdf/TMR2025/FRIDA_Real.urdf.xacro (robot description, xacro)
@@ -77,5 +77,5 @@
    <!-- ZED MACRO -->
   <xacro:include filename="$(find frida_description)/urdf/zed/zed.xacro" />
-  <xacro:load_zed attach_to="zed" xyz="0.015 0 -0.0250" rpy="0 0 0" />
+  <xacro:load_zed attach_to="zed" xyz="0.0 0 0.0" rpy="0 0 0" />
   <!-- <joint name="base_footprint_joint" type="fixed">
       <origin xyz="0 0 ${base_length/2 + caster_radius*2}" rpy="0 0 0" />

Commit message: .

File: robot_description/frida_description/urdf/Gripper/Custom/gripper.xacro (robot description, xacro)
@@ -72,5 +72,5 @@
     <child link="right_finger" />
     <axis xyz="1 0 0" />
-    <limit lower="0" upper="0.056"
+    <limit lower="-0.7" upper="0.7"
            effort="1" velocity="8" />
   </joint>

Commit message: Solved the issue with spawning frida
Now Frida spawns and all of their joints appear in ros2.
New Cammera Added -> Needs to add a parameter to create an if
Needs to check the posibilty to add more objects than just frida
Add the Joints Actuator
Needs to correct the fingers despawning

File: robot_description/frida_description/urdf/Gripper/Custom/gripper.xacro (robot description, xacro)
@@ -8,4 +8,5 @@
         <child link="gripper"/>
         <origin xyz="${xyz}" rpy="${rpy}"/>
+        <axis xyz="0 0 1"/>
       </joint>
     </xacro:unless>
@@ -91,5 +92,5 @@
     <parent link="gripper" />
     <child link="zed" />
-    <axis xyz="0 0 0" />
+    <axis xyz="0 0 1"/>
   </joint>
 </robot>

File: robot_description/frida_description/urdf/RoboCup2024/base.xacro (robot description, xacro)
@@ -29,4 +29,5 @@
     <child link="base_footprint"/>
     <origin xyz="0 0 0" rpy="0 0 0 "/>
+    <axis xyz="0 0 1"/>
   </joint>
   <link name="xarm_base" />
@@ -35,4 +36,5 @@
     <parent link="base_link" />
     <child link="xarm_base" />
+    <axis xyz="0 0 1"/>
   </joint>
 </robot>

File: robot_description/frida_description/urdf/RoboCup2024/castwheel.xacro (robot description, xacro)
@@ -8,4 +8,5 @@
         <child link="caster_wheel_left"/>
         <origin xyz="0.11 0.1 -0.09"/>
+        <axis xyz="0 0 1"/>
     </joint>
     <link name="caster_wheel_left">
@@ -33,4 +34,5 @@
         <child link="caster_wheel_right"/>
         <origin xyz="0.11 -0.1 -0.09"/>
+        <axis xyz="0 0 1"/>
     </joint>
     <link name="caster_wheel_right">

File: robot_description/frida_description/urdf/RoboCup2024/imu.xacro (robot description, xacro)
@@ -11,4 +11,5 @@
     <mass value="0.01"/> <!-- Adjust mass -->
     <inertia ixx="0.00001" ixy="0.0" ixz="0.0" iyy="0.00001" iyz="0.0" izz="0.00001"/>
+    <origin xyz="0 0 0" rpy="0 0 0"></origin>
   </inertial>
 </link>
@@ -16,5 +17,6 @@
   <parent link="base_link"/>
   <child link="imu_link"/>
-  <origin xyz="0 0 0.0" rpy="0 0 0"/> <!-- Adjust position and orientation -->
+  <origin xyz="0 0 0.0" rpy="0 0 0"/>
+  <axis xyz="0 0 1"/>
 </joint>
   <gazebo reference="imu_link">

File: robot_description/frida_description/urdf/TMR2025/FRIDA.urdf.xacro (robot description, xacro)
@@ -17,4 +17,5 @@
   <xacro:arg name="ros2_control_plugin" default="uf_robot_hardware/UFRobotSystemHardware"/>
   <xacro:arg name="ros2_control_params" default=""/>
+  <xacro:arg name="mujoco_plugin" default="false"/>
   <xacro:arg name="add_realsense_d435i" default="false"/>
   <xacro:arg name="add_d435i_links" default="true"/>
@@ -49,4 +50,5 @@
     add_bio_gripper="$(arg add_bio_gripper)" dof="$(arg dof)"
     ros2_control_plugin="$(arg ros2_control_plugin)" robot_type="$(arg robot_type)"
+    mujoco_plugin="$(arg mujoco_plugin)"
     load_gazebo_plugin="true" ros2_control_params="$(arg ros2_control_params)"
     add_realsense_d435i="$(arg add_realsense_d435i)"
@@ -63,13 +65,20 @@
     model1300="$(arg model1300)" attach_to="$(arg attach_to)" attach_xyz="$(arg attach_xyz)" attach_rpy="$(arg attach_rpy)"
     robot_sn="$(arg robot_sn)" use_gazebo_camera="$(arg use_gazebo_camera)" mesh_suffix="$(arg mesh_suffix)" kinematics_suffix="$(arg kinematics_suffix)" />
-    <joint name="gripper_grasp_joint" type="fixed">
+        <!-- Mujoco Config -->
+    <xacro:if value="$(arg mujoco_plugin)">
+      <mujoco>
+        <compiler angle="radian" />
+      </mujoco>
+    </xacro:if>
+<joint name="gripper_grasp_joint" type="fixed">
       <parent link="link_eef"/>
       <child link="gripper_grasp_frame"/>
       <origin xyz="0 0 0" rpy="0 0 -0.7854"/>
+      <axis xyz="0 0 1"/>
     </joint>
     <link name="gripper_grasp_frame"> </link>
     <xacro:if value="$(arg load_zed)">
       <xacro:include filename="$(find frida_description)/urdf/Gripper/Custom/gripper.xacro" />
-      <xacro:load_gripper attach_to="link_eef" xyz="0 0 0.046" rpy="0 0 3.926" fixed_joints="true"/>
+      <xacro:load_gripper attach_to="link_eef" xyz="0 0 0.046" rpy="0 0 3.926" fixed_joints="false"/>
       <!-- ZED MACRO -->
       <xacro:include filename="$(find frida_description)/urdf/zed/zed_macro.urdf.xacro" />

File: robot_description/frida_description/urdf/TMR2025/base.xacro (robot description, xacro)
@@ -29,4 +29,5 @@
     <child link="base_footprint"/>
     <origin xyz="0 0 0" rpy="0 0 0 "/>
+    <axis xyz="0 0 1"/>
   </joint>
   <link name="xarm_base" />
@@ -35,4 +36,5 @@
     <parent link="base_link" />
     <child link="xarm_base" />
+    <axis xyz="0 0 1"/>
   </joint>
 </robot>

File: robot_description/frida_description/urdf/TMR2025/lidar.xacro (robot description, xacro)
@@ -28,5 +28,5 @@
     <parent link="base_link" />
     <child link="laser" />
-    <axis xyz="0 0 0" />
+    <axis xyz="0 0 1"/>
   </joint>
 <link name="imu_base">
@@ -57,5 +57,5 @@
     <parent link="base_link" />
     <child link="imu_base" />
-    <axis xyz="0 0 0" />
+    <axis xyz="0 0 1"/>
   </joint>
 </robot>

File: robot_description/frida_description/urdf/TMR2025/realsense.xacro (robot description, xacro)
@@ -28,5 +28,5 @@
     <parent link="base_link" />
     <child link="intel_realsense" />
-    <axis xyz="0 0 0" />
+    <axis xyz="0 0 1"/>
   </joint>
 </robot>

File: robot_description/frida_description/urdf/xarm/xarm_device_macro.xacro (robot description, xacro)
@@ -42,4 +42,5 @@
     mesh_suffix:='stl'
     kinematics_suffix:=''
+    mujoco_plugin:=true
     "
     >
@@ -65,12 +66,15 @@
     <xacro:property name="model_num" value="${scope_parent_model_num}"/>
     <!-- add one world link if no 'attach_to' specified  -->
-    <xacro:if value="${attach_to == 'world' and create_attach_link}">
-      <link name="world" />
-    </xacro:if>
-    <joint name="${prefix}world_joint" type="fixed">
-      <parent link="${attach_to}" />
-      <child link="${prefix}link_base" />
-      <origin xyz="${attach_xyz}" rpy="${attach_rpy}" />
-    </joint>
+    <xacro:if value = "${create_attach_link}">
+      <xacro:if value="${attach_to == 'world'}">
+        <link name="world" />
+      </xacro:if>
+      <joint name="${prefix}world_joint" type="fixed">
+        <parent link="${attach_to}" />
+        <child link="${prefix}link_base" />
+        <origin xyz="${attach_xyz}" rpy="${attach_rpy}" />
+        <axis xyz="0 0 1"/>
+      </joint>
+    </xacro:if>
     <xacro:if value="${effort_control}">
       <xacro:property name="hard_interface" value="EffortJointInterface" />
@@ -217,4 +221,5 @@
       <parent link="${prefix}link${dof}" />
       <child link="${prefix}link_eef" />
+      <axis xyz="0 0 1"/>
     </joint>
     <xacro:if value="${add_gripper}">

File: robot_description/frida_description/urdf/zed/zed_macro.urdf.xacro (robot description, xacro)
@@ -107,5 +107,11 @@
     </xacro:if>
     <!-- Camera mounting point (the threaded screw hole in the bottom) -->
-    <link name="${name}_camera_link" />
+    <link name="${name}_camera_link" >
+      <inertial>
+        <origin xyz="0 0 0" rpy="0 0 0" />
+        <mass value="0.001"/>
+        <inertia ixx="0.000001" ixy="0" ixz="0" iyy="0.000001" iyz="0" izz="0.000001"/>
+      </inertial>
+    </link>
     <xacro:unless value="${attach_to == ''}">
       <joint name="zed_attach_joint" type="fixed">
@@ -113,8 +119,14 @@
         <child link="${name}_camera_link"/>
         <origin xyz="${xyz}" rpy="${rpy}"/>
+        <axis xyz="0 0 1"/>
       </joint>
     </xacro:unless>
     <!-- Camera Center -->
     <link name="${name}_camera_center">
+      <inertial>
+        <origin xyz="0 0 0" rpy="0 0 0" />
+        <mass value="0.001"/>
+        <inertia ixx="0.000001" ixy="0" ixz="0" iyy="0.000001" iyz="0" izz="0.000001"/>
+      </inertial>
       <xacro:unless value="${model == 'virtual'}">
         <visual>
@@ -137,8 +149,14 @@
       <child link="${name}_camera_center"/>
       <origin xyz="0 0 ${height/2}" rpy="0 ${bottom_slope} 0" />
+      <axis xyz="0 0 1"/>
     </joint>
     <xacro:unless value="${mono}">
       <!-- Left Camera -->
       <link name="${name}_left_camera_frame">
+        <inertial>
+          <origin xyz="0 0 0" rpy="0 0 0" />
+          <mass value="0.001"/>
+          <inertia ixx="0.000001" ixy="0" ixz="0" iyy="0.000001" iyz="0" izz="0.000001"/>
+        </inertial>
         <xacro:if value="${model == 'virtual'}">
           <visual>
@@ -157,12 +175,25 @@
         </xacro:if>
       </link>
+      <mujoco>
+        <reference name="${name}_left_camera_frame">
+          <camera name="${name}_left_camera" mode="fixed" fovy="45" quat="0.5 0.5 -0.5 -0.5"/>
+        </reference>
+      </mujoco>
       <joint name="${name}_left_camera_joint" type="fixed">
         <parent link="${name}_camera_center"/>
         <child link="${name}_left_camera_frame"/>
         <origin xyz="${optical_offset_x} ${baseline/2} 0" rpy="0 0 0" />
-      </joint>
-      <link name="${name}_left_camera_optical_frame"/>
+        <axis xyz="0 0 1"/>
+      </joint>
+      <link name="${name}_left_camera_optical_frame">
+      <inertial>
+        <origin xyz="0 0 0" rpy="0 0 0" />
+        <mass value="0.001"/>
+        <inertia ixx="0.000001" ixy="0" ixz="0" iyy="0.000001" iyz="0" izz="0.000001"/>
+      </inertial>
+      </link>
       <joint name="${name}_left_camera_optical_joint" type="fixed">
         <origin xyz="0 0 0" rpy="-${M_PI/2} 0.0 -${M_PI/2}"/>
+        <axis xyz="0 0 1"/>
         <parent link="${name}_left_camera_frame"/>
         <child link="${name}_left_camera_optical_frame"/>
@@ -170,4 +201,9 @@
       <!-- Right Camera -->
       <link name="${name}_right_camera_frame">
+        <inertial>
+          <origin xyz="0 0 0" rpy="0 0 0" />
+          <mass value="0.001"/>
+          <inertia ixx="0.000001" ixy="0" ixz="0" iyy="0.000001" iyz="0" izz="0.000001"/>
+        </inertial>
         <xacro:if value="${model == 'virtual'}">
           <visual>
@@ -190,8 +226,16 @@
         <child link="${name}_right_camera_frame"/>
         <origin xyz="${optical_offset_x} -${baseline/2} 0" rpy="0 0 0" />
-      </joint>
-      <link name="${name}_right_camera_optical_frame"/>
+        <axis xyz="0 0 1"/>
+      </joint>
+      <link name="${name}_right_camera_optical_frame">
+      <inertial>
+        <origin xyz="0 0 0" rpy="0 0 0" />
+        <mass value="0.001"/>
+        <inertia ixx="0.000001" ixy="0" ixz="0" iyy="0.000001" iyz="0" izz="0.000001"/>
+      </inertial>
+      </link>
       <joint name="${name}_right_camera_optical_joint" type="fixed">
         <origin xyz="0 0 0" rpy="-${M_PI/2} 0.0 -${M_PI/2}"/>
+        <axis xyz="0 0 1"/>
         <parent link="${name}_right_camera_frame"/>
         <child link="${name}_right_camera_optical_frame"/>
@@ -199,41 +243,83 @@
       <!-- ZED2 Sensors -->
       <xacro:if value="${model == 'zed2'}">
-        <link name="${name}_mag_link" />
+        <link name="${name}_mag_link">
+          <inertial>
+            <origin xyz="0 0 0" rpy="0 0 0" />
+            <mass value="0.001"/>
+            <inertia ixx="0.000001" ixy="0" ixz="0" iyy="0.000001" iyz="0" izz="0.000001"/>
+          </inertial>
+        </link>
         <joint name="${name}_mag_joint" type="fixed">
           <parent link="${name}_camera_center"/>
           <child link="${name}_mag_link"/>
-          <origin xyz="0 0 0" rpy="0 0 0" />
-        </joint>
-        <link name="${name}_baro_link" />
+<origin xyz="0 0 0" rpy="0 0 0" />
+        <axis xyz="0 0 1"/>
+      </joint>
+        <link name="${name}_baro_link">
+          <inertial>
+            <origin xyz="0 0 0" rpy="0 0 0" />
+            <mass value="0.001"/>
+            <inertia ixx="0.000001" ixy="0" ixz="0" iyy="0.000001" iyz="0" izz="0.000001"/>
+          </inertial>
+        </link>
         <joint name="${name}_baro_joint" type="fixed">
           <parent link="${name}_camera_center"/>
           <child link="${name}_baro_link"/>
-          <origin xyz="0 0 0" rpy="0 0 0" />
-        </joint>
-        <link name="${name}_temp_left_link" />
+<origin xyz="0 0 0" rpy="0 0 0" />
+        <axis xyz="0 0 1"/>
+      </joint>
+        <link name="${name}_temp_left_link">
+          <inertial>
+            <origin xyz="0 0 0" rpy="0 0 0" />
+            <mass value="0.001"/>
+            <inertia ixx="0.000001" ixy="0" ixz="0" iyy="0.000001" iyz="0" izz="0.000001"/>
+          </inertial>
+        </link>
         <joint name="${name}_temp_left_joint" type="fixed">
           <parent link="${name}_left_camera_frame"/>
           <child link="${name}_temp_left_link"/>
-          <origin xyz="0 0 0" rpy="0 0 0" />
-        </joint>
-        <link name="${name}_temp_right_link" />
+<origin xyz="0 0 0" rpy="0 0 0" />
+        <axis xyz="0 0 1"/>
+      </joint>
+        <link name="${name}_temp_right_link">
+          <inertial>
+            <origin xyz="0 0 0" rpy="0 0 0" />
+            <mass value="0.001"/>
+            <inertia ixx="0.000001" ixy="0" ixz="0" iyy="0.000001" iyz="0" izz="0.000001"/>
+          </inertial>
+        </link>
         <joint name="${name}_temp_right_joint" type="fixed">
           <parent link="${name}_right_camera_frame"/>
           <child link="${name}_temp_right_link"/>
-          <origin xyz="0 0 0" rpy="0 0 0" />
-        </joint>
+<origin xyz="0 0 0" rpy="0 0 0" />
+        <axis xyz="0 0 1"/>
+      </joint>
       </xacro:if>
     </xacro:unless>
     <xacro:if value="${mono}">
       <!-- Camera -->
-      <link name="${name}_camera_frame" />
+      <link name="${name}_camera_frame">
+        <inertial>
+          <origin xyz="0 0 0" rpy="0 0 0" />
+          <mass value="0.001"/>
+          <inertia ixx="0.000001" ixy="0" ixz="0" iyy="0.000001" iyz="0" izz="0.000001"/>
+        </inertial>
+      </link>
       <joint name="${name}_camera_joint" type="fixed">
         <parent link="${name}_camera_center"/>
         <child link="${name}_camera_frame"/>
         <origin xyz="${optical_offset_x} 0 0" rpy="0 0 0" />
-      </joint>
-      <link name="${name}_camera_optical_frame"/>
+        <axis xyz="0 0 1"/>
+      </joint>
+      <link name="${name}_camera_optical_frame">
+        <inertial>
+          <origin xyz="0 0 0" rpy="0 0 0" />
+          <mass value="0.001"/>
+          <inertia ixx="0.000001" ixy="0" ixz="0" iyy="0.000001" iyz="0" izz="0.000001"/>
+        </inertial>
+      </link>
       <joint name="${name}_camera_optical_joint" type="fixed">
         <origin xyz="0 0 0" rpy="-${M_PI/2} 0.0 -${M_PI/2}"/>
+        <axis xyz="0 0 1"/>
         <parent link="${name}_camera_frame"/>
         <child link="${name}_camera_optical_frame"/>
@@ -245,9 +331,16 @@
     </xacro:if>
     <xacro:if value="${enable_gnss}">
-      <link name="${name}_gnss_link" />
+      <link name="${name}_gnss_link">
+        <inertial>
+          <origin xyz="0 0 0" rpy="0 0 0" />
+          <mass value="0.001"/>
+          <inertia ixx="0.000001" ixy="0" ixz="0" iyy="0.000001" iyz="0" izz="0.000001"/>
+        </inertial>
+      </link>
       <joint name="${name}_gnss_joint" type="fixed">
         <parent link="${name}_camera_link"/>
         <child link="${name}_gnss_link"/>
         <xacro:insert_block name="gnss_origin" />
+        <axis xyz="0 0 1"/>
       </joint>
     </xacro:if>

Commit message: Fixed wierd angle in Rviz2 with the camera
When using the camera from mujoco, use the /zed_mujoco_camera/depth/points topic for the point cloud

File: robot_description/frida_description/urdf/Gripper/Custom/gripper.xacro (robot description, xacro)
@@ -94,3 +94,11 @@
     <axis xyz="0 0 1"/>
   </joint>
+  <!-- <mujoco>
+    <reference body="right_finger">
+      <joint name="rightfinger" range="0 0.056" limited="true"/>
+    </reference>
+    <reference body="left_finger">
+      <joint name="leftfinger" range="0 0.056" limited="true"/>
+    </reference>
+  </mujoco> -->
 </robot>

File: robot_description/frida_description/urdf/zed/zed_macro.urdf.xacro (robot description, xacro)
@@ -183,9 +183,4 @@
         </xacro:unless>
       </link>
-      <mujoco>
-        <reference name="${name}_left_camera_frame">
-          <camera name="${name}_left_camera" mode="fixed" fovy="45" quat="0.5 0.5 -0.5 -0.5"/>
-        </reference>
-      </mujoco>
       <joint name="${name}_left_camera_joint" type="fixed">
         <parent link="${name}_camera_center"/>
@@ -337,4 +332,9 @@
       <xacro:include filename="$(find frida_description)/urdf/zed/zed_gazebo.xacro"/>
       <xacro:zed_gazebo prefix="${name}" />
+      <mujoco>
+        <reference name="${name}_left_camera_frame">
+          <camera name="${name}_mujoco_camera" mode="fixed" fovy="45" quat="-0.5 -0.5 0.5 0.5 "/>
+        </reference>
+      </mujoco>
     </xacro:if>
     <xacro:if value="${enable_gnss}">

Commit message: Final Commit: xarm mujoco simulation done
The final implementation in this branch is the inclusion of the gripper controller.
It responds to the topic "/xarm/set_tgpio_digital"  and sets the gripper open or close.
The gripper joints responds to its limits
The gripper joints are symetric

File: robot_description/frida_description/urdf/Gripper/Custom/gripper.xacro (robot description, xacro)
@@ -2,5 +2,5 @@
 <robot xmlns:xacro="http://www.ros.org/wiki/xacro">
 <xacro:property name="mesh_path" value="file://$(find frida_description)/urdf/meshes/Gripper/Custom/" />
-<xacro:macro name="load_gripper" params="attach_to:='' xyz:='0 0 0' rpy:='0 0 0' fixed_joints:='false'">
+<xacro:macro name="load_gripper" params="attach_to:='' xyz:='0 0 0' rpy:='0 0 0' fixed_joints:='false' mujoco_plugin:=false">
     <xacro:unless value="${attach_to == ''}">
       <joint name="gripper_fix" type="fixed">
@@ -86,4 +86,23 @@
     <mimic joint="rightfinger" multiplier="1" offset="0" />
   </joint>
+  <xacro:if value="${mujoco_plugin}">
+    <mujoco>
+      <reference name="right_finger">
+          <joint range="0 0.056" limited="true" />
+      </reference>
+      <reference name="left_finger">
+          <joint range="0 0.056" limited="true" />
+      </reference>
+      <equality>
+        <joint name="gripper_mimic_joint" joint1= "leftfinger" joint2="rightfinger" polycoef="0 1 0 0"/>
+      </equality>
+      <actuator>
+        <position name="finger_actuator_position" joint="rightfinger" ctrlrange="0 0.056" forcerange= "-50 50" kp ="50"/>
+        <velocity name="finger_actuator_velocity" joint="rightfinger" ctrlrange="0 0.056" forcerange= "-50 50" kv ="10"/>
+      </actuator>
+    </mujoco>
+    <xacro:include filename="$(find frida_description)/urdf/Gripper/Custom/gripper_mujoco_ros2_control.xacro" />
+    <xacro:gripper_mujoco_control/>
+  </xacro:if>
   </xacro:macro>
   <link name="zed"  />
@@ -94,11 +113,3 @@
     <axis xyz="0 0 1"/>
   </joint>
-  <!-- <mujoco>
-    <reference body="right_finger">
-      <joint name="rightfinger" range="0 0.056" limited="true"/>
-    </reference>
-    <reference body="left_finger">
-      <joint name="leftfinger" range="0 0.056" limited="true"/>
-    </reference>
-  </mujoco> -->
 </robot>

File: robot_description/frida_description/urdf/TMR2025/FRIDA.urdf.xacro (robot description, xacro)
@@ -47,7 +47,7 @@
     <xacro:if value="$(arg mujoco_plugin)">
       <mujoco>
-        <compiler angle="radian" balanceinertia="true" />
+        <compiler angle="radian" balanceinertia="true" autolimits="true"/>
       </mujoco>
-      <!-- Important to add additional files in the spawn -->
+      <!-- Important in order to add additional files in the spawn -->
       <link name="world" />
       <joint name="world_to_base" type="floating">
@@ -87,5 +87,5 @@
     <xacro:if value="$(arg load_zed)">
       <xacro:include filename="$(find frida_description)/urdf/Gripper/Custom/gripper.xacro" />
-      <xacro:load_gripper attach_to="link_eef" xyz="0 0 0.046" rpy="0 0 3.926" fixed_joints="false"/>
+      <xacro:load_gripper attach_to="link_eef" xyz="0 0 0.046" rpy="0 0 3.926" fixed_joints="false" mujoco_plugin="$(arg mujoco_plugin)" />
       <!-- ZED MACRO -->
       <xacro:include filename="$(find frida_description)/urdf/zed/zed_macro.urdf.xacro" />

File: robot_description/frida_description/urdf/xarm/xarm6/xarm6.mujoco_actuators.xacro (robot description, xacro)
@@ -86,8 +86,4 @@
         velocity="${joint6_velocity}"
         effort="${joint6_effort}" />
-      <xacro:if value="${add_gripper}">
-        <position forcelimited="true" forcerange="-20 20" ctrllimited="true" ctrlrange="0 0.05" joint="${arm_id}_joint7" kp="100" name="pos_joint7"/>
-        <velocity forcelimited="true" forcerange="-20 20" joint="${arm_id}_joint7" kv="10" name="vel_joint7"/>
-      </xacro:if>
     </actuator>
   </xacro:macro>
