Commit message: Physics-based MuJoCo pick reliability + sim-only frame and bridge fixes
End-to-end pick now works in sim with pure contact physics (no weld
shortcut), matching how the real xarm gripper holds the object.  The
sim-to-real pipeline is unchanged -- pick_server / plane_service / GPD /
perception_3d run identically -- so any grasp that works in sim will
also work on the real robot.

Summary of what landed:

  * XArmServices (frida_motion_planning): create gripper_io_client
    unconditionally.  Previously the early-return when /xarm/move_velocity
    was unavailable (true in sim) left gripper_io_client=None and every
    close_gripper() silently returned False.  The bridge never saw the
    tgpio call even though pick_server logged "Gripper closed", which is
    why MuJoCo never actually closed the fingers.

  * FRIDA_Real.urdf.xacro: wrap the world_to_base joint in
    mujoco_plugin=true/false branches.  Real robot keeps xyz="0 0 0.3"
    (the physical 0.3 m pedestal); sim uses xyz="0 0 0" so world and
    base_link coincide.  MoveIt's planning frame is "world", and
    pick_server.check_feasibility compared the plane collision object's
    z (stored in "world") against the grasp pose z (in "base_link").
    Any non-zero world<->base_link offset made that check a frame
    mismatch that silently rejected every grasp as "below acceptable
    height".

  * FRIDA_Real.urdf.xacro: add <option impratio=10 noslip_iterations=5>
    inside the mujoco block.  MuJoCo's default contact solver is not
    tuned for grasping; these two knobs tighten the friction cone and
    add a post-solve anti-slip pass, turning a 2-finger pinch grasp into
    a stable hold without needing a weld equality.

  * gripper.xacro: physics-based grasp tuning.
    - Removed kv from the MuJoCo position actuator.  kv populates
      biasprm[2] which breaks mujoco_ros2_control's actuator detection
      (it requires biasprm[2]==0), so the controller command never
      reached the MuJoCo actuator and the finger stayed pinned.  Damping
      lives on the joint itself via <dynamics> instead.
    - Tuned the actuator to mimic a servo with current limiting: kp=1000
      + forcerange=+-10 N.  Force saturates at ~10 N once contact builds
      even a millimetre of error, matching the near-constant grip force
      of a real servo clamp instead of an unphysical ramp that squeezed
      light objects out.
    - Finger geoms: friction=5/2/0.2 (silicone-on-plastic), solref=
      -50000 -500 (50 kN/m spring damper), solimp=0.98 0.999 0.0001
      (0.1 mm penetration band), condim=4 (slide + torsional friction
      so the cube cannot rotate around the finger normal inside the
      pinch).

  * table_and_object.xacro: matching friction / solref / solimp / condim
    on the cube so MuJoCo keeps the stickier side of each contact.
    Cube reshape (4x4x12 cm, 50 g) for a stable pinch grasp.

  * mujoco_ros2_control submodule (b3ca192): deferred weld-on-attach
    listener.  Shipped in the plugin for completeness but inactive -- the
    sim scene no longer declares the cube_to_eef equality, so the hook
    just logs DEBUG and does nothing.  Kept in-tree in case a future
    scene wants deterministic grasps.

  * perception_3d / pick_and_place launches: new use_sim_time,
    point_cloud_topic, pick_min_height args; plane_service gets the
    sim's /filtered_cloud (MoveIt self-filtered) so RANSAC isn't
    polluted by robot self-reflection; default unchanged for real robot.

  * mujoco_spawn/launch/mujoco_sim_init.launch.py: inline python relay
    from /vision/zero_shot_detections to /vision/detections so
    keyboard_input.py and the pick_server detection handler see
    detections under the same topic name they expect on the real robot.

  * perception_3d/src/masive_testin.cpp: expose point_cloud_topic as a
    parameter (defaults to POINT_CLOUD_TOPIC) so the sim can redirect
    cluster extraction to /filtered_cloud without changing the real
    robot default.

File: robot_description/frida_description/urdf/Gripper/Custom/gripper.xacro (robot description, xacro)
@@ -75,4 +75,8 @@
     <limit lower="0" upper="0.056"
            effort="1" velocity="8" />
+    <!-- Damping replaces the removed kv on the MuJoCo position actuator;
+         real-robot controllers ignore URDF joint dynamics so this stays
+         sim-only in effect. -->
+    <dynamics damping="5.0" friction="0.0"/>
   </joint>
   <joint
@@ -88,9 +92,31 @@
   <xacro:if value="${mujoco_plugin}">
     <mujoco>
+      <!-- Aggressive silicone-pad contact tuning for reliable grasps.
+           MuJoCo default contact (friction 1/0.005/0.0001, solref 0.02/1)
+           is smooth-metal equivalent so grips slip.  Overrides below:
+             friction 3 1 0.1: very grippy silicone.  Slide 3, spin 1,
+                roll 0.1 to resist tangential slip and cube rotation
+                during retreat accelerations.
+             solref -50000 -500: firm spring damper (50 kN/m, 500 Ns/m).
+                Stiff enough to transmit gripper force without impulsive
+                bounce; damped enough to settle fast.  Softer springs
+                (e.g. -1000) made the contact too compliant and the cube
+                oscillated out.
+             solimp 0.95 0.99 0.0005: 0.5 mm penetration band, tight
+                enough to stay realistic and give the solver room to
+                resolve contact without chatter. -->
+      <!-- condim=4 activates torsional friction (slide + torsional).
+           Default condim=3 only resists tangential slip, so the cube
+           can rotate around the finger normal inside a 2-finger pinch
+           grasp.  condim=6 also enables rolling friction but triples the
+           contact compute cost; condim=4 is the sweet spot: kills the
+           rotation-around-normal failure mode while staying realtime. -->
       <reference name="right_finger">
           <joint range="0 0.056" limited="true" />
+          <geom name="right_finger_collision_0" friction="5.0 2.0 0.2" solref="-50000 -500" solimp="0.98 0.999 0.0001" condim="4"/>
       </reference>
       <reference name="left_finger">
           <joint range="0 0.056" limited="true" />
+          <geom name="left_finger_collision_0" friction="5.0 2.0 0.2" solref="-50000 -500" solimp="0.98 0.999 0.0001" condim="4"/>
       </reference>
       <equality>
@@ -98,8 +124,19 @@
       </equality>
       <actuator>
-        <!-- kv adds velocity damping to the position actuator so the finger
-             does not bounce/oscillate around the target (the equality
-             constraint that mimics leftfinger is also underdamped without it). -->
-        <position name="finger_actuator_position" joint="rightfinger" ctrlrange="0 0.056" forcerange= "-1 1" kp ="50" kv="5"/>
+        <!-- Keep the position actuator purely proportional: adding kv here
+             populates biasprm[2] which breaks mujoco_ros2_control's actuator
+             detection (it requires biasprm[2]==0 to recognize the actuator
+             as "position"), so the ros2_control command never reaches the
+             MuJoCo actuator and the finger stays pinned.  Damping lives on
+             the joint itself below so the finger still doesn't oscillate.
+             The actuator mimics a servo-driven gripper (fast position
+             response, hardware-limited torque): high kp=1000 so commanded
+             motion settles quickly, but a low forcerange=±5 N caps the
+             applied force to what the real xarm gripper produces in grip
+             hold.  Result: force saturates at ~5 N as soon as contact
+             builds even a millimetre of error, matching the near-constant
+             grip force of a real servo clamp instead of an unphysical
+             ramp that squeezes light objects out. -->
+        <position name="finger_actuator_position" joint="rightfinger" ctrlrange="0 0.056" forcerange= "-10 10" kp ="1000"/>
         <!-- <velocity name="finger_actuator_velocity" joint="rightfinger" ctrlrange="0 0.056" forcerange= "-1 1" kv ="8"/> -->
       </actuator>

File: robot_description/frida_description/urdf/TMR2025/FRIDA_Real.urdf.xacro (robot description, xacro)
@@ -51,4 +51,19 @@
     <mujoco>
       <compiler angle="radian" balanceinertia="true" autolimits="true"/>
+      <!-- Sim-only solver tuning for reliable physics-based grasping.
+           The combination below keeps the cheap defaults where they work
+           (PGS is fine for articulated dynamics) but adds the two knobs
+           that matter for grasping stability:
+             impratio=10: tightens the friction cone so the tangential
+                friction ceiling stays proportional to normal force under
+                rapid normal-force changes.
+             noslip_iterations=5: post-solve pass that explicitly enforces
+                no-tangential-slip at each contact point.
+           The more aggressive integrator=implicit + solver=Newton +
+           cone=elliptic combo was tested but tripled the physics cost
+           and stalled the sim well below realtime so ros2_control timed
+           out, which looks externally like the pick freezing in place. -->
+      <option impratio="10"
+              noslip_iterations="5"/>
       <reference name="link1"><body gravcomp="1"/></reference>
       <reference name="link2"><body gravcomp="1"/></reference>
@@ -65,10 +80,27 @@
     </mujoco>
   </xacro:if>
+  <!-- The world<->base_link offset matters for MoveIt because "world" is the
+       planning frame: the plane-collision-object added by perception_3d in
+       "base_link" gets stored by MoveIt in "world", and pick_server.check_
+       feasibility compares its z against the grasp pose (in "base_link").
+       Any non-zero offset becomes a silent frame mismatch that fails every
+       pick.  On the real robot the 0.3 m pedestal is the physical mounting;
+       in MuJoCo the arm is attached directly to world and there is no
+       pedestal, so pin world<->base_link at identity for sim only. -->
   <link name="world" />
-  <joint name="world_to_base" type="fixed">
-    <parent link="world" />
-    <child link="base_link" />
-    <origin rpy="0 0 0" xyz="0 0 0.3" />
-  </joint>
+  <xacro:if value="$(arg mujoco_plugin)">
+    <joint name="world_to_base" type="fixed">
+      <parent link="world" />
+      <child link="base_link" />
+      <origin rpy="0 0 0" xyz="0 0 0" />
+    </joint>
+  </xacro:if>
+  <xacro:unless value="$(arg mujoco_plugin)">
+    <joint name="world_to_base" type="fixed">
+      <parent link="world" />
+      <child link="base_link" />
+      <origin rpy="0 0 0" xyz="0 0 0.3" />
+    </joint>
+  </xacro:unless>
   <!-- XARM MACRO -->
   <xacro:include filename="$(find frida_description)/urdf/xarm/xarm_device_macro.xacro" />

File: robot_description/frida_description/urdf/TMR2025/table_and_object.xacro (robot description, xacro)
@@ -40,6 +40,11 @@
   </joint>
   <!-- ============ CUBE (pickable) ============ -->
-  <!-- 5 cm side, 100 g, sitting on the table.
-       Floating joint -> MuJoCo free joint, so it falls/moves with physics. -->
+  <!-- 4x4 cm x 12 cm tall, 100 g, sitting on the table.
+       Narrow enough (4 cm) for the custom gripper's ~5.6 cm opening.
+       The 12 cm height keeps the collision volume small so MoveIt can
+       plan grasp approaches reliably; feasibility is tuned to match via
+       `pick_min_height:=0.05` on the sim's pick_and_place.launch.py.
+       Floating joint -> MuJoCo free joint, so it falls/moves with
+       physics. -->
   <link name="cube_link">
     <visual>
@@ -59,10 +64,13 @@
     </collision>
     <inertial>
-      <mass value="0.1"/>
+      <mass value="0.05"/>
       <origin xyz="0 0 0" rpy="0 0 0"/>
-      <!-- Cuboid inertia for 4 x 4 x 12 cm, 100 g.
-           Ixx = Iyy = (1/12)*m*(a^2 + c^2) = (1/12)*0.1*(0.0016 + 0.0144) = 1.33e-4
-           Izz = (1/12)*m*(a^2 + b^2)       = (1/12)*0.1*(0.0016 + 0.0016) = 2.67e-5 -->
-      <inertia ixx="1.33e-4" ixy="0" ixz="0" iyy="1.33e-4" iyz="0" izz="2.67e-5"/>
+      <!-- Cuboid inertia for 4 x 4 x 12 cm, 50 g.  Halved from the 100 g
+           value because the sim's gripper hold force (~2-4 N effective
+           with kp=200 at small contact error) couldn't resist the
+           inertial spikes from arm retreats on a 100 g load; a 50 g mass
+           keeps the behaviour realistic without requiring unphysical
+           clamping force. -->
+      <inertia ixx="6.7e-5" ixy="0" ixz="0" iyy="6.7e-5" iyz="0" izz="1.33e-5"/>
     </inertial>
   </link>
@@ -73,3 +81,21 @@
     <origin xyz="0.55 0 0.76" rpy="0 0 0"/>
   </joint>
+  <!-- Match the gripper finger contact tuning for consistent behaviour
+       (MuJoCo takes the softer/less-grippy of the two contacting geoms).
+       Aggressive silicone-on-plastic friction (3/1/0.1) plus a firmer
+       solref/solimp so the grasp doesn't bounce the cube out. -->
+  <mujoco>
+    <reference name="cube_link">
+      <geom name="cube_link_collision_0" friction="5.0 2.0 0.2" solref="-50000 -500" solimp="0.98 0.999 0.0001" condim="4"/>
+    </reference>
+    <!-- Weld-on-attach was tested but leaves the cube welded at whatever
+         offset it had when pick_server's attach signal fires (even with a
+         settle delay), which visually and physically freezes the cube in
+         a skewed orientation on the gripper.  Removed in favour of a pure
+         physics grasp: tuned friction + MuJoCo solver options below.  The
+         mujoco_ros2_control_plugin still subscribes to
+         /attached_collision_object and looks for a "cube_to_eef" equality;
+         without the declaration it simply logs DEBUG and does nothing, so
+         no other code changes are needed. -->
+  </mujoco>
 </robot>

Commit message: MuJoCo sim: finger adhesion grasp, taller cube, CLIP at build time
- gripper.xacro: declare three MuJoCo adhesion actuators (right finger,
  left finger, gripper body, gain=200).  Paired with the plugin's
  gripper-trajectory listener, these give a deterministic pick without
  a weld constraint (and without the weld's orientation-freezing and
  detach-timing issues).  Sim-only, gated by mujoco_plugin=true.

- table_and_object.xacro: cube grows from 12 cm to 18 cm tall (50 g
  unchanged) so top grasps clear pick_server's pick_min_height=0.10 m
  safety margin.  This keeps the sim on the same pick_min_height as the
  real robot instead of needing a per-launch override.  Inertia
  recomputed for the new geometry; drop the stale weld-attach comment.

- requirements.txt: pin CLIP (+ ftfy/regex/tqdm) so YOLOE's zero-shot
  detector boots without pip-installing on first use.

- Bump the mujoco_ros2_control submodule to 35f8b40 for the matching
  adhesion sync and non-joint actuator crash fix.

File: robot_description/frida_description/urdf/Gripper/Custom/gripper.xacro (robot description, xacro)
@@ -140,4 +140,23 @@
         <position name="finger_actuator_position" joint="rightfinger" ctrlrange="0 0.056" forcerange= "-10 10" kp ="1000"/>
         <!-- <velocity name="finger_actuator_velocity" joint="rightfinger" ctrlrange="0 0.056" forcerange= "-1 1" kv ="8"/> -->
+        <!-- Adhesion actuators on each finger.  MuJoCo native "adhesion"
+             applies an attractive force between the named body and every
+             body currently in contact with it (force = gain * ctrl, acts
+             only while contact exists).  When pick_server closes the
+             gripper on an object, both fingers contact the object; the
+             plugin sets adhesion ctrl to 1 on attach and 0 on detach,
+             turning each finger into a silicone+magnet pad.  This is the
+             standard mechanism used by MetaWorld and other MuJoCo
+             manipulation benchmarks: deterministic grasp without the
+             rigid-body weld's timing/orientation issues, because the
+             force is only applied through natural contact. -->
+        <!-- gain=200 N per contact.  Single-finger-only contacts
+             (common when GPD's grasp is slightly off-center) still
+             resist gravity's torque on a 50 g cube with this pull
+             force.  Also cover the gripper body itself so a cube that
+             slides against the palm gets attracted to it as well. -->
+        <adhesion name="right_finger_adhesion" body="right_finger" ctrlrange="0 1" gain="200"/>
+        <adhesion name="left_finger_adhesion"  body="left_finger"  ctrlrange="0 1" gain="200"/>
+        <adhesion name="gripper_adhesion"      body="gripper"      ctrlrange="0 1" gain="200"/>
       </actuator>
     </mujoco>

File: robot_description/frida_description/urdf/TMR2025/table_and_object.xacro (robot description, xacro)
@@ -40,9 +40,16 @@
   </joint>
   <!-- ============ CUBE (pickable) ============ -->
-  <!-- 4x4 cm x 12 cm tall, 100 g, sitting on the table.
+  <!-- 4x4 cm x 18 cm tall, 50 g, sitting on the table.
        Narrow enough (4 cm) for the custom gripper's ~5.6 cm opening.
-       The 12 cm height keeps the collision volume small so MoveIt can
-       plan grasp approaches reliably; feasibility is tuned to match via
-       `pick_min_height:=0.05` on the sim's pick_and_place.launch.py.
+       The 18 cm height is deliberate: pick_server.check_feasibility
+       rejects any grasp whose z is below plane.z + pick_min_height, and
+       pick_min_height defaults to 0.10 m (the real-robot safety margin
+       that prevents the gripper from colliding with the table during
+       approach).  A 12 cm cube only gave grasps at 4-8 cm above the
+       table top, mostly below that threshold; 18 cm puts the cube top
+       at 18 cm above the table so top-grasps clear the margin with
+       room to spare.  Sim matches real: no per-environment pick args.
+       50 g mass (not 100 g) so the ~5 N grip force the servo applies at
+       contact holds the cube through arm retreats without slipping.
        Floating joint -> MuJoCo free joint, so it falls/moves with
        physics. -->
@@ -51,5 +58,5 @@
       <origin xyz="0 0 0" rpy="0 0 0"/>
       <geometry>
-        <box size="0.04 0.04 0.12"/>
+        <box size="0.04 0.04 0.18"/>
       </geometry>
       <material name="cube_green">
@@ -60,5 +67,5 @@
       <origin xyz="0 0 0" rpy="0 0 0"/>
       <geometry>
-        <box size="0.04 0.04 0.12"/>
+        <box size="0.04 0.04 0.18"/>
       </geometry>
     </collision>
@@ -66,11 +73,8 @@
       <mass value="0.05"/>
       <origin xyz="0 0 0" rpy="0 0 0"/>
-      <!-- Cuboid inertia for 4 x 4 x 12 cm, 50 g.  Halved from the 100 g
-           value because the sim's gripper hold force (~2-4 N effective
-           with kp=200 at small contact error) couldn't resist the
-           inertial spikes from arm retreats on a 100 g load; a 50 g mass
-           keeps the behaviour realistic without requiring unphysical
-           clamping force. -->
-      <inertia ixx="6.7e-5" ixy="0" ixz="0" iyy="6.7e-5" iyz="0" izz="1.33e-5"/>
+      <!-- Cuboid inertia for 4 x 4 x 18 cm, 50 g.
+           Ixx = Iyy = (1/12)*m*(a^2 + c^2) = (1/12)*0.05*(0.0016 + 0.0324) = 1.42e-4
+           Izz = (1/12)*m*(a^2 + b^2)       = (1/12)*0.05*(0.0016 + 0.0016) = 1.33e-5 -->
+      <inertia ixx="1.42e-4" ixy="0" ixz="0" iyy="1.42e-4" iyz="0" izz="1.33e-5"/>
     </inertial>
   </link>
@@ -78,6 +82,6 @@
     <parent link="world"/>
     <child link="cube_link"/>
-    <!-- Start sitting on the table top (0.7 m) + half the cube height (0.06 m). -->
-    <origin xyz="0.55 0 0.76" rpy="0 0 0"/>
+    <!-- Start sitting on the table top (0.7 m) + half the cube height (0.09 m). -->
+    <origin xyz="0.55 0 0.79" rpy="0 0 0"/>
   </joint>
   <!-- Match the gripper finger contact tuning for consistent behaviour
@@ -89,13 +93,10 @@
       <geom name="cube_link_collision_0" friction="5.0 2.0 0.2" solref="-50000 -500" solimp="0.98 0.999 0.0001" condim="4"/>
     </reference>
-    <!-- Weld-on-attach was tested but leaves the cube welded at whatever
-         offset it had when pick_server's attach signal fires (even with a
-         settle delay), which visually and physically freezes the cube in
-         a skewed orientation on the gripper.  Removed in favour of a pure
-         physics grasp: tuned friction + MuJoCo solver options below.  The
-         mujoco_ros2_control_plugin still subscribes to
-         /attached_collision_object and looks for a "cube_to_eef" equality;
-         without the declaration it simply logs DEBUG and does nothing, so
-         no other code changes are needed. -->
+    <!-- No weld equality: we use MuJoCo's native adhesion actuators on
+         the finger bodies instead (declared in gripper.xacro).  Adhesion
+         is force-based rather than rigid-constraint-based, so the cube
+         stays in whatever grip pose the physics settles into, and the
+         grip releases naturally when the gripper opens.  Same mechanism
+         used in MetaWorld and similar MuJoCo manipulation benchmarks. -->
   </mujoco>
 </robot>
