Commit message: fix(sim): make FRIDA visible in MuJoCo and stabilize gripper fingers (#979)
mujoco_sim_init.launch.py was producing an empty MJCF for FRIDA because
urdf2mjcf.py recurses from a hardcoded "world" root, and the FRIDA URDF
only emits that link when xacro arg mujoco_plugin=true — which the sim
MoveItConfigsBuilder was never passing. Same path also disabled the
custom gripper and ZED camera because they're gated on load_zed.

- arm_pkg/moveit_configs_builder_sim.py: pass mujoco_plugin='true' in
  __urdf_xacro_args so the xacro emits the world link, world_to_base
  floating joint, mujoco compiler block, and the per-link gravcomp
  references the simulation depends on.
- mujoco_spawn/mujoco_sim_init.launch.py: declare load_zed and default
  it to true; propagate to MoveItConfigsBuilder so the custom gripper
  and ZED are included.
- FRIDA.urdf.xacro: swap the official zed_camera macro for the custom
  load_zed (matching FRIDA_Real.urdf.xacro). The official macro pulls
  zed2.stl from zed_msgs — an apt package whose meshes don't ship —
  and lacks the <mujoco><camera name="zed_mujoco_camera_link"/> block
  the launch's topic remappings expect.
- Gripper/Custom/gripper.xacro: add damping=5 and armature=0.01 to the
  finger joint references. urdf2mjcf.py copies dynamics for revolute
  joints but not for prismatic, so the fingers were undamped against
  a kp=1000 position actuator and oscillated.

File: robot_description/frida_description/urdf/Gripper/Custom/gripper.xacro (robot description, xacro)
@@ -113,9 +113,9 @@
            rotation-around-normal failure mode while staying realtime. -->
       <reference name="right_finger">
-          <joint range="0 0.056" limited="true" />
+          <joint range="0 0.056" limited="true" damping="5.0" armature="0.01"/>
           <geom name="right_finger_collision_0" friction="5.0 2.0 0.2" solref="-50000 -500" solimp="0.98 0.999 0.0001" condim="4"/>
       </reference>
       <reference name="left_finger">
-          <joint range="0 0.056" limited="true" />
+          <joint range="0 0.056" limited="true" damping="5.0" armature="0.01"/>
           <geom name="left_finger_collision_0" friction="5.0 2.0 0.2" solref="-50000 -500" solimp="0.98 0.999 0.0001" condim="4"/>
       </reference>

Commit message: Revert "fix(sim): make FRIDA visible in MuJoCo and stabilize gripper fingers …"
This reverts commit 03dd6caabe9f35b7f8d5e2ab7f3dbed53ac1dac3.

File: robot_description/frida_description/urdf/Gripper/Custom/gripper.xacro (robot description, xacro)
@@ -113,9 +113,9 @@
            rotation-around-normal failure mode while staying realtime. -->
       <reference name="right_finger">
-          <joint range="0 0.056" limited="true" damping="5.0" armature="0.01"/>
+          <joint range="0 0.056" limited="true" />
           <geom name="right_finger_collision_0" friction="5.0 2.0 0.2" solref="-50000 -500" solimp="0.98 0.999 0.0001" condim="4"/>
       </reference>
       <reference name="left_finger">
-          <joint range="0 0.056" limited="true" damping="5.0" armature="0.01"/>
+          <joint range="0 0.056" limited="true" />
           <geom name="left_finger_collision_0" friction="5.0 2.0 0.2" solref="-50000 -500" solimp="0.98 0.999 0.0001" condim="4"/>
       </reference>

File: robot_description/frida_description/urdf/TMR2025/FRIDA.urdf.xacro (robot description, xacro)
@@ -88,6 +88,9 @@
       <xacro:include filename="$(find frida_description)/urdf/Gripper/Custom/gripper.xacro" />
       <xacro:load_gripper attach_to="link_eef" xyz="0 0 0.046" rpy="0 0 3.926" fixed_joints="false" mujoco_plugin="$(arg mujoco_plugin)" />
-      <xacro:include filename="$(find frida_description)/urdf/zed/zed.xacro" />
-      <xacro:load_zed attach_to="zed" xyz="0 0 0" rpy="0 0 0" mujoco_plugin="$(arg mujoco_plugin)" />
+      <!-- ZED MACRO -->
+      <xacro:include filename="$(find frida_description)/urdf/zed/zed_macro.urdf.xacro" />
+      <xacro:zed_camera name="zed" model="zed2" custom_baseline="0" enable_gnss="false" simulation="true" attach_to="zed" xyz="0 0 0" rpy="0 0 0">
+          <origin xyz="0 0 0" rpy="0 0 0"/>
+      </xacro:zed_camera>
     </xacro:if>
     <!-- <xacro:if value="$(arg load_zed)"> -->

Commit message: VAMP motion planning integration with OMPL fallback for FRIDA arm (#977)
Integrates VAMP (Vectorized And Motion Planning) as the default MoveIt
planner for the FRIDA xArm6, replacing OMPL for typical plans (~20-100 ms
wall-clock through the full pipeline) while keeping OMPL as an automatic
fallback for the cases where VAMP's sphere collision model disagrees with
FCL's mesh check. The caller — RViz, move_group_interface, pick_server —
sees a single planner named "vamp"; the layered behavior is internal.

Architecture (each layer catches what the previous can miss):

  pipeline "vamp"
    └── VampPlannerManager (loads ompl_interface/OMPLPlanner via pluginlib)
          └── VampPlanningContext::solve()
               ├── (1) VAMP planning via ROS2 service (sphere check, fast)
               ├── (2) FCL post-validation against PlanningScene (mesh, accurate)
               │   PASS → return VAMP plan
               └── (3) runOmplFallback() up to 4 retries
                     ├── ompl_interface::OMPLPlanner::solve()
                     ├── TOTG densify + time-parameterize
                     ├── validate the densified result against scene
                     └── return first attempt that survives

Why each layer matters:
- VAMP's sphere model is an approximation; it occasionally returns plans
  that look collision-free in sphere-space but graze obstacles in mesh
  geometry. The plugin validates with the same isPathValid check the
  outer pipeline would run, so we never return a bad trajectory.
- RRTConnect is stochastic, and TOTG's resampling can land intermediate
  states inside obstacles even when OMPL's own waypoints are clear (most
  often the ZED camera link grazes on interpolated wrist motion). The
  retry loop handles this transparently — user sees one Plan request.
- OMPL's PlanningContext returns a geometric path with zero time stamps
  because timing is normally added by response adapters in the outer
  pipeline. Our context invokes OMPL directly, so we run TOTG ourselves
  before returning — otherwise the controller rejects the trajectory.

Other parts of this change:

- The VAMP submodule's Python bindings live at vamp/src/ rather than
  in PYTHONPATH; docker/manipulation/.bash_aliases now exports the
  right path so interactive shells can `import vamp`. The setup_vamp.sh
  entrypoint also exports it for non-interactive ros2 run invocations.

- vamp_server.py now parses arm joint limits straight from the
  spherized URDF and rejects out-of-limit requests in <1 ms with a
  diagnostic, rather than letting them sink three RRTConnect retries
  (~70 ms) before bottoming out on a geometric validate() failure.

- The 68-sphere full-FRIDA collision model in frida_real.hh covers
  base_link + link1..6 + gripper + both fingers + zed_camera_link +
  intel_realsense + laser. An earlier draft of this work shipped an
  82-sphere model whose URDF source had every collision sphere with
  origin (0,0,0), causing Cricket to emit alias-style y[i]=y[base]
  FK and stacking all spheres at each link's joint. The current model
  is generated from a URDF with proper per-sphere offsets and has zero
  alias copies in its FK.

- The FRIDA Custom gripper's <ros2_control> declaration moved out of
  the <xacro:if mujoco_plugin> block and now picks the hardware plugin
  per mode (UFRobotFakeSystemHardware in fake, MujocoSystem in MuJoCo,
  real plugin on hardware). The fake launch merges custom_gripper_-
  controllers.yaml on top of xarm6 controllers and spawns the
  xarm_gripper_traj_controller alongside the arm controller, so
  rightfinger gets state-published in fake mode (leftfinger follows
  via URDF <mimic>). Before this, the finger meshes rendered at world
  origin and VAMP collision-checked them at the wrong location.

- probe_cuboid.py is a standalone diagnostic that exercises
  vamp.frida_real.fk() to verify sphere positions and collision
  detection against a configurable AABB. It found the alias-FK bug
  in the previous spherization and is useful for verifying any future
  model regen.

- inflate_body_spheres.py is a small offline utility that walks a
  spherized URDF and adds a configurable padding to spheres on body
  links (link_base, link1..6, base_link) while leaving gripper,
  fingers, and sensor links untouched. Not wired into any pipeline,
  kept for a future iteration that wants asymmetric safety margin
  without breaking close-approach picking.

- .gitmodules registers manipulation/packages/vamp (the upstream
  KavrakiLab/vamp submodule) which was missing despite being in the
  tree as a gitlink.

Verified end-to-end against fake_moveit_config: Tier 2.1-2.7 all pass,
including the corner case where VAMP's sphere model misses a real
collision — the OMPL fallback fires automatically and the plan
executes. Worst observed wall-clock for hard obstacle scenarios is
~7 s (RRTConnect retries inside the fallback); typical case is
~100-200 ms. Real-hardware testing (Tier 4) and pick-and-place
integration (Tier 3) are out of scope and follow as separate work.

File: robot_description/frida_description/urdf/Gripper/Custom/gripper.xacro (robot description, xacro)
@@ -2,5 +2,5 @@
 <robot xmlns:xacro="http://www.ros.org/wiki/xacro">
 <xacro:property name="mesh_path" value="file://$(find frida_description)/urdf/meshes/Gripper/Custom/" />
-<xacro:macro name="load_gripper" params="attach_to:='' xyz:='0 0 0' rpy:='0 0 0' fixed_joints:='false' mujoco_plugin:=false">
+<xacro:macro name="load_gripper" params="attach_to:='' xyz:='0 0 0' rpy:='0 0 0' fixed_joints:='false' mujoco_plugin:=false ros2_control_plugin:='uf_robot_hardware/UFRobotFakeSystemHardware'">
     <xacro:unless value="${attach_to == ''}">
       <joint name="gripper_fix" type="fixed">
@@ -161,7 +161,26 @@
       </actuator>
     </mujoco>
-    <xacro:include filename="$(find frida_description)/urdf/Gripper/Custom/gripper_mujoco_ros2_control.xacro" />
-    <xacro:gripper_mujoco_control/>
   </xacro:if>
+  <!-- ros2_control for the gripper: declared only for sim hardware (MuJoCo or
+       the fake plugin used by frida_fake_moveit_config). On real hardware the
+       gripper is driven through xarm's separate service API, NOT ros2_control —
+       UFRobotSystemHardware needs a robot_ip param per <ros2_control> block,
+       and a second instance for the gripper (without its own robot_ip) crashes
+       the controller_manager with "No param named 'robot_ip'" → SIGSEGV. For
+       fake/MuJoCo modes we still need this so rightfinger gets state-published
+       (otherwise the finger meshes render at world origin). initial_value=0.056
+       in MuJoCo opens the gripper at start; defaults to 0 elsewhere. -->
+  <xacro:include filename="$(find frida_description)/urdf/Gripper/Custom/gripper_ros2_control.xacro" />
+  <xacro:if value="${mujoco_plugin}">
+    <xacro:gripper_ros2_control
+        ros2_control_plugin="mujoco_ros2_control/MujocoSystem"
+        initial_value="0.056" />
+  </xacro:if>
+  <xacro:unless value="${mujoco_plugin}">
+    <xacro:if value="${'Fake' in ros2_control_plugin}">
+      <xacro:gripper_ros2_control
+          ros2_control_plugin="${ros2_control_plugin}" />
+    </xacro:if>
+  </xacro:unless>
   </xacro:macro>
   <link name="zed"  />
