Commit message: 1244 remove gazebo and mujoco code (#1281)
* Remove Mujoco and Gazebo related code and configurations

* Remove Gazebo and Mujoco related launch files and configurations

* Remove xArm Gazebo launch file and related configurations

* Remove unused simulation time configuration from pick_and_place launch file

* Refactor XArmServices and perception_3d launch files to remove simulation time configurations

* Remove vendored mujoco_ros2_control submodule and clean CI ignore list

* Remove gazebo world files

* Remove Gazebo and MuJoCo related files and configurations

* Remove MuJoCo related code from xarm6_robot_macro.xacro

* Remove simulation-related Gazebo and MuJoCo code from zed_macro.urdf.xacro

* Remove MuJoCo/gazebo xacro blocks and plumbing

* Remove gazebo/webots sim code from omnibase robot.xacro and IMU

* Fix formatting issues in launch files and remove unused Gazebo configurations

* Fix perception_3d formatting and remove dead worlds install() from CMakeLists

* Remove world link and world_to_base joint from FRIDA_Real.urdf.xacro

* Remove mujoco_ros2_control package

File: robot_description/frida_description/urdf/Gripper/Custom/gripper.xacro (robot description, xacro)
@@ -75,7 +75,6 @@
     <limit lower="0" upper="0.056"
            effort="1" velocity="8" />
-    <!-- Damping replaces the removed kv on the MuJoCo position actuator;
-         real-robot controllers ignore URDF joint dynamics so this stays
-         sim-only in effect. -->
+    <!-- Real-robot controllers ignore URDF joint dynamics, so this has no
+         effect on hardware; kept for completeness/any future simulator. -->
     <dynamics damping="5.0" friction="0.0"/>
   </joint>
@@ -90,97 +89,17 @@
     <mimic joint="rightfinger" multiplier="1" offset="0" />
   </joint>
-  <xacro:if value="${mujoco_plugin}">
-    <mujoco>
-      <!-- Aggressive silicone-pad contact tuning for reliable grasps.
-           MuJoCo default contact (friction 1/0.005/0.0001, solref 0.02/1)
-           is smooth-metal equivalent so grips slip.  Overrides below:
-             friction 3 1 0.1: very grippy silicone.  Slide 3, spin 1,
-                roll 0.1 to resist tangential slip and cube rotation
-                during retreat accelerations.
-             solref -50000 -500: firm spring damper (50 kN/m, 500 Ns/m).
-                Stiff enough to transmit gripper force without impulsive
-                bounce; damped enough to settle fast.  Softer springs
-                (e.g. -1000) made the contact too compliant and the cube
-                oscillated out.
-             solimp 0.95 0.99 0.0005: 0.5 mm penetration band, tight
-                enough to stay realistic and give the solver room to
-                resolve contact without chatter. -->
-      <!-- condim=4 activates torsional friction (slide + torsional).
-           Default condim=3 only resists tangential slip, so the cube
-           can rotate around the finger normal inside a 2-finger pinch
-           grasp.  condim=6 also enables rolling friction but triples the
-           contact compute cost; condim=4 is the sweet spot: kills the
-           rotation-around-normal failure mode while staying realtime. -->
-      <reference name="right_finger">
-          <joint range="0 0.056" limited="true" damping="5.0" armature="0.01"/>
-          <geom name="right_finger_collision_0" friction="5.0 2.0 0.2" solref="-50000 -500" solimp="0.98 0.999 0.0001" condim="4"/>
-      </reference>
-      <reference name="left_finger">
-          <joint range="0 0.056" limited="true" damping="5.0" armature="0.01"/>
-          <geom name="left_finger_collision_0" friction="5.0 2.0 0.2" solref="-50000 -500" solimp="0.98 0.999 0.0001" condim="4"/>
-      </reference>
-      <equality>
-        <joint name="gripper_mimic_joint" joint1= "leftfinger" joint2="rightfinger" polycoef="0 1 0 0"/>
-      </equality>
-      <actuator>
-        <!-- Keep the position actuator purely proportional: adding kv here
-             populates biasprm[2] which breaks mujoco_ros2_control's actuator
-             detection (it requires biasprm[2]==0 to recognize the actuator
-             as "position"), so the ros2_control command never reaches the
-             MuJoCo actuator and the finger stays pinned.  Damping lives on
-             the joint itself below so the finger still doesn't oscillate.
-             The actuator mimics a servo-driven gripper (fast position
-             response, hardware-limited torque): high kp=1000 so commanded
-             motion settles quickly, but a low forcerange=±5 N caps the
-             applied force to what the real xarm gripper produces in grip
-             hold.  Result: force saturates at ~5 N as soon as contact
-             builds even a millimetre of error, matching the near-constant
-             grip force of a real servo clamp instead of an unphysical
-             ramp that squeezes light objects out. -->
-        <position name="finger_actuator_position" joint="rightfinger" ctrlrange="0 0.056" forcerange= "-10 10" kp ="1000"/>
-        <!-- <velocity name="finger_actuator_velocity" joint="rightfinger" ctrlrange="0 0.056" forcerange= "-1 1" kv ="8"/> -->
-        <!-- Adhesion actuators on each finger.  MuJoCo native "adhesion"
-             applies an attractive force between the named body and every
-             body currently in contact with it (force = gain * ctrl, acts
-             only while contact exists).  When pick_server closes the
-             gripper on an object, both fingers contact the object; the
-             plugin sets adhesion ctrl to 1 on attach and 0 on detach,
-             turning each finger into a silicone+magnet pad.  This is the
-             standard mechanism used by MetaWorld and other MuJoCo
-             manipulation benchmarks: deterministic grasp without the
-             rigid-body weld's timing/orientation issues, because the
-             force is only applied through natural contact. -->
-        <!-- gain=200 N per contact.  Single-finger-only contacts
-             (common when GPD's grasp is slightly off-center) still
-             resist gravity's torque on a 50 g cube with this pull
-             force.  Also cover the gripper body itself so a cube that
-             slides against the palm gets attracted to it as well. -->
-        <adhesion name="right_finger_adhesion" body="right_finger" ctrlrange="0 1" gain="200"/>
-        <adhesion name="left_finger_adhesion"  body="left_finger"  ctrlrange="0 1" gain="200"/>
-        <adhesion name="gripper_adhesion"      body="gripper"      ctrlrange="0 1" gain="200"/>
-      </actuator>
-    </mujoco>
-  </xacro:if>
-  <!-- ros2_control for the gripper: declared only for sim hardware (MuJoCo or
-       the fake plugin used by frida_fake_moveit_config). On real hardware the
+  <!-- ros2_control for the gripper: declared only for the fake plugin used
+       by frida_fake_moveit_config. On real hardware the
        gripper is driven through xarm's separate service API, NOT ros2_control —
        UFRobotSystemHardware needs a robot_ip param per <ros2_control> block,
        and a second instance for the gripper (without its own robot_ip) crashes
        the controller_manager with "No param named 'robot_ip'" → SIGSEGV. For
-       fake/MuJoCo modes we still need this so rightfinger gets state-published
-       (otherwise the finger meshes render at world origin). initial_value=0.056
-       in MuJoCo opens the gripper at start; defaults to 0 elsewhere. -->
+       fake mode we still need this so rightfinger gets state-published
+       (otherwise the finger meshes render at world origin). -->
   <xacro:include filename="$(find frida_description)/urdf/Gripper/Custom/gripper_ros2_control.xacro" />
-  <xacro:if value="${mujoco_plugin}">
+  <xacro:if value="${'Fake' in ros2_control_plugin}">
     <xacro:gripper_ros2_control
-        ros2_control_plugin="mujoco_ros2_control/MujocoSystem"
-        initial_value="0.056" />
+        ros2_control_plugin="${ros2_control_plugin}" />
   </xacro:if>
-  <xacro:unless value="${mujoco_plugin}">
-    <xacro:if value="${'Fake' in ros2_control_plugin}">
-      <xacro:gripper_ros2_control
-          ros2_control_plugin="${ros2_control_plugin}" />
-    </xacro:if>
-  </xacro:unless>
   </xacro:macro>
   <link name="zed"  />

File: robot_description/frida_description/urdf/TMR2025/robot.xacro (robot description, xacro)
@@ -11,4 +11,3 @@
 <xacro:include filename="realsense.xacro"/>
 <xacro:include filename="$(find frida_description)/urdf/RoboCup2024/imu.xacro"/>
-<xacro:include filename="$(find frida_description)/urdf/RoboCup2024/gazebo.xacro"/>
 </robot>

File: robot_description/frida_description/urdf/omnibase/FRIDA_Real.urdf.xacro (robot description, xacro)
@@ -34,5 +34,4 @@
   <xacro:arg name="geometry_mesh_tcp_rpy" default="0 0 0"/>
   <xacro:arg name="baud_checkset" default="true"/>
-  <xacro:arg name="mujoco_plugin" default="false"/>
   <xacro:arg name="default_gripper_baud" default="2000000"/>
   <xacro:arg name="attach_to" default="xarm_base"/>
@@ -44,48 +43,4 @@
   <!-- ROBOT COMPONENTS -->
   <xacro:include filename="$(find frida_description)/urdf/omnibase/robot.xacro"/>
-  <!-- MUJOCO PARAMS -->
-  <!-- gravcomp mirrors the xarm6 firmware's internal gravity compensation:
-       the real servos hold pose against gravity on their own, so the sim does the same.
-       Applied only on arm+gripper bodies so world objects still fall realistically. -->
-  <xacro:if value="$(arg mujoco_plugin)">
-    <mujoco>
-      <compiler angle="radian" balanceinertia="true" autolimits="true"/>
-      <!-- Sim-only solver tuning for reliable physics-based grasping.
-           The combination below keeps the cheap defaults where they work
-           (PGS is fine for articulated dynamics) but adds the two knobs
-           that matter for grasping stability:
-             impratio=10: tightens the friction cone so the tangential
-                friction ceiling stays proportional to normal force under
-                rapid normal-force changes.
-             noslip_iterations=5: post-solve pass that explicitly enforces
-                no-tangential-slip at each contact point.
-           The more aggressive integrator=implicit + solver=Newton +
-           cone=elliptic combo was tested but tripled the physics cost
-           and stalled the sim well below realtime so ros2_control timed
-           out, which looks externally like the pick freezing in place. -->
-      <option impratio="10"
-              noslip_iterations="5"/>
-      <reference name="link1"><body gravcomp="1"/></reference>
-      <reference name="link2"><body gravcomp="1"/></reference>
-      <reference name="link3"><body gravcomp="1"/></reference>
-      <reference name="link4"><body gravcomp="1"/></reference>
-      <reference name="link5"><body gravcomp="1"/></reference>
-      <reference name="link6"><body gravcomp="1"/></reference>
-      <reference name="link_eef"><body gravcomp="1"/></reference>
-      <reference name="gripper"><body gravcomp="1"/></reference>
-      <reference name="right_finger"><body gravcomp="1"/></reference>
-      <reference name="left_finger"><body gravcomp="1"/></reference>
-      <reference name="zed"><body gravcomp="1"/></reference>
-      <reference name="zed_camera_link"><body gravcomp="1"/></reference>
-    </mujoco>
-  </xacro:if>
-  <xacro:if value="$(arg mujoco_plugin)">
-    <link name="world" />
-    <joint name="world_to_base" type="fixed">
-      <parent link="world" />
-      <child link="base_footprint" />
-      <origin rpy="0 0 0" xyz="0 0 0" />
-    </joint>
-  </xacro:if>
   <!-- XARM MACRO -->
   <xacro:include filename="$(find frida_description)/urdf/xarm/xarm_device_macro.xacro" />
@@ -95,5 +50,4 @@
     add_bio_gripper="$(arg add_bio_gripper)" dof="$(arg dof)"
     ros2_control_plugin="$(arg ros2_control_plugin)" robot_type="$(arg robot_type)"
-    mujoco_plugin="$(arg mujoco_plugin)"
     load_gazebo_plugin="false" ros2_control_params="$(arg ros2_control_params)"
     add_realsense_d435i="$(arg add_realsense_d435i)"
@@ -126,8 +80,8 @@
   <!-- Gripper -->
   <xacro:include filename="$(find frida_description)/urdf/Gripper/Custom/gripper.xacro" />
-  <xacro:load_gripper attach_to="link_eef" xyz="0 0 0.046" rpy="0 0 3.926" fixed_joints="false" mujoco_plugin="$(arg mujoco_plugin)" ros2_control_plugin="$(arg ros2_control_plugin)"/>
+  <xacro:load_gripper attach_to="link_eef" xyz="0 0 0.046" rpy="0 0 3.926" fixed_joints="false" ros2_control_plugin="$(arg ros2_control_plugin)"/>
    <!-- ZED MACRO -->
   <xacro:include filename="$(find frida_description)/urdf/zed/zed.xacro" />
-  <xacro:load_zed attach_to="zed" xyz="0.0 0 0.0" rpy="0 0 0"  mujoco_plugin="$(arg mujoco_plugin)" />
+  <xacro:load_zed attach_to="zed" xyz="0.0 0 0.0" rpy="0 0 0" />
   <!-- <joint name="base_footprint_joint" type="fixed">
       <origin xyz="0 0 ${base_length/2 + caster_radius*2}" rpy="0 0 0" />

File: robot_description/frida_description/urdf/xarm/xarm6/xarm6_robot_macro.xacro (robot description, xacro)
@@ -66,12 +66,6 @@
         />
     </xacro:unless>
-    <xacro:xarm6_transmission prefix="${prefix}" hard_interface="${hard_interface}" />
+     <xacro:xarm6_transmission prefix="${prefix}" hard_interface="${hard_interface}" />
     <xacro:xarm6_gazebo prefix="${prefix}" />
-    <xacro:if value="${mujoco_plugin}">
-      <xacro:include filename="$(find frida_description)/urdf/xarm/xarm6/xarm6.mujoco_actuators.xacro"/>
-      <mujoco>
-        <xacro:create_xarm_mujoco_actuators/>
-      </mujoco>
-    </xacro:if>
   </xacro:macro>
 </robot>

File: robot_description/frida_description/urdf/zed/zed.xacro (robot description, xacro)
@@ -33,11 +33,4 @@
     </collision>
   </link>
-  <xacro:if value="${mujoco_plugin}">
-    <mujoco>
-      <reference name="${attach_to}">
-        <camera name="zed_mujoco_camera_link" mode="fixed" fovy="45" quat="-0.5 -0.5 0.5 0.5 "/>
-        </reference>
-    </mujoco>
-  </xacro:if>
 </xacro:macro>
 </robot>

File: robot_description/frida_description/urdf/zed/zed_macro.urdf.xacro (robot description, xacro)
@@ -329,13 +329,4 @@
       </joint>
     </xacro:if>
-    <xacro:if value="${simulation}">
-      <xacro:include filename="$(find frida_description)/urdf/zed/zed_gazebo.xacro"/>
-      <xacro:zed_gazebo prefix="${name}" />
-      <mujoco>
-        <reference name="${name}_left_camera_frame">
-          <camera name="${name}_mujoco_camera" mode="fixed" fovy="45" quat="-0.5 -0.5 0.5 0.5 "/>
-        </reference>
-      </mujoco>
-    </xacro:if>
     <xacro:if value="${enable_gnss}">
       <link name="${name}_gnss_link">

Commit message: dev changes, zed offset, pour gpd fallback

File: robot_description/frida_description/urdf/Gripper/Custom/gripper.xacro (robot description, xacro)
@@ -105,5 +105,5 @@
   <link name="zed"  />
   <joint name="ZED" type="fixed">
-    <origin xyz="0 -0.095626 -0.005" rpy="0 -0.7854 -1.5708" />
+    <origin xyz="0 -0.095626 -0.005" rpy="-0.0494 -0.7360 -1.5139" />
     <parent link="gripper" />
     <child link="zed" />

Commit message: recalibrated zed for better perception

File: robot_description/frida_description/urdf/Gripper/Custom/gripper.xacro (robot description, xacro)
@@ -105,5 +105,5 @@
   <link name="zed"  />
   <joint name="ZED" type="fixed">
-    <origin xyz="0 -0.095626 -0.005" rpy="-0.0494 -0.7360 -1.5139" />
+    <origin xyz="0.0082 -0.0871 0.0025" rpy="0.0061 -0.7922 -1.5632" />
     <parent link="gripper" />
     <child link="zed" />

Commit message: Restore the nominal ZED mount so GPD and geometric picks both work

File: robot_description/frida_description/urdf/Gripper/Custom/gripper.xacro (robot description, xacro)
@@ -105,5 +105,5 @@
   <link name="zed"  />
   <joint name="ZED" type="fixed">
-    <origin xyz="0.0082 -0.0871 0.0025" rpy="0.0061 -0.7922 -1.5632" />
+    <origin xyz="0 -0.095626 -0.005" rpy="0 -0.7854 -1.5708" />
     <parent link="gripper" />
     <child link="zed" />
