Commit message: Calibracion z de ZED (gripper-touch) + ROI del gripper + herramienta (#944)
z-fix del joint ZED (+2.6 cm de residuo de montaje, medido por gripper-touch FK-vs-camara; residuo final ~0). ZED region_of_interest (manual_polygon) enmascara el gripper eye-in-hand en la fuente para que no contamine el octomap. zed_touch_calibrate.py: herramienta de calibracion por toque. Probado en hardware: el pick con ZED paralela ejecuta correctamente.

File: robot_description/frida_description/urdf/Gripper/Custom/gripper_assem.xacro (robot description, xacro)
@@ -111,5 +111,8 @@
     </link>
     <joint name="ZED" type="fixed">
-      <origin xyz="0 -0.0594045903873689 -0.0136964999847231" rpy="1.57079632679489 -1.5707963267949 0" />
+      <!-- xyz: CAD + corrección gripper-touch (#944): +2.5 cm z (residuo de montaje
+           medido con 6 toques FK-vs-cámara, δ_z std 1.7 mm). CAD original era
+           "0 -0.0594045903873689 -0.0136964999847231". rpy intacto. -->
+      <origin xyz="-0.004595226903 -0.0642916212 0.0115921721" rpy="1.57079632679489 -1.5707963267949 0" />
       <parent link="base_gripper" />
       <child link="zed" />
