Commit message: in new base

File: robot_description/frida_description/urdf/zed/zed.xacro (robot description, xacro)
@@ -19,5 +19,5 @@
     </inertial>
     <visual>
-      <origin xyz="0 0 0" rpy="0 0 0" />
+      <origin xyz="-0.03 0 0.01404" rpy="0 0 0" />
       <geometry>
         <mesh filename="${mesh_path}ZED.STL" />
@@ -28,5 +28,5 @@
     </visual>
     <collision>
-      <origin xyz="0 0 0" rpy="0 0 0" />
+      <origin xyz="-0.03 0 0.01404" rpy="0 0 0" />
       <geometry>
         <mesh filename="${mesh_path}ZED.STL" />

Commit message: revert with current main changes

File: robot_description/frida_description/urdf/zed/zed.xacro (robot description, xacro)
@@ -2,4 +2,5 @@
 <robot xmlns:xacro="http://www.ros.org/wiki/xacro">
 <xacro:property name="mesh_path" value="file://$(find frida_description)/urdf/meshes/Gripper/Commercial/" />
+<xacro:property name="black_rgba" value="0.102 0.102 0.102 1" />
 <xacro:macro name="load_zed" params="attach_to:='' xyz:='0 0 0' rpy:='0 0 0' mujoco_plugin:=false" >
     <xacro:unless value="${attach_to == ''}">
@@ -18,5 +19,5 @@
     </inertial>
     <visual>
-      <origin xyz="0 0 0" rpy="0 0 0" />
+      <origin xyz="-0.03 0 0.01404" rpy="0 0 0" />
       <geometry>
         <mesh filename="${mesh_path}ZED.STL" />
@@ -27,5 +28,5 @@
     </visual>
     <collision>
-      <origin xyz="0 0 0" rpy="0 0 0" />
+      <origin xyz="-0.03 0 0.01404" rpy="0 0 0" />
       <geometry>
         <mesh filename="${mesh_path}ZED.STL" />

Commit message: Erase color property

File: robot_description/frida_description/urdf/zed/zed.xacro (robot description, xacro)
@@ -2,5 +2,4 @@
 <robot xmlns:xacro="http://www.ros.org/wiki/xacro">
 <xacro:property name="mesh_path" value="file://$(find frida_description)/urdf/meshes/Gripper/Commercial/" />
-<xacro:property name="black_rgba" value="0.102 0.102 0.102 1" />
 <xacro:macro name="load_zed" params="attach_to:='' xyz:='0 0 0' rpy:='0 0 0' mujoco_plugin:=false" >
     <xacro:unless value="${attach_to == ''}">
