Commit message: fix urdf

File: robot_description/frida_description/urdf/omnibase/FRIDA_Real.urdf.xacro (robot description, xacro)
@@ -80,14 +80,18 @@
     </mujoco>
   </xacro:if>
-  <!-- The world<->base_link offset matters for MoveIt because "world" is the
-       planning frame: the plane-collision-object added by perception_3d in
-       "base_link" gets stored by MoveIt in "world", and pick_server.check_
-       feasibility compares its z against the grasp pose (in "base_link").
-       Any non-zero offset becomes a silent frame mismatch that fails every
-       pick.  On the real robot the 0.3 m pedestal is the physical mounting;
-       in MuJoCo the arm is attached directly to world and there is no
-       pedestal, so pin world<->base_link at identity for sim only. -->
-  <link name="world" />
+  <!-- Planning-frame / TF-root policy:
+       In MuJoCo there is no localization running, so the arm is pinned to a
+       fixed "world" root at identity and "world" is MoveIt's planning frame.
+       On the REAL robot, "base_footprint" is the URDF root and the EKF
+       (robot_localization) drives odom -> base_footprint dynamically. We must
+       NOT add a static world -> base_footprint here: it would give
+       base_footprint two parents (this static one and the EKF's), which TF
+       cannot represent. The EKF transform wins, the world branch is orphaned,
+       and MoveIt's planning frame ("world") gets detached from the live
+       map/odom tree -> ghost robot, place collisions, empty octomap. So on the
+       real robot base_footprint is both the URDF root and MoveIt's planning
+       frame, and it stays connected to map via the EKF. -->
   <xacro:if value="$(arg mujoco_plugin)">
+    <link name="world" />
     <joint name="world_to_base" type="fixed">
       <parent link="world" />
@@ -96,11 +100,4 @@
     </joint>
   </xacro:if>
-  <xacro:unless value="$(arg mujoco_plugin)">
-    <joint name="world_to_base" type="fixed">
-      <parent link="world" />
-      <child link="base_footprint" />
-      <origin rpy="0 0 0" xyz="0 0 0.3" />
-    </joint>
-  </xacro:unless>
   <!-- XARM MACRO -->
   <xacro:include filename="$(find frida_description)/urdf/xarm/xarm_device_macro.xacro" />

Commit message: fix urdf (#1052)
* fix urdf

* rm comments

* fix

File: robot_description/frida_description/urdf/omnibase/FRIDA_Real.urdf.xacro (robot description, xacro)
@@ -80,14 +80,6 @@
     </mujoco>
   </xacro:if>
-  <!-- The world<->base_link offset matters for MoveIt because "world" is the
-       planning frame: the plane-collision-object added by perception_3d in
-       "base_link" gets stored by MoveIt in "world", and pick_server.check_
-       feasibility compares its z against the grasp pose (in "base_link").
-       Any non-zero offset becomes a silent frame mismatch that fails every
-       pick.  On the real robot the 0.3 m pedestal is the physical mounting;
-       in MuJoCo the arm is attached directly to world and there is no
-       pedestal, so pin world<->base_link at identity for sim only. -->
-  <link name="world" />
   <xacro:if value="$(arg mujoco_plugin)">
+    <link name="world" />
     <joint name="world_to_base" type="fixed">
       <parent link="world" />
@@ -96,11 +88,4 @@
     </joint>
   </xacro:if>
-  <xacro:unless value="$(arg mujoco_plugin)">
-    <joint name="world_to_base" type="fixed">
-      <parent link="world" />
-      <child link="base_footprint" />
-      <origin rpy="0 0 0" xyz="0 0 0.3" />
-    </joint>
-  </xacro:unless>
   <!-- XARM MACRO -->
   <xacro:include filename="$(find frida_description)/urdf/xarm/xarm_device_macro.xacro" />
