Commit message: Remove world link and world_to_base joint from FRIDA_Real.urdf.xacro

File: robot_description/frida_description/urdf/omnibase/FRIDA_Real.urdf.xacro (robot description, xacro)
@@ -43,11 +43,4 @@
   <!-- ROBOT COMPONENTS -->
   <xacro:include filename="$(find frida_description)/urdf/omnibase/robot.xacro"/>
-  <!-- World link and static transform for real hardware/planning frame -->
-  <link name="world" />
-  <joint name="world_to_base" type="fixed">
-    <parent link="world" />
-    <child link="base_link" />
-    <origin rpy="0 0 0" xyz="0 0 0" />
-  </joint>
   <!-- XARM MACRO -->
   <xacro:include filename="$(find frida_description)/urdf/xarm/xarm_device_macro.xacro" />
