Commit message: done2

File: robot_description/frida_description/urdf/omnibase/robot.xacro (robot description, xacro)
@@ -21,5 +21,5 @@
   <link name="${prefix}_base_footprint"/>
   <joint name="${prefix}_base_footprint_joint" type="fixed">
-    <origin xyz="0 0 0.0385" rpy="0 0 90"/>
+    <origin xyz="0 0 0.0385" rpy="0 0 0"/>
     <parent link="${prefix}_base_footprint"/>
     <child link="${prefix}_base_link"/>

Commit message: use_sim_time changes

File: robot_description/frida_description/urdf/omnibase/robot.xacro (robot description, xacro)
@@ -67,10 +67,19 @@
     </collision>
   </link>
-  <joint name="wheel_FL_joint" type="continuous">
-    <origin xyz="0.184790699909997 0.219394995052441 0.0376959841787657" rpy="-1.5707963267949 0 0"/>
-    <parent link="base_link"/>
-    <child link="wheel_FL"/>
-    <axis xyz="0 0 1"/>
-  </joint>
+  <xacro:if value="${use_sim_time}">
+    <joint name="wheel_FL_joint" type="continuous">
+      <origin xyz="0.184790699909997 0.219394995052441 0.0376959841787657" rpy="-1.5707963267949 0 0"/>
+      <parent link="base_link"/>
+      <child link="wheel_FL"/>
+      <axis xyz="0 0 1"/>
+    </joint>
+  </xacro:if>
+  <xacro:unless value="${use_sim_time}">
+    <joint name="wheel_FL_joint" type="fixed">
+      <origin xyz="0.184790699909997 0.219394995052441 0.0376959841787657" rpy="-1.5707963267949 0 0"/>
+      <parent link="base_link"/>
+      <child link="wheel_FL"/>
+    </joint>
+  </xacro:unless>
   <!-- =================== wheel_FR =================== -->
   <link name="wheel_FR">
@@ -95,10 +104,19 @@
     </collision>
   </link>
-  <joint name="wheel_FR_joint" type="continuous">
-    <origin xyz="0.184790699909996 -0.219395004947559 0.0376959841787653" rpy="-1.5707963267949 0 0"/>
-    <parent link="base_link"/>
-    <child link="wheel_FR"/>
-    <axis xyz="0 0 1"/>
-  </joint>
+  <xacro:if value="${use_sim_time}">
+    <joint name="wheel_FR_joint" type="continuous">
+      <origin xyz="0.184790699909996 -0.219395004947559 0.0376959841787653" rpy="-1.5707963267949 0 0"/>
+      <parent link="base_link"/>
+      <child link="wheel_FR"/>
+      <axis xyz="0 0 1"/>
+    </joint>
+  </xacro:if>
+  <xacro:unless value="${use_sim_time}">
+    <joint name="wheel_FR_joint" type="fixed">
+      <origin xyz="0.184790699909996 -0.219395004947559 0.0376959841787653" rpy="-1.5707963267949 0 0"/>
+      <parent link="base_link"/>
+      <child link="wheel_FR"/>
+    </joint>
+  </xacro:unless>
   <!-- =================== wheel_RL =================== -->
   <link name="wheel_RL">
@@ -123,10 +141,19 @@
     </collision>
   </link>
-  <joint name="wheel_RL_joint" type="continuous">
-    <origin xyz="-0.184790699909991 0.219394995052441 0.0376959841787652" rpy="-1.5707963267949 0 0"/>
-    <parent link="base_link"/>
-    <child link="wheel_RL"/>
-    <axis xyz="0 0 1"/>
-  </joint>
+  <xacro:if value="${use_sim_time}">
+    <joint name="wheel_RL_joint" type="continuous">
+      <origin xyz="-0.184790699909991 0.219394995052441 0.0376959841787652" rpy="-1.5707963267949 0 0"/>
+      <parent link="base_link"/>
+      <child link="wheel_RL"/>
+      <axis xyz="0 0 1"/>
+    </joint>
+  </xacro:if>
+  <xacro:unless value="${use_sim_time}">
+    <joint name="wheel_RL_joint" type="fixed">
+      <origin xyz="-0.184790699909991 0.219394995052441 0.0376959841787652" rpy="-1.5707963267949 0 0"/>
+      <parent link="base_link"/>
+      <child link="wheel_RL"/>
+    </joint>
+  </xacro:unless>
   <!-- =================== wheel_RR =================== -->
   <link name="wheel_RR">
@@ -151,10 +178,19 @@
     </collision>
   </link>
-  <joint name="wheel_RR_joint" type="continuous">
-    <origin xyz="-0.184790699909991 -0.219395004947559 0.0376959841787661" rpy="-1.5707963267949 0 0"/>
-    <parent link="base_link"/>
-    <child link="wheel_RR"/>
-    <axis xyz="0 0 1"/>
-  </joint>
+  <xacro:if value="${use_sim_time}">
+    <joint name="wheel_RR_joint" type="continuous">
+      <origin xyz="-0.184790699909991 -0.219395004947559 0.0376959841787661" rpy="-1.5707963267949 0 0"/>
+      <parent link="base_link"/>
+      <child link="wheel_RR"/>
+      <axis xyz="0 0 1"/>
+    </joint>
+  </xacro:if>
+  <xacro:unless value="${use_sim_time}">
+    <joint name="wheel_RR_joint" type="fixed">
+      <origin xyz="-0.184790699909991 -0.219395004947559 0.0376959841787661" rpy="-1.5707963267949 0 0"/>
+      <parent link="base_link"/>
+      <child link="wheel_RR"/>
+    </joint>
+  </xacro:unless>
   <!-- =================== lidar_front =================== -->
   <link name="lidar_front">

Commit message: Update stl

File: robot_description/frida_description/urdf/omnibase/robot.xacro (robot description, xacro)
@@ -41,5 +41,7 @@
       <origin xyz="0 0 0" rpy="0 0 0"/>
       <geometry>
-        <mesh filename="${mesh_dir}/base_link.STL"/>
+        <!-- decimated collision mesh (~3.9k tris) to avoid MoveIt/FCL
+             "too many vertices in collision geometry" on the 430k visual mesh -->
+        <mesh filename="${mesh_dir}/base_link_collision.stl"/>
       </geometry>
     </collision>
@@ -63,5 +65,6 @@
       <origin xyz="0 0 0" rpy="0 0 0"/>
       <geometry>
-        <mesh filename="${mesh_dir}/wheel.STL"/>
+        <!-- cylinder collision mesh (~190 tris) replacing the 264k visual mesh -->
+        <mesh filename="${mesh_dir}/wheel_collision.stl"/>
       </geometry>
     </collision>
@@ -100,5 +103,6 @@
       <origin xyz="0 0 0" rpy="0 0 0"/>
       <geometry>
-        <mesh filename="${mesh_dir}/wheel.STL"/>
+        <!-- cylinder collision mesh (~190 tris) replacing the 264k visual mesh -->
+        <mesh filename="${mesh_dir}/wheel_collision.stl"/>
       </geometry>
     </collision>
@@ -137,5 +141,6 @@
       <origin xyz="0 0 0" rpy="0 0 0"/>
       <geometry>
-        <mesh filename="${mesh_dir}/wheel.STL"/>
+        <!-- cylinder collision mesh (~190 tris) replacing the 264k visual mesh -->
+        <mesh filename="${mesh_dir}/wheel_collision.stl"/>
       </geometry>
     </collision>
@@ -174,5 +179,6 @@
       <origin xyz="0 0 0" rpy="0 0 0"/>
       <geometry>
-        <mesh filename="${mesh_dir}/wheel.STL"/>
+        <!-- cylinder collision mesh (~190 tris) replacing the 264k visual mesh -->
+        <mesh filename="${mesh_dir}/wheel_collision.stl"/>
       </geometry>
     </collision>

Commit message: Update color

File: robot_description/frida_description/urdf/omnibase/robot.xacro (robot description, xacro)
@@ -1,4 +1,5 @@
 <?xml version="1.0"?>
 <robot name="home_base" xmlns:xacro="http://ros.org/wiki/xacro">
+  <xacro:property name="black_rgba" value="0.102 0.102 0.102 1" />
   <!-- Launch arguments -->
   <xacro:arg name="use_sim_time" default="false"/>

Commit message: Update laser urdf

File: robot_description/frida_description/urdf/omnibase/robot.xacro (robot description, xacro)
@@ -223,5 +223,5 @@
   </link>
   <joint name="lidar_front_joint" type="fixed">
-    <origin xyz="0.287749512711774 -0.207249957761446 0.135795984178765" rpy="0 0 -1.5707963267949"/>
+    <origin xyz="0.287749512711774 -0.207249957761446 0.135795984178765" rpy="0 0 1.57"/>
     <parent link="base_link"/>
     <child link="lidar_front"/>
@@ -250,5 +250,5 @@
   </link>
   <joint name="lidar_rear_joint" type="fixed">
-    <origin xyz="-0.287749512711767 0.207249947866326 0.135795984178765" rpy="0 0 1.5707963267949"/>
+    <origin xyz="-0.287749512711767 0.207249947866326 0.135795984178765" rpy="0 0 -1.57"/>
     <parent link="base_link"/>
     <child link="lidar_rear"/>

Commit message: place dlc

File: robot_description/frida_description/urdf/omnibase/robot.xacro (robot description, xacro)
@@ -17,11 +17,4 @@
     <color rgba="0.792156862745098 0.819607843137255 0.933333333333333 1"/>
   </material>
-  <!-- =================== base_footprint (root) =================== -->
-  <link name="base_footprint"/>
-  <joint name="base_footprint_joint" type="fixed">
-    <origin xyz="0 0 0.0385" rpy="0 0 0"/>
-    <parent link="base_footprint"/>
-    <child link="base_link"/>
-  </joint>
   <!-- =================== base_link =================== -->
   <link name="base_link">

Commit message: clean

File: robot_description/frida_description/urdf/omnibase/robot.xacro (robot description, xacro)
@@ -17,4 +17,11 @@
     <color rgba="0.792156862745098 0.819607843137255 0.933333333333333 1"/>
   </material>
+    <!-- =================== base_footprint (root) =================== -->
+  <link name="base_footprint"/>
+  <joint name="base_footprint_joint" type="fixed">
+    <origin xyz="0 0 0.0385" rpy="0 0 0"/>
+    <parent link="base_footprint"/>
+    <child link="base_link"/>
+  </joint>
   <!-- =================== base_link =================== -->
   <link name="base_link">
