Commit message: A2 sim: head-mounted ZED, angle-bracket top-down grasps, self-filtered cloud and clamped start state

File: robot_description/frida_description/urdf/omnibase/FRIDA_A2.urdf.xacro (robot description, xacro)
@@ -4,6 +4,8 @@
   <xacro:arg name="shoulder_height" default="0.5"/>
   <xacro:arg name="shoulder_y" default="0.06"/>
-  <xacro:arg name="flange_z" default="0.095"/>
+  <xacro:arg name="flange_z" default="0.13"/>
   <xacro:arg name="flange_yaw" default="-1.5708"/>
+  <!-- Angle bracket between the A2 flange and the gripper (0 = gripper in line with the forearm); flange_z includes its length -->
+  <xacro:arg name="flange_pitch" default="-1.5708"/>
   <xacro:property name="shoulder_height" value="$(arg shoulder_height)"/>
   <xacro:property name="shoulder_y" value="$(arg shoulder_y)"/>
@@ -64,5 +66,5 @@
     <parent link="openarm_right_link7"/>
     <child link="link_eef"/>
-    <origin xyz="0 0 $(arg flange_z)" rpy="0 0 $(arg flange_yaw)"/>
+    <origin xyz="0 0 $(arg flange_z)" rpy="0 $(arg flange_pitch) $(arg flange_yaw)"/>
   </joint>
   <joint name="gripper_grasp_joint" type="fixed">
@@ -72,8 +74,15 @@
   </joint>
   <link name="gripper_grasp_frame"/>
-  <!-- FRIDA custom gripper and wrist ZED, same mounting as on the xArm flange -->
+  <!-- FRIDA custom gripper, same mounting as on the xArm flange -->
   <xacro:include filename="$(find frida_description)/urdf/Gripper/Custom/gripper.xacro"/>
   <xacro:load_gripper attach_to="link_eef" xyz="0 0 0.046" rpy="0 0 3.926" fixed_joints="false" ros2_control_plugin="none"/>
+  <!-- ZED on a head bracket above the shoulders, pitched down at the table in front of the right arm -->
+  <link name="a2_head"/>
+  <joint name="a2_head_joint" type="fixed">
+    <parent link="a2_shoulder_mount"/>
+    <child link="a2_head"/>
+    <origin xyz="0.05 0 0.25" rpy="0 0.9 -0.6"/>
+  </joint>
   <xacro:include filename="$(find frida_description)/urdf/zed/zed.xacro"/>
-  <xacro:load_zed attach_to="zed" xyz="0.0 0 0.0" rpy="0 0 0"/>
+  <xacro:load_zed attach_to="a2_head" xyz="0.0 0 0.0" rpy="0 0 0"/>
 </robot>
