Commit message: Add navigation to the Gazebo sim: arena from the robocup2026_1 map, mobile base and nav_central

File: simulation/frida_gz_sim/urdf/frida_gz.urdf.xacro (robot description, xacro)
@@ -5,13 +5,74 @@
   <xacro:arg name="image_height" default="360"/>
   <xacro:arg name="camera_rate" default="10"/>
+  <!-- Mobile base: drop the world anchor and add the gz drive, odometry and lidars -->
+  <xacro:arg name="mobile_base" default="false"/>
+  <xacro:arg name="cmd_vel_topic" default="/sim/cmd_vel"/>
+  <xacro:arg name="lidar_rate" default="10"/>
+  <xacro:property name="mobile_base" value="$(arg mobile_base)"/>
   <!-- Real robot description; pass ros2_control_plugin:=gz_ros2_control/GazeboSimSystem -->
   <xacro:include filename="$(find frida_description)/urdf/omnibase/FRIDA_Real.urdf.xacro"/>
-  <!-- Static base: the sim does not navigate -->
-  <link name="world"/>
-  <joint name="world_to_base_link" type="fixed">
-    <parent link="world"/>
-    <child link="base_link"/>
-    <origin xyz="0 0 0" rpy="0 0 0"/>
-  </joint>
+  <!-- Static base for the manipulation worlds; the nav worlds drive base_link instead -->
+  <xacro:unless value="${mobile_base}">
+    <link name="world"/>
+    <joint name="world_to_base_link" type="fixed">
+      <parent link="world"/>
+      <child link="base_link"/>
+      <origin xyz="0 0 0" rpy="0 0 0"/>
+    </joint>
+  </xacro:unless>
+  <xacro:if value="${mobile_base}">
+    <!-- Holonomic drive: gz sets the base velocity directly, like the mecanum base does -->
+    <gazebo>
+      <plugin filename="gz-sim-velocity-control-system" name="gz::sim::systems::VelocityControl">
+        <topic>$(arg cmd_vel_topic)</topic>
+      </plugin>
+      <plugin filename="gz-sim-odometry-publisher-system" name="gz::sim::systems::OdometryPublisher">
+        <odom_frame>odom</odom_frame>
+        <robot_base_frame>base_link</robot_base_frame>
+        <odom_topic>/sim/odom</odom_topic>
+        <tf_topic>/sim/odom_tf</tf_topic>
+        <odom_publish_frequency>50</odom_publish_frequency>
+        <dimensions>2</dimensions>
+      </plugin>
+    </gazebo>
+    <!-- The base is velocity-driven, so gravity would only fight the controller -->
+    <gazebo reference="base_link">
+      <gravity>false</gravity>
+    </gazebo>
+    <!-- RPLIDAR C1 pair. Each one is blind over the ~90 deg wedge its own chassis
+         covers, the same wedge the real driver drops with ignore_array. -->
+    <xacro:macro name="omni_lidar" params="link topic">
+      <gazebo reference="${link}">
+        <sensor name="${link}_scan" type="gpu_lidar">
+          <always_on>true</always_on>
+          <update_rate>$(arg lidar_rate)</update_rate>
+          <topic>${topic}</topic>
+          <gz_frame_id>${link}</gz_frame_id>
+          <lidar>
+            <scan>
+              <horizontal>
+                <samples>370</samples>
+                <resolution>1</resolution>
+                <min_angle>1.6057</min_angle>
+                <max_angle>6.2483</max_angle>
+              </horizontal>
+            </scan>
+            <range>
+              <min>0.20</min>
+              <max>12.0</max>
+              <resolution>0.01</resolution>
+            </range>
+            <noise>
+              <type>gaussian</type>
+              <mean>0.0</mean>
+              <stddev>0.01</stddev>
+            </noise>
+          </lidar>
+        </sensor>
+      </gazebo>
+    </xacro:macro>
+    <xacro:omni_lidar link="lidar_front" topic="scan_front"/>
+    <xacro:omni_lidar link="lidar_rear" topic="scan_rear"/>
+  </xacro:if>
   <!-- Gripper fingers, both commanded directly (no mimic in sim) -->
   <ros2_control name="FridaGripperSystem" type="system">

Commit message: Add Agility A2 dual arm to the FRIDA Gazebo sim behind FRIDA_ARM=a2

File: simulation/frida_gz_sim/urdf/frida_gz.urdf.xacro (robot description, xacro)
@@ -10,6 +10,15 @@
   <xacro:arg name="lidar_rate" default="10"/>
   <xacro:property name="mobile_base" value="$(arg mobile_base)"/>
+  <!-- Arm on the robot: xarm6 (current hardware) or a2 (Agility A2 / OpenArm dual arm) -->
+  <xacro:arg name="arm" default="xarm6"/>
+  <xacro:property name="arm" value="$(arg arm)"/>
   <!-- Real robot description; pass ros2_control_plugin:=gz_ros2_control/GazeboSimSystem -->
-  <xacro:include filename="$(find frida_description)/urdf/omnibase/FRIDA_Real.urdf.xacro"/>
+  <xacro:if value="${arm == 'xarm6'}">
+    <xacro:include filename="$(find frida_description)/urdf/omnibase/FRIDA_Real.urdf.xacro"/>
+  </xacro:if>
+  <xacro:if value="${arm == 'a2'}">
+    <xacro:include filename="$(find frida_description)/urdf/omnibase/FRIDA_A2.urdf.xacro"/>
+    <xacro:include filename="$(find frida_gz_sim)/urdf/a2_gz.xacro"/>
+  </xacro:if>
   <!-- Static base for the manipulation worlds; the nav worlds drive base_link instead -->
   <xacro:unless value="${mobile_base}">
@@ -105,10 +114,16 @@
     </gazebo>
   </xacro:macro>
-  <xacro:no_gravity link="link1"/>
-  <xacro:no_gravity link="link2"/>
-  <xacro:no_gravity link="link3"/>
-  <xacro:no_gravity link="link4"/>
-  <xacro:no_gravity link="link5"/>
-  <xacro:no_gravity link="link6"/>
+  <xacro:if value="${arm == 'xarm6'}">
+    <xacro:no_gravity link="link1"/>
+    <xacro:no_gravity link="link2"/>
+    <xacro:no_gravity link="link3"/>
+    <xacro:no_gravity link="link4"/>
+    <xacro:no_gravity link="link5"/>
+    <xacro:no_gravity link="link6"/>
+  </xacro:if>
+  <xacro:if value="${arm == 'a2'}">
+    <xacro:a2_no_gravity side="right" index="1"/>
+    <xacro:a2_no_gravity side="left" index="1"/>
+  </xacro:if>
   <!-- Grippy finger pads -->
   <xacro:macro name="finger_pad" params="link">
